File: usb_hub.kicad_sch (KiCad schematic)
At the start: 32 parts, among them U25 RTS5411S-GR, Y3 K3A120002010

Commit message: Add files via upload
Parts:
- C204: renamed from C146; value 100n -> 1u
- C205: renamed from C147; value 100n -> 1u
- C206: renamed from C148; value 100n -> 1u
- C207: renamed from C149; value 100n -> 1u
- C209: renamed from C151; value 100n -> 1u
- C211: renamed from C153; value 100n -> 1u
- C212: renamed from C154; value 100n -> 1u
- C213: renamed from C155; value 100n -> 1u
- C214: renamed from C156; value 100n -> 1u
- C215: renamed from C157; value 100n -> 1u
- C216: renamed from C158; value 100n -> 1u
- C217: renamed from C159; value 100n -> 1u
- C218: renamed from C160; value 100n -> 1u
- C219: renamed from C161; value 100n -> 1u
- C220: renamed from C162; value 100n -> 1u
- C221: renamed from C163; value 100n -> 1u
- C222: renamed from C164; value 100n -> 1u
- C225: renamed from C167; value 100n -> 1u
- C226: renamed from C168; value 100n -> 1u
- C227: renamed from C169; value ??? -> 20pF
- C228: renamed from C170; value ??? -> 20pF
- renumbered C150 to C208, C152 to C210, C165 to C223, C166 to C224, L4 to L11, R88 to R73, R89 to R74, R90 to R75, R91 to R76, U25 to U16
Other:
- note added: "Large cpacitor"
- moved on the sheet: C204, C205, C206, C207, C211, C212, C213, C214, C215, C216, C217, C218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
