File: usb_power.kicad_sch (KiCad schematic)
At the start: 12 parts, among them J7 USB_C_Receptacle_PowerOnly_6P, U33 AP2553W6-7

Commit message: Add files via upload
Parts:
- removed D23: PESD5V0S1BA, PCM_Diode_SMD_AKL:D_SOD-323_TVS, symbol PCM_Diode_TVS_AKL:PESD5V0S1BA
- removed R166: 10k, PCM_Resistor_SMD_AKL:R_0402_1005Metric, symbol Device:R_Small
- removed R168: 100k, PCM_Resistor_SMD_AKL:R_0402_1005Metric, symbol Device:R_Small
- removed U33: AP2553W6-7, symbol New_Library:AP2553W6-7
- added C365: 1u, Capacitor_SMD:C_0402_1005Metric_Pad0.74x0.62mm_HandSolder, symbol New_Library_0:C_Small_edited
- added D18: SMBJ5.0CA, PCM_Diode_SMD_AKL:D_SMB_TVS, symbol PCM_Diode_TVS_AKL:SMBJ5.0CA
- added R45: 100k, PCM_Resistor_SMD_AKL:R_0402_1005Metric, symbol Device:R_Small
- added U29: ETA7014S2G, PCM_Package_TO_SOT_SMD_AKL:TSOT-23-6, symbol New_Library:ETA7014S2G
- renumbered C406 to C163, C69 to C164, J7 to J2, R167 to R43, R169 to R44, R51 to R47, R52 to R48, R117 to R49
Connections:
- net GND: now also C365.2, D18.1 (K), U29.6 (GND)
- net Vbus_USB_{PWR}: now also U29.3 (OUT)
- net at C164.1, J2.A9 (VBUS), J2.B9 (VBUS): now also D18.2 (A), R45.1, U29.2 (EN), U29.4 (IN)
- new net: C365.1, R45.2, U29.5 (VCC)
Other:
- note removed: "We have Error, The MAX current is 2.1A"
- moved on the sheet: C163, C164, R43, R44
