File: 40pin_header.kicad_sch (KiCad schematic)
At the start: 5 parts, among them J13 Raspberry_Pi_4

Commit message: Add files via upload
Parts:
- added D27, D28: SMBJ5.0CA, PCM_Diode_SMD_AKL:D_SMB_TVS, symbol PCM_Diode_TVS_AKL:SMBJ5.0CA
- added J15: JST_03, Connector:FanPinHeader_1x03_P2.54mm_Vertical, symbol PCM_SL_Connectors:JST_03
- added R176: 22R, PCM_Resistor_SMD_AKL:R_0402_1005Metric_Pad0.72x0.64mm, symbol Device:R_Small
- renumbered C333 to C361, C334 to C362, R137 to R155, R138 to R156
Connections:
- net GND: now also D27.1 (K), D28.1 (K), J15.3
- new net: D28.2 (A), J15.2, R176.2
- new net PWM_FAN: R176.1
- new net VCC5V0_SYS: D27.2 (A), J15.1

Commit message: SBC Board V0.2
The SBC schematics before footprint and part number check
Parts:
- removed C361, C362: 22u, Capacitor_SMD:C_0402_1005Metric_Pad0.74x0.62mm_HandSolder, symbol New_Library_0:C_Small_edited
- added C372, C374: 1u, Capacitor_SMD:C_0402_1005Metric_Pad0.74x0.62mm_HandSolder, symbol New_Library_0:C_Small_edited
- added C373, C375: 22u, Capacitor_SMD:C_0603_1608Metric, symbol New_Library_0:C_Small_edited
- added D18, D19: SMBJ5.0CA, PCM_Diode_SMD_AKL:D_SMB_TVS, symbol PCM_Diode_TVS_AKL:SMBJ5.0CA
- added R164, R167: 2.2k, PCM_Resistor_SMD_AKL:R_0402_1005Metric, symbol Device:R_Small
- added R165, R168: 15k, PCM_Resistor_SMD_AKL:R_0402_1005Metric, symbol Device:R_Small
- added R166, R169: 100k, PCM_Resistor_SMD_AKL:R_0402_1005Metric, symbol Device:R_Small
- added U33, U34: AP2553W6-7, symbol New_Library:AP2553W6-7
- renumbered D28 to D20, D27 to D21, J13 to J12, J15 to J13, R155 to R170, R156 to R171, R176 to R172
Connections:
- net +3.3V_{GPIO}: now also C375.1, D19.2 (A), U34.6 (OUT)
- net +5V_{GPIO}: now also C373.1, D18.2 (A), U33.6 (OUT)
- net GND: now also C372.2, C373.2, C374.2, C375.2, D18.1 (K), D19.1 (K), R165.2, R166.2, R168.2, R169.2, U33.2 (GND), U34.2 (GND)
- net VCC5V0_SYS: now also C372.1, U33.1 (IN)
- new net: R165.1, U33.5 (ILIM)
- new net: R164.1, R166.1, U33.3 (EN)
- new net: R168.1, U34.5 (ILIM)
- new net: R167.1, R169.1, U34.3 (EN)
- new net 40GPIOs_PWR_EN: R164.2, R167.2
- new net VCCA_3V3_S0: C374.1, U34.1 (IN)
- no-connect marks 0 -> 2
Other:
- moved on the sheet: D20, D21, J12, J13, R170, R171, R172

Commit message: SBCv0.3
there is no big thing update just some LCSC & Mouser parts
and Big problem deleted alot of component values (:
Parts:
- C372, C374: footprint Capacitor_SMD:C_0402_1005Metric_Pad0.74x0.62mm_HandSolder -> Capacitor_SMD:C_0201_0603Metric_Pad0.64x0.40mm_HandSolder; LCSC Part (none) -> C5209398; Mouser Part (none) -> CL03A105KP3NSNC
- C373, C375: LCSC Part (none) -> C86295; Mouser Part (none) -> CL10A226MP8NUNE
- D18, D19, D20, D21: LCSC Part (none) -> C113975; Mouser Part (none) -> 581-SMBJ5.0CA
- J12: value Raspberry_Pi_4 -> B-2100S40P-B110; LCSC Part (none) -> C124383
- J13: value JST_03 -> B3B-XH-A(LF)(SN); LCSC Part (none) -> C144394
- R164, R167: value 2.2k -> (none); LCSC Part (none) -> (do_not_autoplace no)
- R165, R168: value 15k -> (none); LCSC Part (none) -> (hide yes)
- R166, R169: value 100k -> (none); LCSC Part (none) -> (show_name no)
- R170, R171: value 10K -> (none); LCSC Part (none) -> )
- R172: value 22R -> (property "Description" "Unpolarized capacitor, small symbol"
- U33, U34: footprint (none) -> Package_TO_SOT_SMD:SOT-23-6_Handsoldering; LCSC Part (none) -> C212302; Mouser Part (none) -> 621-AP2553W6-7

Commit message: SBCv0.4
add LCSC & Mouser parts 
and solve the deleted value in the past version
Parts:
- R164, R167: value (none) -> 2.2k; LCSC Part (do_not_autoplace no) -> C114762; Mouser Part (none) -> 603-RC0402FR-072K2L
- R165, R168: value (none) -> 15k; LCSC Part (hide yes) -> C114761; Mouser Part (none) -> 603-RC0402FR-0715KL
- R166, R169: value (none) -> 100k; LCSC Part (show_name no) -> C60491; Mouser Part (none) -> 603-RC0402FR-07100KL
- R170, R171: value (none) -> 10K; footprint PCM_Resistor_SMD_AKL:R_0402_1005Metric_Pad0.72x0.64mm -> PCM_Resistor_SMD_AKL:R_0402_1005Metric; LCSC Part ) -> C60490; Mouser Part (none) -> 603-RC0402FR-0710KL
- R172: value (property "Description" "Unpolarized capacitor, small symbol" -> 22R; footprint PCM_Resistor_SMD_AKL:R_0402_1005Metric_Pad0.72x0.64mm -> PCM_Resistor_SMD_AKL:R_0402_1005Metric; LCSC Part (none) -> C114765; Mouser Part (none) -> 603-RC0402FR-0722RL
