File: ethernet.kicad_sch (KiCad schematic)
At the start: 42 parts, among them J5 POE Connector, J6 LPJG0926HENL, U19 RTL8211F-CG, Y1 SX32Y025000BC1T001

Commit message: Add files via upload
Parts:
- removed R47, R48: 510R, PCM_Resistor_SMD_AKL:R_0402_1005Metric, symbol Device:R_Small
- added R104, R107: 510R, PCM_Resistor_SMD_AKL:R_0402_1005Metric_Pad0.72x0.64mm, symbol Device:R_Small
- added R84, R86, R87, R89, R91, R93, R95, R97: 0R, PCM_Resistor_SMD_AKL:R_0402_1005Metric_Pad0.72x0.64mm, symbol Device:R_Small
- C291: renamed from C91; value 100n -> 1u
- C292: renamed from C92; value 100n -> 1u
- C293: renamed from C93; value 100n -> 1u
- C294: renamed from C94; value 100n -> 1u
- C295: renamed from C95; value 100n -> 1u
- C297: renamed from C396; value 100n -> 1u
- C299: renamed from C97; value 100n -> 1u
- C301: renamed from C99; value 100n -> 1u
- C302: renamed from C100; value ??? -> 18pF
- C303: renamed from C101; value ??? -> 18pF
- C304: renamed from C102; value 100n -> 1u
- J6: renamed from J5; footprint Connector_PinHeader_1.00mm:PinHeader_2x02_P1.00mm_Vertical -> Connector_PinHeader_2.54mm:PinHeader_2x02_P2.54mm_Vertical
- renumbered C96 to C296, C397 to C298, C98 to C300, C103 to C305, J6 to J7, L1 to L12, R39 to R100, R40 to R101, R41 to R102, R44 to R103, R45 to R105, R46 to R106, R27 to R78, R28 to R79, R29 to R80, R30 to R81, R31 to R82, R32 to R83, R33 to R85, R34 to R88, R35 to R90, R36 to R92, R37 to R94, R42 to R96, R43 to R98, R38 to R99, U19 to U18, Y1 to Y4
Connections:
- net +3.3V: now also R104.2
- net ETH_{PHY}_MDI[0]-: now also R86.1; no longer U18.2 (MDIN0)
- net ETH_{PHY}_MDI[1]+: now also R84.1; no longer U18.1 (MDIP0)
- net ETH_{PHY}_MDI[2]+: now also R87.1; no longer U18.4 (MDIP1)
- net ETH_{PHY}_MDI[2]-: now also R89.1; no longer U18.5 (MDIN1)
- net ETH_{PHY}_MDI[3]+: now also R91.1; no longer U18.6 (MDIP2)
- net ETH_{PHY}_MDI[3]-: now also R93.1; no longer U18.7 (MDIN2)
- net ETH_{PHY}_MDI[4]+: now also R95.1; no longer U18.9 (MDIP3)
- net ETH_{PHY}_MDI[4]-: now also R97.1; no longer U18.10 (MDIN3)
- net PHY_LED2: now also R107.2
- net at J7.18: now also R107.1
- net at J7.16: now also R104.1
- new net: R89.2, U18.5 (MDIN1)
- new net: R95.2, U18.9 (MDIP3)
- new net: R97.2, U18.10 (MDIN3)
- new net: R93.2, U18.7 (MDIN2)
- new net: R87.2, U18.4 (MDIP1)
- new net: R84.2, U18.1 (MDIP0)
- new net: R86.2, U18.2 (MDIN0)
- new net: R91.2, U18.6 (MDIP2)

Commit message: SBC Board V0.2
The SBC schematics before footprint and part number check
Parts:
- removed C304: 1u, Capacitor_SMD:C_0201_0603Metric_Pad0.64x0.40mm_HandSolder, symbol New_Library_0:C_Small_edited
- removed C305: 1u, Capacitor_SMD:C_0402_1005Metric_Pad0.74x0.62mm_HandSolder, symbol New_Library_0:C_Small_edited
- removed J6: POE Connector, Connector_PinHeader_2.54mm:PinHeader_2x02_P2.54mm_Vertical, symbol Connector_Generic:Conn_01x04
- removed J7: LPJG0926HENL, LPJG0926HENL:LINK-PP_LPJG0926HENL, symbol LPJG0926HENL:LPJG0926HENL
- removed R104, R107: 510R, PCM_Resistor_SMD_AKL:R_0402_1005Metric_Pad0.72x0.64mm, symbol Device:R_Small
- added C308: 1u, Capacitor_SMD:C_0201_0603Metric_Pad0.64x0.40mm_HandSolder, symbol New_Library_0:C_Small_edited
- added C309: 1u, Capacitor_SMD:C_0402_1005Metric_Pad0.74x0.62mm_HandSolder, symbol New_Library_0:C_Small_edited
- added J5: POE Connector, Connector_PinHeader_2.54mm:PinHeader_2x02_P2.54mm_Vertical, symbol Connector_Generic:Conn_01x04
- added J6: LPJG0926HENL, LPJG0926HENL:LINK-PP_LPJG0926HENL, symbol LPJG0926HENL:LPJG0926HENL
- added R76, R80: 510R, PCM_Resistor_SMD_AKL:R_0402_1005Metric_Pad0.72x0.64mm, symbol Device:R_Small
- renumbered C291 to C300, C292 to C301, C293 to C302, C294 to C303, C295 to C304, C296 to C305, C297 to C306, C298 to C307, C299 to C310, C300 to C311, C301 to C312, C302 to C313, C303 to C314, R105 to R100, R106 to R101, R78 to R72, R79 to R73, R80 to R74, R81 to R75, R82 to R77, R83 to R78, R85 to R79, R84 to R81, R86 to R82, R87 to R83, R88 to R84, R89 to R85, R90 to R86, R91 to R87, R92 to R88, R93 to R89, R94 to R90, R95 to R91, R96 to R92, R97 to R93, R98 to R94, R99 to R95, R100 to R96, R101 to R97, R102 to R98, R103 to R99, U18 to U19
Connections:
- net +3.3V: now also R76.2
- net ETH_{PHY}_MDI[0]-: now also J6.2 (TD1-)
- net ETH_{PHY}_MDI[1]+: now also J6.1 (TD1+)
- net ETH_{PHY}_MDI[2]+: now also J6.3 (TD2+)
- net ETH_{PHY}_MDI[2]-: now also J6.6 (TD2-)
- net ETH_{PHY}_MDI[3]+: now also J6.7 (TD3+)
- net ETH_{PHY}_MDI[3]-: now also J6.8 (TD3-)
- net ETH_{PHY}_MDI[4]+: now also J6.9 (TD4+)
- net ETH_{PHY}_MDI[4]-: now also J6.10 (TD4-)
- net GND: now also C308.2, C309.2, J6.15, J6.17, J6.S1 (SHIELD), J6.S2 (SHIELD)
- net PHY_LED2: now also R80.2
- net RJ45_VC1: now also J5.1 (Pin_1), J6.11 (VC1)
- net RJ45_VC2: now also J5.2 (Pin_2), J6.12 (VC2)
- net RJ45_VC3: now also J5.3 (Pin_3), J6.13 (VC3)
- net RJ45_VC4: now also J5.4 (Pin_4), J6.14 (VC4)
- net Crystal_{ETH}_OUT: now reaches C314.1, U19.37 (XTAL_OUT/EXT_CLK), Y4.3
- net Crystal_{ETH}_IN: now reaches C313.1, U19.36 (XTAL_IN), Y4.1
- new net: J6.16, R76.1
- new net: J6.18, R80.1
- new net: C308.1, C309.1, J6.4 (CT), J6.5 (CT)
Other:
- moved on the sheet: C300, C301, C302, C303, C304, C305, C306, C307, C310, C311, C312, C313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

Commit message: SBCv0.3
there is no big thing update just some LCSC & Mouser parts
and Big problem deleted alot of component values (:
Parts:
- removed C305, C307, C311: 10u, Capacitor_SMD:C_0402_1005Metric, symbol New_Library_0:C_Small_edited
- added C329, C333, C400: 10u, Capacitor_SMD:C_0603_1608Metric, symbol New_Library_0:C_Small_edited
- C300, C301, C302, C303, C304, C306, C308, C310, C312: LCSC Part (none) -> C5209398; Mouser Part (none) -> CL03A105KP3NSNC
- C309: footprint Capacitor_SMD:C_0402_1005Metric_Pad0.74x0.62mm_HandSolder -> Capacitor_SMD:C_0201_0603Metric_Pad0.64x0.40mm_HandSolder; LCSC Part (none) -> C5209398; Mouser Part (none) -> CL03A105KP3NSNC
- C313, C314: LCSC Part (none) -> C541431; Mouser Part (none) -> 603-CC402FRNPO9BN180
- J5: LCSC Part (none) -> C66690; Mouser Part (none) -> 200-TSW10207GDLL001
- J6: footprint LPJG0926HENL:LINK-PP_LPJG0926HENL -> Datasheet_Footprints:LPJG0926HENL; LCSC Part (none) -> C22457393
- L12: LCSC Part (none) -> (do_not_autoplace no)
- R100, R101, R99: value 1.2k -> (none); LCSC Part (none) -> (show_name no)
- R72, R73, R74, R77, R78, R79, R95, R96, R98: value 4.7k -> (none); LCSC Part (none) -> (show_name no)
- R75: value 2.49k -> )
- R76, R80: value 510R -> (property "ki_fp_filters" "C_*"
- R81, R82, R83, R85, R87, R89, R91, R93: value 0R -> (none); LCSC Part (none) -> )
- R84, R86, R88, R90, R92, R94: value 22R -> (none); LCSC Part (none) -> (do_not_autoplace no)
- R97: value 4.7k -> (none); LCSC Part (none) -> (at 0 0 0)
- U19: value RTL8211F-CG -> )
- Y4: value SX32Y025000BC1T001 -> (none); footprint Crystal:Crystal_SMD_3225-4Pin_3.2x2.5mm_HandSoldering -> )
Connections:
- net AVDD10: now also C333.1
- net AVDD33: now also C329.1
- net GND: now also C329.2, C333.2, C400.2
- net VCC_1V8_S3: now also C400.1

Commit message: SBCv0.4
add LCSC & Mouser parts 
and solve the deleted value in the past version
Parts:
- removed R84, R86, R88, R90, R92, R94: (no value), PCM_Resistor_SMD_AKL:R_0402_1005Metric, symbol Device:R_Small
- added R118, R119, R147, R158, R173, R174: 22R, PCM_Resistor_SMD_AKL:R_0402_1005Metric, symbol Device:R_Small
- L12: value 2.2uH -> 3.3uH; footprint (none) -> Inductor_SMD:L_Coilcraft_0805HQ_2012Metric; LCSC Part (do_not_autoplace no) -> C2926398
- R100, R101, R99: value (none) -> 1.2k; LCSC Part (show_name no) -> C138040; Mouser Part (none) -> 603-RC0402FR-071K2L
- R72, R73, R74, R77, R78, R79, R95, R96, R98: value (none) -> 4.7k; LCSC Part (show_name no) -> C105871; Mouser Part (none) -> 603-RC0402FR-074K7L
- R75: value ) -> 2.49k; LCSC Part (none) -> C854254; Mouser Part (none) -> 603-RT0402FRE072K49L
- R76, R80: value (property "ki_fp_filters" "C_*" -> 590R; footprint PCM_Resistor_SMD_AKL:R_0402_1005Metric_Pad0.72x0.64mm -> PCM_Resistor_SMD_AKL:R_0402_1005Metric; LCSC Part (none) -> C327335; Mouser Part (none) -> 603-RC0402FR-07590RL
- R81, R82, R83, R85, R87, R89, R91, R93: value (none) -> 0R; footprint PCM_Resistor_SMD_AKL:R_0402_1005Metric_Pad0.72x0.64mm -> PCM_Resistor_SMD_AKL:R_0402_1005Metric; LCSC Part ) -> C106231; Mouser Part (none) -> 603-RC0402FR-070RL
- R97: value (none) -> 4.7k; LCSC Part (at 0 0 0) -> C105871; Mouser Part (none) -> 603-RC0402FR-074K7L; now fitted
- U19: value ) -> RTL8211F-CG; LCSC Part (none) -> C187932
- Y4: value (none) -> SX32Y025000BC1T001; footprint ) -> Crystal:Crystal_SMD_3225-4Pin_3.2x2.5mm_HandSoldering; LCSC Part (none) -> C20612981
Connections:
- net at U19.23 (RXD2/PLLOFF): now also R147.1
- net at U19.24 (RXD1/TXDLY): now also R119.1
- net at U19.27 (RXC/PHYAD1): now also R158.1
- net at U19.25 (RXD0/RXDLY): now also R118.1
- net at U19.26 (RXCTL/PHYAD2): now also R173.1
- net at U19.22 (RXD3/PHYAD0): now also R174.1
