File: gpio0.kicad_sch (KiCad schematic)
At the start: 28 parts, among them J12 Conn_01x04_Pin, Q6 2SK3018, U27 RK3576, Y4 TXM24M0004322FBCDO00T

Commit message: Add files via upload
Parts:
- removed D14, D15, D16: PESD5V0S1BA, PCM_Diode_SMD_AKL:D_SOD-323_TVS, symbol PCM_Diode_TVS_AKL:PESD5V0S1BA
- removed J12: Conn_01x04_Pin, Connector:FanPinHeader_1x04_P2.54mm_Vertical, symbol Connector:Conn_01x04_Pin
- removed LED3: LED_0603_Red, PCM_LED_SMD_AKL:LED_0603_1608Metric, symbol PCM_LED_AKL:LED_0603_Red
- removed Q6: 2SK3018, PCM_Package_TO_SOT_SMD_AKL:SOT-323_SC-70, symbol PCM_Transistor_MOSFET_AKL:2SK3018
- removed R106: 220R, PCM_Resistor_SMD_AKL:R_0402_1005Metric_Pad0.72x0.64mm, symbol Device:R_Small
- removed R107, R108: 1k, PCM_Resistor_SMD_AKL:R_0402_1005Metric_Pad0.72x0.64mm, symbol Device:R_Small
- removed R109: 100ki, PCM_Resistor_SMD_AKL:R_0402_1005Metric_Pad0.72x0.64mm, symbol Device:R_Small
- removed R110, R111, R112: 22R, PCM_Resistor_SMD_AKL:R_0402_1005Metric_Pad0.72x0.64mm, symbol Device:R_Small
- added C364: 1u, Capacitor_SMD:C_0402_1005Metric_Pad0.74x0.62mm_HandSolder, symbol New_Library_0:C_Small_edited
- added D2, D3, D4: PESD5V0S1BA, PCM_Diode_SMD_AKL:D_SOD-323_TVS, symbol PCM_Diode_TVS_AKL:PESD5V0S1BA
- added J1: Conn_01x04_Pin, Connector:FanPinHeader_1x04_P2.54mm_Vertical, symbol Connector:Conn_01x04_Pin
- added LED1: LED_0603_Red, PCM_LED_SMD_AKL:LED_0603_1608Metric, symbol PCM_LED_AKL:LED_0603_Red
- added Q1: 2SK3018, PCM_Package_TO_SOT_SMD_AKL:SOT-323_SC-70, symbol PCM_Transistor_MOSFET_AKL:2SK3018
- added R15: 220R, PCM_Resistor_SMD_AKL:R_0402_1005Metric_Pad0.72x0.64mm, symbol Device:R_Small
- added R16, R17: 1k, PCM_Resistor_SMD_AKL:R_0402_1005Metric_Pad0.72x0.64mm, symbol Device:R_Small
- added R18: 100ki, PCM_Resistor_SMD_AKL:R_0402_1005Metric_Pad0.72x0.64mm, symbol Device:R_Small
- added R19, R20, R21: 22R, PCM_Resistor_SMD_AKL:R_0402_1005Metric_Pad0.72x0.64mm, symbol Device:R_Small
- C89: renamed from C232; value 100n -> 1u
- C90: renamed from C233; value 100n -> 1u
- C91: renamed from C231; value 100n -> 1u
- C92: renamed from C229; value ??? -> 12pF
- C93: renamed from C230; value ??? -> 12pF
- C94: renamed from C234; value 100n -> 1u
- C95: renamed from C235; value 100n -> 1u
- C96: renamed from C236; value 100n -> 1u
- C97: renamed from C237; value 100n -> 1u
- renumbered R103 to R12, R105 to R13, R104 to R14, U27 to U2, Y4 to Y1
Connections:
- net BT_CTRL: now also U2.AD28 (REF_CLK1_OUT); no longer U2.1P23 (SPI2_MISO_M0)
- net GND: now also LED2.1 (K), C364.2, D2.1 (K), D3.1 (K), D4.1 (K), J1.4 (Pin_4), Q1.2 (S), R18.2
- net JTAG_TCK_M1 & UART0_TX_M0: now also D2.2 (A), J1.1 (Pin_1), R19.2
- net JTAG_TMS_M1 & UART0_RX_M0: now also D3.2 (A), J1.2 (Pin_2), R20.2
- net Reset: now also R21.1; no longer C90.1, R13.2, U2.W28 (NPOR)
- net USBC_C_INT_L: now also U2.1W22 (SAI0_MCLK_M1); no longer U2.AD28 (REF_CLK1_OUT)
- net USER_LED: now also R17.1
- net VCC_3.3v_S0: now also R15.1, R16.1
- net VDD_3.3v_S3: now also C364.1
- net at LED2.2 (A): now also R16.2
- net at U2.AA28 (UART0_RX_M0): now also R20.1
- net at U2.1U24 (UART0_TX_M0): now also R19.1
- net I2C1_SCL_M0_RK806 renamed SPI2_CLK_M0
- net I2C1_SDA_M0_RK806 renamed SPI2_MOSI_M0
- net JTAG_Reset renamed RESET_L
- net RESET_L: now also C90.1, R13.2, U2.W28 (NPOR)
- new net: Q1.1 (G), R17.2, R18.1
- new net: D4.2 (A), J1.3 (Pin_3), R21.2
- new net: LED1.1 (K), Q1.3 (D)
- new net: LED1.2 (A), R15.2
- new net SPI2_MISO_M0: U2.1P23 (SPI2_MISO_M0)
- no-connect marks 1 -> 0
Other:
- moved on the sheet: C89, C90, C91, C92, C93, C94, C95, C96, C97, R13, R14, Y1

Commit message: SBC Board V0.2
The SBC schematics before footprint and part number check
Parts:
- U3: renamed from U2; footprint (none) -> easyeda2kicad:FCCSP-698_L17.2-W16.1-TL_RK3576
- renumbered C93 to C100, C94 to C101, C95 to C102, C96 to C103, C97 to C104, C364 to C105, C89 to C96, C90 to C97, C91 to C98, C92 to C99
Connections:
- net 40GPIOs_ACK renamed HDMI_PWREN_H
- net 40GPIOs_PWR_EN renamed 40GPIOs
- net BT_CTRL renamed BT_WAKE_HOST_H
- net RTC_INT_L renamed Vdet_USB_{OTG}
- net USBC_C_INT_L renamed USB_{OTG}_CON_INT
- net WIFI_CTRL renamed WIFI_WAKE_HOST_H
- net uSD_DETECT renamed uSD_DET
Other:
- moved on the sheet: C100, C101, C102, C103, C104, C105, C96, C97, C98, C99, D2, D3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

Commit message: SBCv0.3
there is no big thing update just some LCSC & Mouser parts
and Big problem deleted alot of component values (:
Parts:
- C100, C99: LCSC Part (none) -> C26406; Mouser Part (none) -> 187-CL05C120JB5NNNC
- C101, C102, C103, C104, C105, C96, C97, C98: footprint Capacitor_SMD:C_0402_1005Metric_Pad0.74x0.62mm_HandSolder -> Capacitor_SMD:C_0201_0603Metric_Pad0.64x0.40mm_HandSolder; LCSC Part (none) -> C5209398; Mouser Part (none) -> CL03A105KP3NSNC
- D2, D3, D4: LCSC Part (none) -> C5158048; Mouser Part (none) -> 771-PESD5V0S1BA-T/R
- J1: value Conn_01x04_Pin -> B4B Connector; LCSC Part (none) -> C144395; Mouser Part (none) -> 306-B4BXHALFSN
- LED1, LED2: LCSC Part (none) -> (effects
- R12: value 0R -> (none); LCSC Part (none) -> )
- R13: value 10k -> )
- R14, R19, R20, R21: value 22R -> (property "Description" "Unpolarized capacitor, small symbol"
- R15: value 220R -> (none); LCSC Part (none) -> (at 0 0 0)
- R16, R17: value 1k -> (none); LCSC Part (none) -> (show_name no)
- R18: value 100ki -> (none); LCSC Part (none) -> (do_not_autoplace no)
- U3: value RK3576 -> (none); LCSC Part (none) -> (polyline
- Y1: value TXM24M0004322FBCDO00T -> (none); Mouser Part (none) -> (number "1"

Commit message: SBCv0.4
add LCSC & Mouser parts 
and solve the deleted value in the past version
Parts:
- removed R12, R15, R16: (no value), PCM_Resistor_SMD_AKL:R_0402_1005Metric_Pad0.72x0.64mm, symbol Device:R_Small
- removed R13: ), PCM_Resistor_SMD_AKL:R_0402_1005Metric_Pad0.72x0.64mm, symbol Device:R_Small
- removed Y1: (no value), Crystal:Crystal_SMD_3225-4Pin_3.2x2.5mm, symbol Device:Crystal_GND24
- added C211: 1u, Capacitor_SMD:C_0201_0603Metric_Pad0.64x0.40mm_HandSolder, symbol New_Library_0:C_Small_edited
- added R138, R139: 1k, PCM_Resistor_SMD_AKL:R_0402_1005Metric, symbol Device:R_Small
- added R196: 10k, PCM_Resistor_SMD_AKL:R_0402_1005Metric, symbol Device:R_Small
- added R198: 0R, PCM_Resistor_SMD_AKL:R_0402_1005Metric, symbol Device:R_Small
- added U2: M24C64-RMN6TP, Package_SO:SOIC-8_3.9x4.9mm_P1.27mm, symbol Memory_NVRAM:FM24C64B
- added Y2: TXM24M0004322FBCDO00T, Crystal:Crystal_SMD_3225-4Pin_3.2x2.5mm, symbol Device:Crystal_GND24
- LED1, LED2: value LED_0603_Red -> XL-1608SURC-06; LCSC Part (effects -> C965799
- Q1: LCSC Part (none) -> C20069148
- R14, R19, R20, R21: value (property "Description" "Unpolarized capacitor, small symbol" -> 22R; footprint PCM_Resistor_SMD_AKL:R_0402_1005Metric_Pad0.72x0.64mm -> PCM_Resistor_SMD_AKL:R_0402_1005Metric; LCSC Part (none) -> C114765; Mouser Part (none) -> 603-RC0402FR-0722RL
- R17: value (none) -> 1k; footprint PCM_Resistor_SMD_AKL:R_0402_1005Metric_Pad0.72x0.64mm -> PCM_Resistor_SMD_AKL:R_0402_1005Metric; LCSC Part (show_name no) -> C106235; Mouser Part (none) -> 603-RC0402FR-071KL
- R18: value (none) -> 100k; footprint PCM_Resistor_SMD_AKL:R_0402_1005Metric_Pad0.72x0.64mm -> PCM_Resistor_SMD_AKL:R_0402_1005Metric; LCSC Part (do_not_autoplace no) -> C60491; Mouser Part (none) -> 603-RC0402FR-07100KL
- U3: value (none) -> RK3576; LCSC Part (polyline -> C42388007
Connections:
- net GND: now also C211.2, U2.1 (A0), U2.2 (A1), U2.3 (A2), U2.4 (VSS), Y2.2 (G), Y2.4 (G)
- net I2C2_SCL_M0_CC_RTC: no longer U3.1W24 (I2C2_SCL_M0)
- net I2C2_SDA_M0_CC_RTC: no longer U3.AB29 (I2C2_SDA_M0)
- net RESET_L: now also R196.2, R198.2
- net TSADC_CTRL_M0: now also R198.1
- net VCC_1.8v_S3: now also R196.1
- net VCC_3.3v_S0: now also C211.1, U2.8 (VDD)
- net at C99.1, R14.1: now also Y2.1
- net at LED2.2 (A): now also R139.2
- net at C100.1, U3.U28 (OSC_XIN): now also Y2.3
- net at LED1.2 (A): now also R138.2
- new net EEPROM_WP: U2.7 (WP)
- new net I2C2_SCL_M0_CC_RTC_EEPROM: U2.6 (SCL), U3.1W24 (I2C2_SCL_M0)
- new net I2C2_SDA_M0_CC_RTC_EEPROM: U2.5 (SDA), U3.AB29 (I2C2_SDA_M0)
- new net VCC5V0_SYS: R138.1, R139.1

Commit message: SBCv0.5
small update for Josa watch the final version
Parts:
- U2: LCSC Part (none) -> C79988; Mouser Part (none) -> 511-M24C64-RMN6TP
Changed lines of the file:
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@@
 					(reference "C103")
 					(unit 1)
-					(variant
-						(name "Test")
-					)
 				)
 			)
@@
 					(reference "C96")
 					(unit 1)
-					(variant
-						(name "Test")
-					)
 				)
 			)
@@
 					(reference "LED2")
 					(unit 1)
-					(variant
-						(name "Test")
-					)
 				)
 			)
@@
 					(reference "C99")
 					(unit 1)
-					(variant
-						(name "Test")
-					)
 				)
 			)
@@
 					(reference "C211")
 					(unit 1)
-					(variant
-						(name "Test")
-					)
 				)
 			)
@@
 					(reference "C104")
 					(unit 1)
-					(variant
-						(name "Test")
-					)
 				)
 			)
@@
 					(reference "C97")
 					(unit 1)
-					(variant
-						(name "Test")
-					)
 				)
 			)
@@
 					(reference "C105")
 					(unit 1)
-					(variant
-						(name "Test")
-					)
 				)
 			)
@@
 					(reference "U3")
 					(unit 1)
-					(variant
-						(name "Test")
-					)
 				)
 			)
@@
 					(reference "C100")
 					(unit 1)
-					(variant
-						(name "Test")
-					)
 				)
 			)
@@
 					(reference "C102")
 					(unit 1)
-					(variant
-						(name "Test")
-					)
 				)
 			)
@@
 					(reference "C101")
 					(unit 1)
-					(variant
-						(name "Test")
-					)
 				)
 			)
@@
 					(reference "J1")
 					(unit 1)
-					(variant
-						(name "Test")
-					)
 				)
 			)
@@
 					(reference "LED1")
 					(unit 1)
-					(variant
-						(name "Test")
-					)
 				)
 			)
@@
 			)
 		)
+		(property "LCSC Part" "C79988"
+			(at 101.6 226.06 0)
+			(hide yes)
+			(show_name no)
+			(do_not_autoplace no)
+			(effects
+				(font
+					(size 1.27 1.27)
+				)
+			)
+		)
+		(property "Mouser Part" "511-M24C64-RMN6TP "
+			(at 101.6 226.06 0)
+			(hide yes)
+			(show_name no)
+			(do_not_autoplace no)
+			(effects
+				(font
+					(size 1.27 1.27)
+				)
+			)
+		)
 		(pin "6"
 		)
@@
 					(reference "D2")
 					(unit 1)
-					(variant
-						(name "Test")
-					)
 				)
 			)
@@
 					(reference "Q1")
 					(unit 1)
-					(variant
-						(name "Test")
-					)
 				)
 			)
@@
 					(reference "C98")
 					(unit 1)
-					(variant
-						(name "Test")
-					)
 				)
 			)
@@
 					(reference "D3")
 					(unit 1)
-					(variant
-						(name "Test")
-					)
 				)
 			)
@@
 					(reference "D4")
 					(unit 1)
-					(variant
-						(name "Test")
-					)
 				)
 			)
