File: hdmi.kicad_sch (KiCad schematic)
At the start: 37 parts, among them J4 HDMI_A, Q1 2SK3018, Q2 2SK3018, Q3 2SK3018, Q4 2SK3018, U14 AP2171W, U15 TXB0104PW, U16 TPD4E05U06DQA, U17 TPD4E05U06DQA, U18 TPD4E05U06DQA

Commit message: Add files via upload
Parts:
- removed C78: 1u, Capacitor_SMD:C_0402_1005Metric_Pad0.74x0.62mm_HandSolder, symbol New_Library_0:C_Small_edited
- removed C79: 22u, Capacitor_SMD:C_0603_1608Metric, symbol New_Library_0:C_Small_edited
- removed D9: PESD5V0S1BA, PCM_Diode_SMD_AKL:D_SOD-323_TVS, symbol PCM_Diode_TVS_AKL:PESD5V0S1BA
- removed R16: 2.2k, PCM_Resistor_SMD_AKL:R_0402_1005Metric, symbol Device:R_Small
- removed R17: 100k, PCM_Resistor_SMD_AKL:R_0402_1005Metric, symbol Device:R_Small
- removed R18: 10k, PCM_Resistor_SMD_AKL:R_0402_1005Metric, symbol Device:R_Small
- removed U14: AP2171W, Package_TO_SOT_SMD:SOT-23-5, symbol Power_Management:AP2171W
- added C374: 22u, Capacitor_SMD:C_0603_1608Metric, symbol New_Library_0:C_Small_edited
- added C375: 1u, Capacitor_SMD:C_0402_1005Metric_Pad0.74x0.62mm_HandSolder, symbol New_Library_0:C_Small_edited
- added D24: SMBJ5.0CA, PCM_Diode_SMD_AKL:D_SMB_TVS, symbol PCM_Diode_TVS_AKL:SMBJ5.0CA
- added R118, R158, R171: 2.2k, PCM_Resistor_SMD_AKL:R_0402_1005Metric, symbol Device:R_Small
- added R157: 10k, PCM_Resistor_SMD_AKL:R_0402_1005Metric_Pad0.72x0.64mm, symbol Device:R_Small
- added R169: 10k, PCM_Resistor_SMD_AKL:R_0402_1005Metric, symbol Device:R_Small
- added R170: 100k, PCM_Resistor_SMD_AKL:R_0402_1005Metric, symbol Device:R_Small
- added U34: AP2553W6-7, symbol New_Library:AP2553W6-7
- C317: renamed from C88; value 100n -> 1u
- C318: renamed from C89; value 100n -> 1u
- J8: renamed from J4; footprint (none) -> Connector_Video:HDMI_A_Amphenol_10029449-x01xLF_Horizontal
- renumbered C80 to C308, C81 to C309, C82 to C310, C83 to C311, C84 to C312, C85 to C313, C86 to C314, C87 to C315, C90 to C316, D10 to D17, Q1 to Q2, Q2 to Q3, Q3 to Q4, Q4 to Q5, R19 to R108, R20 to R109, R21 to R110, R22 to R111, R23 to R112, R24 to R113, R25 to R114, R26 to R115, R118 to R119, U15 to U20, U16 to U21, U17 to U22, U18 to U23
Connections:
- net +5V_{HDMI}: now also C374.1, D24.2 (A), U34.6 (OUT)
- net GND: now also C374.2, C375.2, D24.1 (K), R157.2, R169.2, R170.2, U34.2 (GND)
- net at U20.8 (OE): now also R157.1
- net +3.3V renamed VCC_3V3_S0
- net VCC_3V3_S0: now also R118.1, R158.1
- net HDMI_CEC renamed HDMI_TX_CEC_M0
- net HDMI_CTRL renamed HDMI_GPIOs
- net HDMI_HPD renamed HDMI_TX_HPDIN_M0
- net SCL_HDMI renamed HDMI_TX_SCL
- net HDMI_TX_SCL: now also R118.2
- net SDA_HDMI renamed HDMI_TX_SDA
- net HDMI_TX_SDA: now also R158.2
- new net: R170.1, R171.1, U34.3 (EN)
- new net: R169.1, U34.5 (ILIM)
- new net HDMI_PWREN_H: R171.2
- new net VCC5V0_SYS: C375.1, U34.1 (IN)
Other:
- moved on the sheet: C317, C318

Commit message: SBC Board V0.2
The SBC schematics before footprint and part number check
Parts:
- added C326: 220n, Capacitor_SMD:C_0201_0603Metric_Pad0.64x0.40mm_HandSolder, symbol New_Library_0:C_Small_edited
- renumbered C375 to C315, C374 to C316, C308 to C317, C309 to C318, C310 to C319, C311 to C320, C312 to C321, C313 to C322, C314 to C323, C315 to C324, C316 to C325, C317 to C327, C318 to C328, D24 to D14, D17 to D15, J8 to J7, R171 to R102, R108 to R103, R109 to R104, R110 to R105, R111 to R106, R112 to R107, R113 to R108, R114 to R109, R115 to R110, R169 to R111, R170 to R112, R118 to R113, R158 to R114, R157 to R115, R119 to R116, U34 to U20, U20 to U21, U21 to U22, U22 to U23, U23 to U24
Connections:
- net CHDMI_HPD: now also C326.2
- net HDMI_GPIOs: no longer Q2.1 (G), Q3.1 (G), Q4.1 (G), Q5.1 (G)
- net HDMI_UTILITY renamed HDMI_TX_SBD_P
- new net HDMI_TX_ON: Q2.1 (G), Q3.1 (G), Q4.1 (G), Q5.1 (G)
- new net HDMI_TX_SBD_N: C326.1
Other:
- moved on the sheet: C327, C328, Q2, Q3, Q4, Q5, R103, R104, R105, R106, R107, R108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

Commit message: SBCv0.3
there is no big thing update just some LCSC & Mouser parts
and Big problem deleted alot of component values (:
Parts:
- C315: footprint Capacitor_SMD:C_0402_1005Metric_Pad0.74x0.62mm_HandSolder -> Capacitor_SMD:C_0201_0603Metric_Pad0.64x0.40mm_HandSolder; LCSC Part (none) -> C5209398; Mouser Part (none) -> CL03A105KP3NSNC
- C316: LCSC Part (none) -> C86295; Mouser Part (none) -> CL10A226MP8NUNE
- C317, C318, C319, C320, C321, C322, C323, C324, C325, C326: LCSC Part (none) -> C326658; Mouser Part (none) -> 603-CC0201KRX56BB224
- C327, C328: LCSC Part (none) -> C5209398; Mouser Part (none) -> CL03A105KP3NSNC
- D14: LCSC Part (none) -> C113975; Mouser Part (none) -> 581-SMBJ5.0CA
- D15: LCSC Part (none) -> C5158048; Mouser Part (none) -> 771-PESD5V0S1BA-T/R
- J7: value HDMI_A -> HDMI-001S; LCSC Part (none) -> C720616
- R102, R113, R114: value 2.2k -> (none); LCSC Part (none) -> (do_not_autoplace no)
- R103, R104, R105, R106, R107, R108, R109, R110: value 590R -> (none); LCSC Part (none) -> (do_not_autoplace no)
- R111: LCSC Part (none) -> (at 0 0 0)
- R112: value 100k -> (none); LCSC Part (none) -> (show_name no)
- R115: value 10k -> )
- R116: value 0R -> (none); LCSC Part (none) -> )
- U20: footprint (none) -> Package_TO_SOT_SMD:SOT-23-6_Handsoldering; LCSC Part (none) -> C212302; Mouser Part (none) -> 621-AP2553W6-7
- U21: value TXB0104PW -> (symbol "C_Small_edited_1_1"
- U22, U23, U24: value TPD4E05U06DQA -> (none); Mouser Part (none) -> )

Commit message: SBCv0.4
add LCSC & Mouser parts 
and solve the deleted value in the past version
Parts:
- Q2, Q3, Q4, Q5: LCSC Part (none) -> C20069148
- R102, R113, R114: value (none) -> 2.2k; LCSC Part (do_not_autoplace no) -> C114762; Mouser Part (none) -> 603-RC0402FR-072K2L
- R103, R104, R105, R106, R107, R108, R109, R110: value (none) -> 590R; LCSC Part (do_not_autoplace no) -> C327335; Mouser Part (none) -> 603-RC0402FR-07590RL
- R111: LCSC Part (at 0 0 0) -> C60490; Mouser Part (none) -> 603-RC0402FR-0710KL
- R112: value (none) -> 100k; LCSC Part (show_name no) -> C60491; Mouser Part (none) -> 603-RC0402FR-07100KL
- R115: value ) -> 10k; footprint PCM_Resistor_SMD_AKL:R_0402_1005Metric_Pad0.72x0.64mm -> PCM_Resistor_SMD_AKL:R_0402_1005Metric; LCSC Part (none) -> C60490; Mouser Part (none) -> 603-RC0402FR-0710KL
- R116: value (none) -> 0R; footprint PCM_Resistor_SMD_AKL:R_0402_1005Metric_Pad0.72x0.64mm -> PCM_Resistor_SMD_AKL:R_0402_1005Metric; LCSC Part ) -> C106231; Mouser Part (none) -> 603-RC0402FR-070RL
- U21: value (symbol "C_Small_edited_1_1" -> TXB0104PWR; LCSC Part (none) -> C60708; Mouser Part (none) -> 595-TXB0104PWR
- U22, U23, U24: value (none) -> TPD4E05U06DQAR; LCSC Part (none) -> C138714; Mouser Part ) -> 595-TPD4E05U06DQAR
