File: lpddr5.kicad_sch (KiCad schematic)
At the start: 64 parts, among them U1 MT62F1G32D4DR-031

Commit message: Add files via upload
Parts:
- C229: renamed from C362; value 100n -> 1u
- C230: renamed from C363; value 100n -> 1u
- C231: renamed from C364; value 100n -> 1u
- C232: renamed from C365; value 100n -> 1u
- C233: renamed from C366; value 100n -> 1u
- C234: renamed from C367; value 100n -> 1u
- C235: renamed from C368; value 100n -> 1u
- C236: renamed from C340; value 100n -> 1u
- C237: renamed from C339; value 100n -> 1u
- C238: renamed from C338; value 100n -> 1u
- C239: renamed from C337; value 100n -> 1u
- C243: renamed from C347; value 100n -> 1u
- C244: renamed from C346; value 100n -> 1u
- C245: renamed from C345; value 100n -> 1u
- C246: renamed from C344; value 100n -> 1u
- C247: renamed from C343; value 100n -> 1u
- C248: renamed from C342; value 100n -> 1u
- C249: renamed from C341; value 100n -> 1u
- C250: renamed from C355; value 100n -> 1u
- C251: renamed from C356; value 100n -> 1u
- C252: renamed from C357; value 100n -> 1u
- C253: renamed from C358; value 100n -> 1u
- C254: renamed from C359; value 100n -> 1u
- C255: renamed from C360; value 100n -> 1u
- C256: renamed from C361; value 100n -> 1u
- C258: renamed from C393; value 100n -> 1u
- C259: renamed from C394; value 100n -> 1u
- C260: renamed from C395; value 100n -> 1u
- C264: renamed from C377; value 100n -> 1u
- C265: renamed from C378; value 100n -> 1u
- C266: renamed from C379; value 100n -> 1u
- C267: renamed from C353; value 100n -> 1u
- C268: renamed from C354; value 100n -> 1u
- C269: renamed from C382; value 100n -> 1u
- C270: renamed from C384; value 100n -> 1u
- C271: renamed from C371; value 100n -> 1u
- C272: renamed from C370; value 100n -> 1u
- C273: renamed from C369; value 100n -> 1u
- C276: renamed from C350; value 100n -> 1u
- C277: renamed from C351; value 100n -> 1u
- C278: renamed from C352; value 100n -> 1u
- C279: renamed from C380; value 100n -> 1u
- C280: renamed from C381; value 100n -> 1u
- C281: renamed from C383; value 100n -> 1u
- C282: renamed from C385; value 100n -> 1u
- C283: renamed from C387; value 100n -> 1u
- C284: renamed from C389; value 100n -> 1u
- C285: renamed from C391; value 100n -> 1u
- C286: renamed from C372; value 100n -> 1u
- C287: renamed from C373; value 100n -> 1u
- C288: renamed from C374; value 100n -> 1u
- C289: renamed from C375; value 100n -> 1u
- C290: renamed from C376; value 100n -> 1u
- renumbered C336 to C240, C335 to C241, C328 to C242, C392 to C257, C386 to C261, C388 to C262, C390 to C263, C349 to C274, C348 to C275, R1 to R77, U1 to U17
Connections:
- net VDD_DDR_S0 renamed VDDQ_DDR_S0
Other:
- note added: "0.51V NOM"
- note removed: "0.5V NOM"

Commit message: SBC Board V0.2
The SBC schematics before footprint and part number check
Parts:
- renumbered C229 to C238, C230 to C239, C231 to C240, C232 to C241, C233 to C242, C234 to C243, C235 to C244, C236 to C245, C237 to C246, C238 to C247, C239 to C248, C240 to C249, C241 to C250, C242 to C251, C243 to C252, C244 to C253, C245 to C254, C246 to C255, C247 to C256, C248 to C257, C249 to C258, C250 to C259, C251 to C260, C252 to C261, C253 to C262, C254 to C263, C255 to C264, C256 to C265, C257 to C266, C258 to C267, C259 to C268, C260 to C269, C261 to C270, C262 to C271, C263 to C272, C264 to C273, C265 to C274, C266 to C275, C267 to C276, C268 to C277, C269 to C278, C270 to C279, C271 to C280, C272 to C281, C273 to C282, C274 to C283, C275 to C284, C276 to C285, C277 to C286, C278 to C287, C279 to C288, C280 to C289, C281 to C290, C282 to C291, C283 to C292, C284 to C293, C285 to C294, C286 to C295, C287 to C296, C288 to C297, C289 to C298, C290 to C299, R77 to R71, U17 to U18

Commit message: SBCv0.3
there is no big thing update just some LCSC & Mouser parts
and Big problem deleted alot of component values (:
Parts:
- removed C283: 1u, Capacitor_SMD:C_01005_0402Metric, symbol New_Library_0:C_Small_edited
- added C397: 1u, Capacitor_SMD:C_0201_0603Metric_Pad0.64x0.40mm_HandSolder, symbol New_Library_0:C_Small_edited
- C238, C239, C240, C241, C242, C243, C244, C245, C246, C247, C248, C252, C253, C254, C255, C256, C257, C258, C259, C260, C261, C262, C263, C264, C265, C267, C268, C269, C273, C274, C275, C276, C277, C278, C279, C280, C281, C282, C285, C286, C287, C288, C289, C290, C291, C292, C293, C294, C295, C296, C297, C298, C299: LCSC Part (none) -> C5209398; Mouser Part (none) -> CL03A105KP3NSNC
- C249, C250, C251, C266, C270, C271, C272, C284: LCSC Part (none) -> C86295; Mouser Part (none) -> CL10A226MP8NUNE
- R71: value R_240R_0402 -> (none); LCSC Part (none) -> )
- U18: value MT62F1G32D4DR-031 -> (none); LCSC Part (none) -> )
Connections:
- net GND: now also C397.2
- net VDD2L_0V9_DDR_S3: now also C397.1

Commit message: SBCv0.4
add LCSC & Mouser parts 
and solve the deleted value in the past version
Parts:
- R71: value (none) -> 240R; LCSC Part ) -> C114755; Mouser Part (none) -> 603-RC0402FR-07240RL
- U18: value (none) -> MT62F1G32D4DR-031 WT:B; LCSC Part ) -> (none); Mouser Part (none) -> 340-450481-TRAY
Changed lines of the file:
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@@
 			)
 		)
-		(property "Value" ""
+		(property "Value" "MT62F1G32D4DR-031 WT:B"
 			(at 185.42 187.96 0)
 			(hide yes)
@@
 			)
 		)
-		(property "LCSC Part" ")"
+		(property "LCSC Part" ""
 			(at 140.97 182.88 0)
 			(hide yes)
@@
 			)
 		)
+		(property "Mouser Part" "340-450481-TRAY "
+			(at 140.97 182.88 0)
+			(hide yes)
+			(show_name no)
+			(do_not_autoplace no)
+			(effects
+				(font
+					(size 1.27 1.27)
+				)
+			)
+		)
 		(pin "A1"
 		)
@@
 			)
 		)
-		(property "Value" ""
+		(property "Value" "MT62F1G32D4DR-031 WT:B"
 			(at 224.79 88.9 0)
 			(hide yes)
@@
 			)
 		)
-		(property "LCSC Part" ")"
+		(property "LCSC Part" ""
 			(at 180.34 83.82 0)
 			(hide yes)
@@
 			)
 		)
+		(property "Mouser Part" "340-450481-TRAY "
+			(at 180.34 83.82 0)
+			(hide yes)
+			(show_name no)
+			(do_not_autoplace no)
+			(effects
+				(font
+					(size 1.27 1.27)
+				)
+			)
+		)
 		(pin "A1"
 		)
@@
 			)
 		)
-		(property "Value" ""
+		(property "Value" "MT62F1G32D4DR-031 WT:B"
 			(at 312.42 187.96 0)
 			(hide yes)
@@
 			)
 		)
-		(property "LCSC Part" ")"
+		(property "LCSC Part" ""
 			(at 267.97 182.88 0)
 			(hide yes)
@@
 			)
 		)
+		(property "Mouser Part" "340-450481-TRAY "
+			(at 267.97 182.88 0)
+			(hide yes)
+			(show_name no)
+			(do_not_autoplace no)
+			(effects
+				(font
+					(size 1.27 1.27)
+				)
+			)
+		)
 		(pin "A1"
 		)
@@
 			)
 		)
-		(property "Value" ""
+		(property "Value" "240R"
 			(at 184.15 92.71 0)
 			(hide yes)
@@
 			)
 		)
-		(property "LCSC Part" ")"
+		(property "LCSC Part" "C114755"
 			(at 171.45 113.03 90)
 			(hide yes)
@@
 			(at 171.45 113.03 90)
 			(hide yes)
+			(show_name no)
+			(do_not_autoplace no)
+			(effects
+				(font
+					(size 1.27 1.27)
+				)
+			)
+		)
+		(property "Mouser Part" "603-RC0402FR-07240RL"
+			(at 171.45 113.03 90)
+			(hide yes)

Commit message: SBCv0.5
small update for Josa watch the final version
Parts:
- R71: footprint antmicro-footprints:R_0402_1005Metric -> PCM_Resistor_SMD_AKL:R_0402_1005Metric
