File: mipi.kicad_sch (KiCad schematic)
At the start: 14 parts, among them J10 Conn_01x30_MountingPin, J9 Conn_01x30_MountingPin

Commit message: Add files via upload
Parts:
- C348: renamed from C109; value 100n -> 1u
- C350: renamed from C111; value 100n -> 1u
- C352: renamed from C113; value 100n -> 1u
- C354: renamed from C115; value 100n -> 1u
- C356: renamed from C117; value 100n -> 1u
- R146: renamed from R60; value 4.7k -> 2.2k
- R147: renamed from R61; value 4.7k -> 2.2k
- renumbered C108 to C347, C110 to C349, C112 to C351, C114 to C353, C116 to C355, J9 to J10, J10 to J11
Connections:
- net +1.8V renamed VCC_1V8_S3
- net +3.3V renamed VCC_3V3_S0
- net +5V renamed VCC5V0_SYS
- net CAM1_CLK1_OUT renamed CAM1_CLK1_OUT_M0_1V8
- net CAM1_CLK1_OUT_M0_1V8: no longer R146.2
- net CAM2_CLK2_OUT renamed CAM2_CLK2_OUT_M0_1V8
- net CAM2_CLK2_OUT_M0_1V8: no longer R147.2
- net CSI_CAM1_PDN renamed MIPI_DPHY_CSI_CAM1_PDN_H
- net CSI_CAM2_PDN renamed MIPI_DPHY_CSI_CAM2_PDN_H
- net CSI_CAM2_RESET renamed MIPI_DPHY_CSI_CAM2_RST_H
- net LCD_BL_PWM1_CH1 renamed LCD_BL_PWM1_CH1_M0
- net LCD_PWR_EN renamed LCD_PWREN_H
- net LCD_RST renamed LCD_RST_L
- net SCL renamed I2C0_SCL_M1_TP
- net SCL_MIPI_CAM2 renamed I2C4_SCL_M3_MIPI_CAM2
- net I2C4_SCL_M3_MIPI_CAM2: now also R147.2
- net SDA renamed I2C0_SDA_M1_TP
- net SDA_MIPI_CAM2 renamed I2C4_SDA_M3_MIPI_CAM2
- net I2C4_SDA_M3_MIPI_CAM2: now also R146.2
- net TP_INT renamed TP_INT_L
- net TP_RST renamed TP_RST_L
Other:
- moved on the sheet: C347, C348, C349, C350, C351, C352, C353, C354, C355, C356, J10, J11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

Commit message: SBC Board V0.2
The SBC schematics before footprint and part number check
Parts:
- removed J11: Conn_01x30_MountingPin, symbol Connector_Generic_MountingPin:Conn_01x30_MountingPin
- added J10: DSI Connector, easyeda2kicad:FPC-SMD_30P-L20.5-W2.0-P0.50, symbol Connector_Generic_MountingPin:Conn_01x30_MountingPin
- J9: renamed from J10; value Conn_01x30_MountingPin -> CSI Connector; footprint (none) -> easyeda2kicad:FPC-SMD_30P-L20.5-W2.0-P0.50
- renumbered C347 to C356, C348 to C357, C349 to C358, C350 to C359, C351 to C360, C352 to C361, C353 to C362, C354 to C363, C355 to C364, C356 to C365, R146 to R149, R147 to R150
Connections:
- net DSI0_TX_CLK_N: now also J10.8 (Pin_8)
- net DSI0_TX_CLK_P: now also J10.9 (Pin_9)
- net DSI0_TX_D0_N: now also J10.2 (Pin_2)
- net DSI0_TX_D0_P: now also J10.3 (Pin_3)
- net DSI0_TX_D1_N: now also J10.5 (Pin_5)
- net DSI0_TX_D1_P: now also J10.6 (Pin_6)
- net DSI0_TX_D2_N: now also J10.11 (Pin_11)
- net DSI0_TX_D2_P: now also J10.12 (Pin_12)
- net DSI0_TX_D3_N: now also J10.14 (Pin_14)
- net DSI0_TX_D3_P: now also J10.15 (Pin_15)
- net GND: now also J10.1 (Pin_1), J10.10 (Pin_10), J10.13 (Pin_13), J10.16 (Pin_16), J10.24 (Pin_24), J10.25 (Pin_25), J10.4 (Pin_4), J10.7 (Pin_7), J10.MP (MountPin)
- net I2C0_SCL_M1_TP: now also J10.22 (Pin_22)
- net I2C0_SDA_M1_TP: now also J10.23 (Pin_23)
- net LCD_BL_PWM1_CH1_M0: now also J10.17 (Pin_17)
- net LCD_PWREN_H: now also J10.19 (Pin_19)
- net LCD_RST_L: now also J10.18 (Pin_18)
- net TP_INT_L: now also J10.20 (Pin_20)
- net TP_RST_L: now also J10.21 (Pin_21)
- net VCC5V0_SYS: now also J10.29 (Pin_29), J10.30 (Pin_30)
- net VCC_1V8_S3: now also J10.26 (Pin_26)
- net VCC_3V3_S0: now also J10.27 (Pin_27), J10.28 (Pin_28)

Commit message: SBCv0.3
there is no big thing update just some LCSC & Mouser parts
and Big problem deleted alot of component values (:
Parts:
- C356, C358, C360, C362, C364: LCSC Part (none) -> C86295; Mouser Part (none) -> CL10A226MP8NUNE
- C357, C359, C361, C363, C365: LCSC Part (none) -> C5209398; Mouser Part (none) -> CL03A105KP3NSNC
- J10: value DSI Connector -> AFC11-S30ICC-00; LCSC Part (none) -> C11078; Mouser Part (none) -> 38-52559-3052
- J9: value CSI Connector -> AFC11-S30ICC-00; LCSC Part (none) -> C11078; Mouser Part (none) -> 38-52559-3052
- R149, R150: value 2.2k -> (none); LCSC Part (none) -> (do_not_autoplace no)

Commit message: SBCv0.4
add LCSC & Mouser parts 
and solve the deleted value in the past version
Parts:
- R149, R150: value (none) -> 2.2k; LCSC Part (do_not_autoplace no) -> C114762; Mouser Part (none) -> 603-RC0402FR-072K2L
