File: mipi_phy.kicad_sch (KiCad schematic)
At the start: 12 parts, among them U27 RK3576

Commit message: Add files via upload
Parts:
- C154: renamed from C316; value 100n -> 1u
- C157: renamed from C318; value 100n -> 1u
- renumbered C310 to C148, C309 to C149, C307 to C150, C308 to C151, C311 to C152, C312 to C153, C313 to C155, C317 to C156, C319 to C158, U27 to U2

Commit message: SBC Board V0.2
The SBC schematics before footprint and part number check
Parts:
- U3: renamed from U2; footprint (none) -> easyeda2kicad:FCCSP-698_L17.2-W16.1-TL_RK3576
- renumbered C148 to C156, C149 to C157, C150 to C158, C151 to C159, C152 to C160, C153 to C161, C154 to C162, C155 to C163, C156 to C164, C157 to C165, C158 to C166

Commit message: SBCv0.3
there is no big thing update just some LCSC & Mouser parts
and Big problem deleted alot of component values (:
Parts:
- C156, C157, C158, C159, C160, C161, C162, C163, C164, C165, C166: footprint Capacitor_SMD:C_0402_1005Metric_Pad0.74x0.62mm_HandSolder -> Capacitor_SMD:C_0201_0603Metric_Pad0.64x0.40mm_HandSolder; LCSC Part (none) -> C5209398; Mouser Part (none) -> CL03A105KP3NSNC
- U3: value RK3576 -> (none); LCSC Part (none) -> (polyline

Commit message: SBCv0.4
add LCSC & Mouser parts 
and solve the deleted value in the past version
Parts:
- U3: value (none) -> RK3576; LCSC Part (polyline -> C42388007
Changed lines of the file:
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@@
 			)
 		)
-		(property "Value" ""
+		(property "Value" "RK3576"
 			(at 139.7 22.86 0)
 			(show_name no)
@@
 			)
 		)
-		(property "LCSC Part" "(polyline"
+		(property "LCSC Part" "C42388007"
 			(at 139.7 105.41 0)
 			(hide yes)
