File: rk3576_ufs.kicad_sch (KiCad schematic)
At the start: 13 parts, among them U27 RK3576, Y6 XTM32026000FT00351001

Commit message: Add files via upload
Parts:
- C139: renamed from C260; value 100n -> 1u
- C140: renamed from C262; value 100n -> 1u
- renumbered C253 to C135, C254 to C136, C257 to C137, C258 to C138, C256 to C141, C255 to C142, R122 to R39, R121 to R40, R119 to R41, U27 to U2, Y6 to Y2

Commit message: SBC Board V0.2
The SBC schematics before footprint and part number check
Parts:
- U3: renamed from U2; footprint (none) -> easyeda2kicad:FCCSP-698_L17.2-W16.1-TL_RK3576
- renumbered C135 to C143, C136 to C144, C137 to C145, C138 to C146, C139 to C147, C140 to C148, C141 to C149, C142 to C150
Changed lines of the file:
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@@
 		(dnp no)
 		(fields_autoplaced yes)
-		(property "Reference" "C135"
+		(property "Reference" "C143"
 			(at 74.93 87.6362 0)
 			(show_name no)
@@
 			(project "RK3576 SBC"
 				(path "/b79dbff4-0cad-4ff7-bec2-7c0e4f8b14d3/34f9b0cb-aeae-42b4-a2af-a0a79afcf392/51173a63-65bb-4420-9c6d-af77ebfb98d4"
-					(reference "C135")
+					(reference "C143")
 					(unit 1)
 				)
@@
 		(in_pos_files yes)
 		(dnp no)
-		(property "Reference" "#PWR0196"
+		(property "Reference" "#PWR0208"
 			(at 96.52 97.79 0)
 			(hide yes)
@@
 			(project "RK3576 SBC"
 				(path "/b79dbff4-0cad-4ff7-bec2-7c0e4f8b14d3/34f9b0cb-aeae-42b4-a2af-a0a79afcf392/51173a63-65bb-4420-9c6d-af77ebfb98d4"
-					(reference "#PWR0196")
+					(reference "#PWR0208")
 					(unit 1)
 				)
@@
 		(dnp no)
 		(fields_autoplaced yes)
-		(property "Reference" "U2"
+		(property "Reference" "U3"
 			(at 146.05 66.04 0)
 			(show_name no)
@@
 			)
 		)
-		(property "Footprint" ""
+		(property "Footprint" "easyeda2kicad:FCCSP-698_L17.2-W16.1-TL_RK3576"
 			(at 78.74 36.195 0)
 			(hide yes)
@@
 			(project "RK3576 SBC"
 				(path "/b79dbff4-0cad-4ff7-bec2-7c0e4f8b14d3/34f9b0cb-aeae-42b4-a2af-a0a79afcf392/51173a63-65bb-4420-9c6d-af77ebfb98d4"
-					(reference "U2")
+					(reference "U3")
 					(unit 14)
 				)
@@
 		(in_pos_files yes)
 		(dnp no)
-		(property "Reference" "#PWR0202"
+		(property "Reference" "#PWR0214"
 			(at 60.96 115.57 0)
 			(hide yes)
@@
 			(project "RK3576 SBC"
 				(path "/b79dbff4-0cad-4ff7-bec2-7c0e4f8b14d3/34f9b0cb-aeae-42b4-a2af-a0a79afcf392/51173a63-65bb-4420-9c6d-af77ebfb98d4"
-					(reference "#PWR0202")
+					(reference "#PWR0214")
 					(unit 1)
 				)
@@
 		(dnp no)
 		(fields_autoplaced yes)
-		(property "Reference" "C139"
+		(property "Reference" "C147"
 			(at 48.26 105.4162 0)
 			(show_name no)
@@
 			(project "RK3576 SBC"
 				(path "/b79dbff4-0cad-4ff7-bec2-7c0e4f8b14d3/34f9b0cb-aeae-42b4-a2af-a0a79afcf392/51173a63-65bb-4420-9c6d-af77ebfb98d4"
-					(reference "C139")
+					(reference "C147")
 					(unit 1)
 				)
@@
 		(in_pos_files yes)
 		(dnp no)
-		(property "Reference" "#PWR0197"
+		(property "Reference" "#PWR0209"
 			(at 106.68 97.79 0)
 			(hide yes)
@@
 			(project "RK3576 SBC"
 				(path "/b79dbff4-0cad-4ff7-bec2-7c0e4f8b14d3/34f9b0cb-aeae-42b4-a2af-a0a79afcf392/51173a63-65bb-4420-9c6d-af77ebfb98d4"
-					(reference "#PWR0197")
+					(reference "#PWR0209")
 					(unit 1)
 				)
@@
 		(dnp no)
 		(fields_autoplaced yes)
-		(property "Reference" "C142"
+		(property "Reference" "C150"
 			(at 234.95 128.2762 0)
 			(show_name no)
@@
 			(project "RK3576 SBC"
 				(path "/b79dbff4-0cad-4ff7-bec2-7c0e4f8b14d3/34f9b0cb-aeae-42b4-a2af-a0a79afcf392/51173a63-65bb-4420-9c6d-af77ebfb98d4"
-					(reference "C142")
+					(reference "C150")
 					(unit 1)
 				)
@@
 		(dnp no)
 		(fields_autoplaced yes)
-		(property "Reference" "C137"
+		(property "Reference" "C145"
 			(at 99.06 87.6362 0)
 			(show_name no)
@@
 			(project "RK3576 SBC"
 				(path "/b79dbff4-0cad-4ff7-bec2-7c0e4f8b14d3/34f9b0cb-aeae-42b4-a2af-a0a79afcf392/51173a63-65bb-4420-9c6d-af77ebfb98d4"
-					(reference "C137")
+					(reference "C145")
 					(unit 1)
 				)
@@
 		(in_pos_files yes)
 		(dnp no)
-		(property "Reference" "#PWR0198"
+		(property "Reference" "#PWR0210"
 			(at 45.72 99.06 0)
 			(hide yes)
@@
 			(project "RK3576 SBC"
 				(path "/b79dbff4-0cad-4ff7-bec2-7c0e4f8b14d3/34f9b0cb-aeae-42b4-a2af-a0a79afcf392/51173a63-65bb-4420-9c6d-af77ebfb98d4"
-					(reference "#PWR0198")
+					(reference "#PWR0210")
 					(unit 1)
 				)
@@
 		(in_pos_files yes)
 		(dnp no)
-		(property "Reference" "#PWR0195"
+		(property "Reference" "#PWR0207"
 			(at 82.55 97.79 0)
 			(hide yes)
@@
 			(project "RK3576 SBC"
 				(path "/b79dbff4-0cad-4ff7-bec2-7c0e4f8b14d3/34f9b0cb-aeae-42b4-a2af-a0a79afcf392/51173a63-65bb-4420-9c6d-af77ebfb98d4"
-					(reference "#PWR0195")
+					(reference "#PWR0207")
 					(unit 1)
 				)
@@
 		(in_pos_files yes)
 		(dnp no)
-		(property "Reference" "#PWR0201"
+		(property "Reference" "#PWR0213"
 			(at 45.72 115.57 0)
 			(hide yes)
@@
 			(project "RK3576 SBC"
 				(path "/b79dbff4-0cad-4ff7-bec2-7c0e4f8b14d3/34f9b0cb-aeae-42b4-a2af-a0a79afcf392/51173a63-65bb-4420-9c6d-af77ebfb98d4"
-					(reference "#PWR0201")
+					(reference "#PWR0213")
 					(unit 1)
 				)
@@
 		(dnp no)
 		(fields_autoplaced yes)
-		(property "Reference" "C141"
+		(property "Reference" "C149"
 			(at 207.01 128.2762 0)
 			(show_name no)
@@
 			(project "RK3576 SBC"
 				(path "/b79dbff4-0cad-4ff7-bec2-7c0e4f8b14d3/34f9b0cb-aeae-42b4-a2af-a0a79afcf392/51173a63-65bb-4420-9c6d-af77ebfb98d4"
-					(reference "C141")
+					(reference "C149")
 					(unit 1)
 				)
@@
 		(in_pos_files yes)
 		(dnp no)
-		(property "Reference" "#PWR0192"
+		(property "Reference" "#PWR0204"
 			(at 72.39 82.55 0)
 			(hide yes)
@@
 			(project "RK3576 SBC"
 				(path "/b79dbff4-0cad-4ff7-bec2-7c0e4f8b14d3/34f9b0cb-aeae-42b4-a2af-a0a79afcf392/51173a63-65bb-4420-9c6d-af77ebfb98d4"
-					(reference "#PWR0192")
+					(reference "#PWR0204")
 					(unit 1)
 				)
@@
 		(dnp no)
 		(fields_autoplaced yes)
-		(property "Reference" "C140"
+		(property "Reference" "C148"
 			(at 63.5 105.4162 0)
 			(show_name no)
@@
 			(project "RK3576 SBC"
 				(path "/b79dbff4-0cad-4ff7-bec2-7c0e4f8b14d3/34f9b0cb-aeae-42b4-a2af-a0a79afcf392/51173a63-65bb-4420-9c6d-af77ebfb98d4"
-					(reference "C140")
+					(reference "C148")
 					(unit 1)
 				)
@@
 		(in_pos_files yes)
 		(dnp no)
-		(property "Reference" "#PWR0199"
+		(property "Reference" "#PWR0211"
 			(at 60.96 99.06 0)
 			(hide yes)
@@
 			(project "RK3576 SBC"
 				(path "/b79dbff4-0cad-4ff7-bec2-7c0e4f8b14d3/34f9b0cb-aeae-42b4-a2af-a0a79afcf392/51173a63-65bb-4420-9c6d-af77ebfb98d4"
-					(reference "#PWR0199")
+					(reference "#PWR0211")
 					(unit 1)
 				)
@@
 		(in_pos_files yes)
 		(dnp no)
-		(property "Reference" "#PWR0203"
+		(property "Reference" "#PWR0215"
 			(at 218.44 139.7 0)
 			(hide yes)
@@
 			(project "RK3576 SBC"
 				(path "/b79dbff4-0cad-4ff7-bec2-7c0e4f8b14d3/34f9b0cb-aeae-42b4-a2af-a0a79afcf392/51173a63-65bb-4420-9c6d-af77ebfb98d4"
-					(reference "#PWR0203")
+					(reference "#PWR0215")
 					(unit 1)
 				)
@@
 		(in_pos_files yes)
 		(dnp no)
-		(property "Reference" "#PWR0193"
+		(property "Reference" "#PWR0205"
 			(at 96.52 82.55 0)
 			(hide yes)
@@
 			(project "RK3576 SBC"
 				(path "/b79dbff4-0cad-4ff7-bec2-7c0e4f8b14d3/34f9b0cb-aeae-42b4-a2af-a0a79afcf392/51173a63-65bb-4420-9c6d-af77ebfb98d4"
-					(reference "#PWR0193")
+					(reference "#PWR0205")
 					(unit 1)
 				)
@@
 		(dnp no)
 		(fields_autoplaced yes)
-		(property "Reference" "C136"
+		(property "Reference" "C144"
 			(at 85.09 87.6362 0)
 			(show_name no)
@@
 			(project "RK3576 SBC"
 				(path "/b79dbff4-0cad-4ff7-bec2-7c0e4f8b14d3/34f9b0cb-aeae-42b4-a2af-a0a79afcf392/51173a63-65bb-4420-9c6d-af77ebfb98d4"
-					(reference "C136")
+					(reference "C144")
 					(unit 1)
 				)
@@
 		(in_pos_files yes)
 		(dnp no)
-		(property "Reference" "#PWR0194"
+		(property "Reference" "#PWR0206"
 			(at 72.39 97.79 0)
 			(hide yes)
@@
 			(project "RK3576 SBC"
 				(path "/b79dbff4-0cad-4ff7-bec2-7c0e4f8b14d3/34f9b0cb-aeae-42b4-a2af-a0a79afcf392/51173a63-65bb-4420-9c6d-af77ebfb98d4"
-					(reference "#PWR0194")
+					(reference "#PWR0206")
 					(unit 1)
 				)
@@
 		(dnp no)
 		(fields_autoplaced yes)
-		(property "Reference" "C138"
+		(property "Reference" "C146"
 			(at 109.22 87.6362 0)
 			(show_name no)
@@
 			(project "RK3576 SBC"
 				(path "/b79dbff4-0cad-4ff7-bec2-7c0e4f8b14d3/34f9b0cb-aeae-42b4-a2af-a0a79afcf392/51173a63-65bb-4420-9c6d-af77ebfb98d4"
-					(reference "C138")
+					(reference "C146")
 					(unit 1)
 				)
@@
 		(in_pos_files yes)
 		(dnp no)
-		(property "Reference" "#PWR0200"
+		(property "Reference" "#PWR0212"
 			(at 210.82 111.76 0)
 			(hide yes)
@@
 			(project "RK3576 SBC"
 				(path "/b79dbff4-0cad-4ff7-bec2-7c0e4f8b14d3/34f9b0cb-aeae-42b4-a2af-a0a79afcf392/51173a63-65bb-4420-9c6d-af77ebfb98d4"
-					(reference "#PWR0200")
+					(reference "#PWR0212")
 					(unit 1)
 				)

Commit message: SBCv0.3
there is no big thing update just some LCSC & Mouser parts
and Big problem deleted alot of component values (:
Parts:
- C143, C144, C145, C146, C147, C148: footprint Capacitor_SMD:C_0402_1005Metric_Pad0.74x0.62mm_HandSolder -> Capacitor_SMD:C_0201_0603Metric_Pad0.64x0.40mm_HandSolder; LCSC Part (none) -> C5209398; Mouser Part (none) -> CL03A105KP3NSNC
- C149, C150: LCSC Part (none) -> C541431; Mouser Part (none) -> 603-CC402FRNPO9BN180
- R39: value 8.2k -> (property "ki_keywords" "capacitor cap"
- R40: value 22R -> (property "Description" "Unpolarized capacitor, small symbol"
- R41: value 510k -> (none); LCSC Part (none) -> (at 0 0 0)
- U3: value RK3576 -> (none); LCSC Part (none) -> (polyline
- Y2: value XTM32026000FT00351001 -> (none); footprint Crystal:Crystal_SMD_3225-4Pin_3.2x2.5mm -> (effects

Commit message: SBCv0.4
add LCSC & Mouser parts 
and solve the deleted value in the past version
Parts:
- removed R39: (property "ki_keywords" "capacitor cap", PCM_Resistor_SMD_AKL:R_0402_1005Metric_Pad0.72x0.64mm, symbol Device:R_Small
- removed R40: (property "Description" "Unpolarized capacitor, s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, PCM_Resistor_SMD_AKL:R_0402_1005Metric_Pad0.72x0.64mm, symbol Device:R_Small
- removed R41: (no value), PCM_Resistor_SMD_AKL:R_0402_1005Metric_Pad0.72x0.64mm, symbol Device:R_Small
- removed Y2: (no value), (effects, symbol Device:Crystal_GND24
- added R215: 510k, PCM_Resistor_SMD_AKL:R_0402_1005Metric, symbol Device:R_Small
- added R216: 22R, PCM_Resistor_SMD_AKL:R_0402_1005Metric, symbol Device:R_Small
- added R217: 8.2k, PCM_Resistor_SMD_AKL:R_0402_1005Metric, symbol Device:R_Small
- added Y7: XTM32026000FT00351001, Crystal:Crystal_SMD_3225-4Pin_3.2x2.5mm, symbol Device:Crystal_GND24
- U3: value (none) -> RK3576; LCSC Part (polyline -> C42388007
Connections:
- net GND: now also R217.2, Y7.2 (G), Y7.4 (G)
- net UFS3.1_TX_REXT: now also R217.1
- net at U3.AK5 (OSC_UFS_XIN): now also R215.1, R216.1
- net at C149.1, U3.AL5 (OSC_UFS_XOUT): now also R215.2, Y7.3
- net at C150.1: now also R216.2, Y7.1
