File: rk3576_usb2.kicad_sch (KiCad schematic)
At the start: 8 parts, among them U27 RK3576

Commit message: Add files via upload
Parts:
- C115: renamed from C321; value 100n -> 1u
- C116: renamed from C322; value 100n -> 1u
- C117: renamed from C323; value 100n -> 1u
- renumbered R134 to R31, R133 to R32, R135 to R33, R136 to R34, U27 to U2

Commit message: SBC Board V0.2
The SBC schematics before footprint and part number check
Parts:
- U3: renamed from U2; footprint (none) -> easyeda2kicad:FCCSP-698_L17.2-W16.1-TL_RK3576
- renumbered C115 to C123, C116 to C124, C117 to C125

Commit message: SBCv0.3
there is no big thing update just some LCSC & Mouser parts
and Big problem deleted alot of component values (:
Parts:
- C123, C124, C125: footprint Capacitor_SMD:C_0402_1005Metric_Pad0.74x0.62mm_HandSolder -> Capacitor_SMD:C_0201_0603Metric_Pad0.64x0.40mm_HandSolder; LCSC Part (none) -> C5209398; Mouser Part (none) -> CL03A105KP3NSNC
- R31, R33: value 4.7k -> (none); LCSC Part (none) -> )
- R32, R34: value 200R -> )
- U3: value RK3576 -> (none); LCSC Part (none) -> (polyline

Commit message: SBCv0.4
add LCSC & Mouser parts 
and solve the deleted value in the past version
Parts:
- removed R31, R33: (no value), PCM_Resistor_SMD_AKL:R_0402_1005Metric_Pad0.72x0.64mm, symbol Device:R_Small
- removed R32, R34: ), PCM_Resistor_SMD_AKL:R_0402_1005Metric_Pad0.72x0.64mm, symbol Device:R_Small
- added R208, R210: 4.7k, PCM_Resistor_SMD_AKL:R_0402_1005Metric, symbol Device:R_Small
- added R209, R211: 200R, PCM_Resistor_SMD_AKL:R_0402_1005Metric, symbol Device:R_Small
- U3: value (none) -> RK3576; LCSC Part (polyline -> C42388007
Connections:
- net GND: now also R209.2, R211.2
- net VCC_3V3_S0: now also R208.2, R210.2
- net at U3.2R3 (USB2_OTG0_REXT): now also R209.1
- net at U3.2T10 (USB2_OTG1_VBUSDET): now also R210.1
- net at U3.2P3 (USB2_OTG0_VBUSDET): now also R208.1
- net at U3.2U8 (USB2_OTG1_REXT): now also R211.1
