File: rtc.kicad_sch (KiCad schematic)
At the start: 13 parts, among them J14 B2B Connector, Q7 AO3401A, U3 RV-3028-C7

Commit message: SBC Board V0.2
The SBC schematics before footprint and part number check
Parts:
- removed J14: B2B Connector, Connector_JST:JST_EH_S2B-EH_1x02_P2.50mm_Horizontal, symbol PCM_SL_Connectors:JST_02
- added BT1: BS-06-B4AA012, easyeda2kicad:BAT-SMD_BS-06-B4AA012, symbol PCM_fab:Battery-Holder_Coin-Cell_CR2032_Linx_BAT-HLD-001
- renumbered C367 to C370, C379 to C371, D26 to D17, R51 to R158, R175 to R160, R50 to R161, R134 to R162, R143 to R163, U3 to U32
Connections:
- net GND: now also BT1.2 (-)
- net at F1.2: now also BT1.1 (+)
Other:
- moved on the sheet: C370, C371, D17, F1, Q7, R158, R159, R160, R161, R162, R163, U32

Commit message: SBCv0.3
there is no big thing update just some LCSC & Mouser parts
and Big problem deleted alot of component values (:
Parts:
- BT1: LCSC Part (none) -> C964758
- C370, C371: footprint Capacitor_SMD:C_0402_1005Metric_Pad0.74x0.62mm_HandSolder -> Capacitor_SMD:C_0201_0603Metric_Pad0.64x0.40mm_HandSolder; LCSC Part (none) -> C5209398; Mouser Part (none) -> CL03A105KP3NSNC
- D17: LCSC Part (none) -> C113975; Mouser Part (none) -> 581-SMBJ5.0CA
- F1: value 500mA -> 1A; footprint (none) -> Fuse:Fuse_1812_4532Metric; LCSC Part (none) -> C28326708
- R158, R161: value 10k -> (none); LCSC Part (none) -> (at 0 0 0)
- R159, R160: value 2.2k -> (none); LCSC Part (none) -> (do_not_autoplace no)
- R162, R163: value 22R -> (property "Description" "Unpolarized capacitor, small symbol"
- U32: value RV-3028-C7 -> (none); footprint Package_SON:MicroCrystal_C7_SON-8_1.5x3.2mm_P0.9mm -> (effects

Commit message: SBCv0.4
add LCSC & Mouser parts 
and solve the deleted value in the past version
Parts:
- removed R158: (no value), PCM_Resistor_SMD_AKL:R_0402_1005Metric, symbol Device:R_Small
- added R241: 22R, PCM_Resistor_SMD_AKL:R_0402_1005Metric, symbol Device:R_Small
- Q7: LCSC Part (none) -> C347476
- R159, R160: value (none) -> 2.2k; LCSC Part (do_not_autoplace no) -> C114762; Mouser Part (none) -> 603-RC0402FR-072K2L
- R161: value (none) -> 10k; LCSC Part (at 0 0 0) -> C60490; Mouser Part (none) -> 603-RC0402FR-0710KL
- R162: value (property "Description" "Unpolarized capacitor, small symbol" -> 10k; footprint PCM_Resistor_SMD_AKL:R_0402_1005Metric_Pad0.72x0.64mm -> PCM_Resistor_SMD_AKL:R_0402_1005Metric; LCSC Part (none) -> C60490; Mouser Part (none) -> 603-RC0402FR-0710KL
- R163: value (property "Description" "Unpolarized capacitor, small symbol" -> 22R; footprint PCM_Resistor_SMD_AKL:R_0402_1005Metric_Pad0.72x0.64mm -> PCM_Resistor_SMD_AKL:R_0402_1005Metric; LCSC Part (none) -> C114765; Mouser Part (none) -> 603-RC0402FR-0722RL
- U32: value (none) -> RV-3028-C7; footprint (effects -> Package_SON:MicroCrystal_C7_SON-8_1.5x3.2mm_P0.9mm; Mouser Part (none) -> 428-203591-MG01
Connections:
- net GND: now also R162.2
- net RTC_32KOUT_SOC: now also R163.2; no longer R162.2
- net RTC_32KOUT_WIFI: now also R241.2; no longer R163.2
- net at Q7.1 (G): now also R162.1
- net at R161.2, R163.1, U32.1 (CLKOUT): now also R241.1; no longer R162.1
- net I2C2_SCL_M0_CC_RTC renamed I2C2_SCL_M0_CC_RTC_EEPROM
- net I2C2_SDA_M0_CC_RTC renamed I2C2_SDA_M0_CC_RTC_EEPROM
