File: saradc.kicad_sch (KiCad schematic)
At the start: 25 parts, among them SW2 SW_DIP_x03, SW3 SW_Push, SW4 SW_Push, U27 RK3576

Commit message: Add files via upload
Parts:
- renumbered C314 to C105, C315 to C106, C299 to C107, C300 to C108, C301 to C109, C302 to C110, C303 to C111, C304 to C112, C305 to C113, C306 to C114, D18 to D5, D19 to D6, R125 to R22, R126 to R23, R127 to R24, R120 to R25, R128 to R26, R129 to R27, R130 to R28, R131 to R29, R132 to R30, U27 to U2

Commit message: SBC Board V0.2
The SBC schematics before footprint and part number check
Parts:
- U3: renamed from U2; footprint (none) -> easyeda2kicad:FCCSP-698_L17.2-W16.1-TL_RK3576
- renumbered C105 to C113, C106 to C114, C107 to C115, C108 to C116, C109 to C117, C110 to C118, C111 to C119, C112 to C120, C113 to C121, C114 to C122

Commit message: SBCv0.3
there is no big thing update just some LCSC & Mouser parts
and Big problem deleted alot of component values (:
Parts:
- C113, C114, C115, C116, C117, C118, C119, C120, C121, C122: footprint Capacitor_SMD:C_0402_1005Metric_Pad0.74x0.62mm_HandSolder -> Capacitor_SMD:C_0201_0603Metric_Pad0.64x0.40mm_HandSolder; LCSC Part (none) -> C5209398; Mouser Part (none) -> CL03A105KP3NSNC
- D5, D6: LCSC Part (none) -> C113975; Mouser Part (none) -> 581-SMBJ5.0CA
- R22: value 6.8k -> (none); LCSC Part (none) -> (hide yes)
- R23: value 23.2k -> (none); LCSC Part (none) -> (effects
- R24: value 88.7k -> (none); Mouser Part (none) -> (font (size 1.27 1.27))
- R25, R26, R27, R28, R29, R30: value 10k -> )
- SW2: value SW_DIP_x03 -> (none); footprint (none) -> (xy -1.524 0.508) (xy 1.524 0.508)
- SW3: value SW_Push -> (none); Mouser Part (none) -> (pts
- SW4: value SW_Push -> (none); Mouser Part (none) -> )
- U3: value RK3576 -> (none); LCSC Part (none) -> (polyline

Commit message: SBCv0.4
add LCSC & Mouser parts 
and solve the deleted value in the past version
Parts:
- removed R22, R23, R24: (no value), PCM_Resistor_SMD_AKL:R_0402_1005Metric_Pad0.72x0.64mm, symbol Device:R_Small
- removed R25, R26, R27, R28, R29, R30: ), PCM_Resistor_SMD_AKL:R_0402_1005Metric_Pad0.72x0.64mm, symbol Device:R_Small
- removed SW2: (no value), (xy -1.524 0.508) (xy 1.524 0.508), symbol Switch:SW_DIP_x03
- removed SW3, SW4: (no value), Button_Switch_SMD:SW_Push_1P1T_NO_CK_PTS125Sx85SMTR, symbol Switch:SW_Push
- added R199: 6.8k, PCM_Resistor_SMD_AKL:R_0402_1005Metric, symbol Device:R_Small
- added R200: 23.2k, PCM_Resistor_SMD_AKL:R_0402_1005Metric, symbol Device:R_Small
- added R201: 88.7k, PCM_Resistor_SMD_AKL:R_0402_1005Metric, symbol Device:R_Small
- added R202, R203, R204, R205, R206, R207: 10k, PCM_Resistor_SMD_AKL:R_0402_1005Metric, symbol Device:R_Small
- added SW7: DSHP03TS-S, Button_Switch_SMD:SW_DIP_SPSTx03_Slide_KingTek_DSHP03TJ_W5.25mm_P1.27mm_JPin, symbol Switch:SW_DIP_x03
- added SW8, SW9: XUNPU TS-1089S-02526, easyeda2kicad:XUNPU TS-1089S-02526, symbol Switch:SW_Push
- U3: value (none) -> RK3576; LCSC Part (polyline -> C42388007
Connections:
- net GND: now also R199.1, R200.1, R201.1, R205.2, R207.2, SW8.2, SW9.2
- net SARADC_VIN0_BOOT: now also R202.2, SW7.4, SW7.5, SW7.6, SW8.1
- net SARADC_VIN1_KEY/RECOVERY: now also R203.2, SW9.1
- net SARADC_VIN2_HW_ID: now also R206.2, R207.1
- net SARADC_VIN5_BOM_ID: now also R204.2, R205.1
- net VCCA_1V8_S0: now also R202.1, R203.1, R204.1, R206.1
- new net: R201.2, SW7.3
- new net: R199.2, SW7.1
- new net: R200.2, SW7.2
