File: usb3.2_host.kicad_sch (KiCad schematic)
At the start: 58 parts, among them J2 USB3_A_Stacked, J3 USB3_A_Stacked, U10 TPD4E05U06DQA, U11 TPD4E05U06DQA, U12 TPD4E05U06DQA, U13 TPD4E05U06DQA, U29 AP2553W6-7, U30 AP2553W6-7, U31 AP2553W6-7, U32 AP2553W6-7

Commit message: Add files via upload
Parts:
- removed C400, C67, C68: 22u, Capacitor_SMD:C_0603_1608Metric, symbol New_Library_0:C_Small_edited
- removed C403, C404, C405: 1u, Capacitor_SMD:C_0402_1005Metric_Pad0.74x0.62mm_HandSolder, symbol New_Library_0:C_Small_edited
- removed C59, C61, C63, C65, C70, C72, C74, C76: 100n, Capacitor_SMD:C_0201_0603Metric_Pad0.64x0.40mm_HandSolder, symbol New_Library_0:C_Small_edited
- removed D20, D21, D22, D5: PESD5V0S1BA, PCM_Diode_SMD_AKL:D_SOD-323_TVS, symbol PCM_Diode_TVS_AKL:PESD5V0S1BA
- removed R152, R159: 15k, PCM_Resistor_SMD_AKL:R_0402_1005Metric, symbol Device:R_Small
- removed R153: 100k, PCM_Resistor_SMD_AKL:R_0402_1005Metric, symbol Device:R_Small
- removed R155: 2.2k, PCM_Resistor_SMD_AKL:R_0402_1005Metric, symbol Device:R_Small
- removed U30: AP2553W6-7, symbol New_Library:AP2553W6-7
- added C185, C187, C189, C191, C197, C199, C201, C203: 100n, Capacitor_SMD:C_0201_0603Metric_Pad0.64x0.40mm_HandSolder, symbol New_Library_0:C_Small_edited
- added C368, C370, C372: 22u, Capacitor_SMD:C_0603_1608Metric, symbol New_Library_0:C_Small_edited
- added C369, C371, C373: 1u, Capacitor_SMD:C_0402_1005Metric_Pad0.74x0.62mm_HandSolder, symbol New_Library_0:C_Small_edited
- added D19, D21, D22, D23: SMBJ5.0CA, PCM_Diode_SMD_AKL:D_SMB_TVS, symbol PCM_Diode_TVS_AKL:SMBJ5.0CA
- added R165, R168: 2.2k, PCM_Resistor_SMD_AKL:R_0402_1005Metric, symbol Device:R_Small
- added R166: 15k, PCM_Resistor_SMD_AKL:R_0402_1005Metric, symbol Device:R_Small
- added R167: 100k, PCM_Resistor_SMD_AKL:R_0402_1005Metric, symbol Device:R_Small
- added U33: AP2553W6-7, symbol New_Library:AP2553W6-7
- R160, R163: value 100k -> 15k
- R161, R164: value 2.2k -> 100k
- R162: value 15k -> 2.2k
- renumbered C401 to C180, C56 to C182, C58 to C184, C60 to C186, C62 to C188, C64 to C190, C71 to C196, C73 to C198, C75 to C200, C77 to C202, FL5 to FL4, FL4 to FL5, J2 to J4, J3 to J5, R148 to R57, R151 to R59, R147 to R60, R156 to R63, R154 to R64, R157 to R71, R158 to R72, U10 to U14, U11 to U15, U29 to U8
Connections:
- net CUSB_{HOST3}_SSRX1_N: now also C185.2
- net CUSB_{HOST3}_SSRX1_P: now also C187.2
- net CUSB_{HOST3}_SSTX1_N: now also C189.2
- net CUSB_{HOST3}_SSTX1_P: now also C191.2
- net CUSB_{HOST4}_SSRX1_N: now also C197.2
- net CUSB_{HOST4}_SSRX1_P: now also C199.2
- net CUSB_{HOST4}_SSTX1_N: now also C201.2
- net CUSB_{HOST4}_SSTX1_P: now also C203.2
- net GND: now also R161.2, R164.2, C368.2, C369.2, C370.2, C371.2, C372.2, C373.2, D19.1 (K), D21.1 (K), D22.1 (K), D23.1 (K), R166.2, R167.2, U33.2 (GND); no longer R162.2
- net USB_{HOST3}_SSRX1_N: now also C185.1
- net USB_{HOST3}_SSRX1_P: now also C187.1
- net USB_{HOST3}_SSTX1_N: now also C189.1
- net USB_{HOST3}_SSTX1_P: now also C191.1
- net USB_{HOST4}_SSRX1_N: now also C197.1
- net USB_{HOST4}_SSRX1_P: now also C199.1
- net USB_{HOST4}_SSTX1_N: now also C201.1
- net USB_{HOST4}_SSTX1_P: now also C203.1
- net Vbus_USB_{HOST1}: now also D19.2 (A)
- net Vbus_USB_{HOST2}: now also U31.6 (OUT), C368.1, D21.2 (A); no longer U32.6 (OUT)
- net Vbus_USB_{HOST3}: now also U32.6 (OUT), C370.1, D22.2 (A)
- net Vbus_USB_{HOST4}: now also C372.1, D23.2 (A), U33.6 (OUT); no longer U31.6 (OUT)
- net at R161.1, U31.3 (EN): now also R162.1; no longer R160.1
- net at U31.5 (ILIM): now also R160.1
- net at U32.5 (ILIM): now also R163.1; no longer R162.1
- net at R164.1, U32.3 (EN): now also R165.1; no longer R163.1
- net +5V renamed VCC5V0_SYS
- net VCC5V0_SYS: now also C369.1, C371.1, C373.1, U33.1 (IN)
- removed net USB_{HOST}_PWR_EN: R161.2, R164.2, R57.2
- new net: R166.1, U33.5 (ILIM)
- new net: R167.1, R168.1, U33.3 (EN)
- new net USB3_HOST_PWREN_H: R162.2, R165.2, R168.2, R57.2
Other:
- moved on the sheet: C180, C182, FL3, FL5, J5A, J5B, R57, R59, R60, R64, R72, U12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

Commit message: SBC Board V0.2
The SBC schematics before footprint and part number check
Parts:
- added C191, C192, C193, C194, C199, C202, C203, C204, C206, C207, C208, C209, C210, C211, C212, C213, C216, C222: 1u, Capacitor_SMD:C_0201_0603Metric_Pad0.64x0.40mm_HandSolder, symbol New_Library_0:C_Small_edited
- added C198, C200, C217, C218: 10u, Capacitor_SMD:C_0603_1608Metric, symbol New_Library_0:C_Small_edited
- added C214: 10u, Capacitor_SMD:C_0201_0603Metric_Pad0.64x0.40mm_HandSolder, symbol New_Library_0:C_Small_edited
- added C226, C227: 20pF, Capacitor_SMD:C_0402_1005Metric_Pad0.74x0.62mm_HandSolder, symbol New_Library_0:C_Small_edited
- added L11: ???, Inductor_SMD:L_1008_2520Metric, symbol Device:L_Small
- added R58, R59: 100k, PCM_Resistor_SMD_AKL:R_0402_1005Metric, symbol Device:R_Small
- added R64: 6.2k, PCM_Resistor_SMD_AKL:R_0402_1005Metric, symbol Device:R_Small
- added R65: 0R, PCM_Resistor_SMD_AKL:R_0402_1005Metric, symbol Device:R_Small
- added U11: RTS5411S-GR, Package_DFN_QFN:QFN-76-1EP_9x9mm_P0.4mm_EP5.81x6.31mm_ThermalVias, symbol New_Library:RTS5411S-GR
- added Y3: K3A120002010, Crystal:Crystal_SMD_3225-4Pin_3.2x2.5mm_HandSoldering, symbol Device:Crystal_GND24
- renumbered C180 to C189, C182 to C190, C184 to C195, C186 to C196, C188 to C197, C190 to C201, C369 to C205, C368 to C215, C196 to C219, C198 to C220, C200 to C221, C202 to C223, C371 to C224, C370 to C225, C185 to C228, C187 to C229, C189 to C230, C191 to C231, C373 to C232, C372 to C233, C197 to C234, C199 to C235, C201 to C236, C203 to C237, D19 to D10, D21 to D11, D22 to D12, D23 to D13, FL4 to FL3, FL3 to FL4, J4 to J3, J5 to J4, R57 to R51, R59 to R52, R60 to R53, R63 to R54, R162 to R55, R160 to R56, R161 to R57, R71 to R60, R165 to R61, R163 to R62, R164 to R63, R64 to R66, R168 to R67, R166 to R68, R167 to R69, R72 to R70, U31 to U10, U32 to U12, U33 to U13, U12 to U14, U13 to U15, U14 to U16, U15 to U17, U8 to U9
Connections:
- net GND: now also C191.2, C192.2, C193.2, C194.2, C198.2, C199.2, C200.2, C202.2, C203.2, C204.2, C206.2, C207.2, C208.2, C209.2, C210.2, C211.2, C212.2, C213.2, C214.2, C216.2, C217.2, C218.2, C222.2, C226.2, C227.2, R59.2, R64.2, R65.2, U11.51 (SWR_GND), U11.61 (GND), U11.77 (EPAD), Y3.2 (G), Y3.4 (G)
- net USB_{HOST1}_D_N: now also U11.72 (DSP1_DM)
- net USB_{HOST1}_D_P: now also U11.71 (DSP1_DP)
- net USB_{HOST1}_SSRX1_N: now also U11.66 (DSP1_SSTX-)
- net USB_{HOST1}_SSRX1_P: now also U11.65 (DSP1_SSTX+)
- net USB_{HOST1}_SSTX1_N: now also U11.69 (DSP1_SSRX-)
- net USB_{HOST1}_SSTX1_P: now also U11.68 (DSP1_SSRX+)
- net USB_{HOST2}_D_N: now also U11.6 (DSP2_DM)
- net USB_{HOST2}_D_P: now also U11.5 (DSP2_DP)
- net USB_{HOST2}_SSRX1_N: now also U11.9 (DSP2_SSTX-)
- net USB_{HOST2}_SSRX1_P: now also U11.8 (DSP2_SSTX+)
- net USB_{HOST2}_SSTX1_N: now also U11.12 (DSP2_SSRX-)
- net USB_{HOST2}_SSTX1_P: now also U11.11 (DSP2_SSRX+)
- net USB_{HOST3}_D_N: now also U11.21 (DSP3_DM)
- net USB_{HOST3}_D_P: now also U11.20 (DSP3_DP)
- net USB_{HOST3}_SSRX1_N: now also U11.15 (DSP3_SSTX-)
- net USB_{HOST3}_SSRX1_P: now also U11.14 (DSP3_SSTX+)
- net USB_{HOST3}_SSTX1_N: now also U11.18 (DSP3_SSRX-)
- net USB_{HOST3}_SSTX1_P: now also U11.17 (DSP3_SSRX+)
- net USB_{HOST4}_D_N: now also U11.24 (DSP4_DM)
- net USB_{HOST4}_D_P: now also U11.23 (DSP4_DP)
- net USB_{HOST4}_SSRX1_N: now also U11.27 (DSP4_SSTX-)
- net USB_{HOST4}_SSRX1_P: now also U11.26 (DSP4_SSTX+)
- net USB_{HOST4}_SSTX1_N: now also U11.30 (DSP4_SSRX-)
- net USB_{HOST4}_SSTX1_P: now also U11.29 (DSP4_SSRX+)
- net VCC5V0_SYS: now also C216.1, C217.1, C218.1, C222.1, R58.1, U11.53 (SWR_V5_IN), U11.54 (LDO_V5_IN), U11.76 (SPWR_DET)
- net USB3_HOST_PWREN_H renamed USB_{HOST}_PWREN_H
- new net: R64.1, U11.1 (RREF)
- new net: R58.2, R59.1, U11.2 (BPWR_DET)
- new net: R65.1, U11.45 (SCS)
- new net: L11.2, U11.55 (V33_OUT)
- new net +1.2V_{HUB}: C191.1, C192.1, C193.1, C194.1, C200.1, C202.1, C203.1, C204.1, L11.1, U11.22 (DV33), U11.3 (DV12), U11.4 (DV33), U11.48 (DV33), U11.49 (DV12), U11.50 (DV12), U11.73 (DV33)
- new net +3.3V_{HUB}: C198.1, C199.1, C206.1, C207.1, C208.1, C209.1, C210.1, C211.1, C212.1, C213.1, C214.1, U11.13 (AV12), U11.19 (AV12), U11.25 (AV12), U11.31 (AV12), U11.52 (SWR_OUT), U11.58 (AV12), U11.64 (AV12), U11.7 (AV12), U11.70 (AV12)
- new net Crystal_{HUB}_IN: C227.1, U11.74 (XTLI), Y3.1
- new net Crystal_{HUB}_OUT: C226.1, U11.75 (XTLO), Y3.3
- new net USB_{HUB}_D_N: U11.57 (USP_DM)
- new net USB_{HUB}_D_P: U11.56 (USP_DP)
- new net USB_{HUB}_SSRX1_N: U11.59 (USP_SSTX-)
- new net USB_{HUB}_SSRX1_P: U11.60 (USP_SSTX+)
- new net USB_{HUB}_SSTX1_N: U11.62 (USP_SSRX-)
- new net USB_{HUB}_SSTX1_P: U11.63 (USP_SSRX+)
- no-connect marks 20 -> 39
Other:
- moved on the sheet: C189, C190, C195, C196, C197, C201, C205, C215, C219, C220, C221, C223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

Commit message: SBCv0.3
there is no big thing update just some LCSC & Mouser parts
and Big problem deleted alot of component values (:
Parts:
- removed C214: 10u, Capacitor_SMD:C_0201_0603Metric_Pad0.64x0.40mm_HandSolder, symbol New_Library_0:C_Small_edited
- removed C228, C229, C230, C231, C234, C235, C236, C237: 100n, Capacitor_SMD:C_0201_0603Metric_Pad0.64x0.40mm_HandSolder, symbol New_Library_0:C_Small_edited
- removed FL2, FL3, FL4, FL5: 0603USB-142, Inductor_SMD:L_CommonModeChoke_Coilcraft_0603USB, symbol Filter:0603USB-142
- added C399: 10u, Capacitor_SMD:C_0603_1608Metric, symbol New_Library_0:C_Small_edited
- added C402, C403, C404, C405, C406, C407, C408, C409: 100n, Capacitor_SMD:C_0201_0603Metric_Pad0.64x0.40mm_HandSolder, symbol New_Library_0:C_Small_edited
- added U40, U42, U44, U45: ICMEF112P900MFR, Datasheet_Footprints:ICMEF112P900MFR, symbol Datasheet_Symbols:ICMEF112P900MFR
- C189, C205, C224, C232: footprint Capacitor_SMD:C_0402_1005Metric_Pad0.74x0.62mm_HandSolder -> Capacitor_SMD:C_0201_0603Metric_Pad0.64x0.40mm_HandSolder; LCSC Part (none) -> C5209398; Mouser Part (none) -> CL03A105KP3NSNC
- C190, C215, C225, C233: LCSC Part (none) -> C86295; Mouser Part (none) -> CL10A226MP8NUNE
- C191, C192, C193, C194, C199, C202, C203, C204, C206, C207, C208, C209, C210, C211, C212, C213, C216, C222: LCSC Part (none) -> C5209398; Mouser Part (none) -> CL03A105KP3NSNC
- C195, C196, C197, C201, C219, C220, C221, C223: LCSC Part (none) -> C307380; Mouser Part (none) -> 187-CL03A104KO3NNNC; now left out of the parts list
- C198, C200, C217, C218: LCSC Part (none) -> C19702; Mouser Part (none) -> 187-CL10A106KP8NNNC
- C226, C227: value 20pF -> 34pF; LCSC Part (none) -> C114394; Mouser Part (none) -> CC402JRNPO9BN360
- D10, D11, D12, D13: LCSC Part (none) -> C113975; Mouser Part (none) -> 581-SMBJ5.0CA
- J3, J4: LCSC Part (none) -> C42403016
- L11: LCSC Part (none) -> (show_name no)
- R51, R55, R61, R67: value 2.2k -> (none); LCSC Part (none) -> (do_not_autoplace no)
- R52, R56, R62, R68: value 15k -> (none); LCSC Part (none) -> (hide yes)
- R53, R57, R58, R59, R63, R69: value 100k -> (none); LCSC Part (none) -> (show_name no)
- R54, R60, R65, R66, R70: value 0R -> (none); LCSC Part (none) -> (effects
- R64: value 6.2k -> (none); Mouser Part (none) -> (font (size 1.27 1.27))
- U10, U12, U13, U9: footprint (none) -> Package_TO_SOT_SMD:SOT-23-6_Handsoldering; LCSC Part (none) -> C212302; Mouser Part (none) -> 621-AP2553W6-7
- U11: value RTS5411S-GR -> (none); Mouser Part (none) -> (fill (type none))
- U14, U15, U16, U17: value TPD4E05U06DQA -> (none); Mouser Part (none) -> )
- Y3: value K3A120002010 -> (none); footprint Crystal:Crystal_SMD_3225-4Pin_3.2x2.5mm_HandSoldering -> (none)
Connections:
- net +3.3V_{HUB}: now also C399.1
- net CUSB_{HOST1}_D_N: now also U40.1 (IN1)
- net CUSB_{HOST1}_D_P: now also U40.2 (IN2)
- net CUSB_{HOST2}_D_N: now also U42.1 (IN1)
- net CUSB_{HOST2}_D_P: now also U42.2 (IN2)
- net CUSB_{HOST3}_D_N: now also U44.1 (IN1)
- net CUSB_{HOST3}_D_P: now also U44.2 (IN2)
- net CUSB_{HOST3}_SSRX1_N: now also C402.2
- net CUSB_{HOST3}_SSRX1_P: now also C403.2
- net CUSB_{HOST3}_SSTX1_N: now also C404.2
- net CUSB_{HOST3}_SSTX1_P: now also C405.2
- net CUSB_{HOST4}_D_N: now also U45.1 (IN1)
- net CUSB_{HOST4}_D_P: now also U45.2 (IN2)
- net CUSB_{HOST4}_SSRX1_N: now also C406.2
- net CUSB_{HOST4}_SSRX1_P: now also C407.2
- net CUSB_{HOST4}_SSTX1_N: now also C408.2
- net CUSB_{HOST4}_SSTX1_P: now also C409.2
- net GND: now also C399.2, U40.5 (GND), U40.6 (GND), U42.5 (GND), U42.6 (GND), U44.5 (GND), U44.6 (GND), U45.5 (GND), U45.6 (GND)
- net USB_{HOST1}_D_N: now also U40.3 (OUT1)
- net USB_{HOST1}_D_P: now also U40.4 (OUT2)
- net USB_{HOST2}_D_N: now also U42.3 (OUT1)
- net USB_{HOST2}_D_P: now also U42.4 (OUT2)
- net USB_{HOST3}_D_N: now also U44.3 (OUT1)
- net USB_{HOST3}_D_P: now also U44.4 (OUT2)
- net USB_{HOST3}_SSRX1_N: now also C402.1
- net USB_{HOST3}_SSRX1_P: now also C403.1
- net USB_{HOST3}_SSTX1_N: now also C404.1
- net USB_{HOST3}_SSTX1_P: now also C405.1
- net USB_{HOST4}_D_N: now also U45.3 (OUT1)
- net USB_{HOST4}_D_P: now also U45.4 (OUT2)
- net USB_{HOST4}_SSRX1_N: now also C406.1
- net USB_{HOST4}_SSRX1_P: now also C407.1
- net USB_{HOST4}_SSTX1_N: now also C408.1
- net USB_{HOST4}_SSTX1_P: now also C409.1
Other:
- moved on the sheet: C195, C196, C197, C201, C219, C220, C221, C223

Commit message: SBCv0.4
add LCSC & Mouser parts 
and solve the deleted value in the past version
Parts:
- removed C200: 10u, Capacitor_SMD:C_0603_1608Metric, symbol New_Library_0:C_Small_edited
- removed C211: 1u, Capacitor_SMD:C_0201_0603Metric_Pad0.64x0.40mm_HandSolder, symbol New_Library_0:C_Small_edited
- removed L11: ???, Inductor_SMD:L_1008_2520Metric, symbol Device:L_Small
- removed R51, R52, R53, R54, R55, R56, R57, R58, R59, R60, R61, R62, R63, R64, R65, R66, R67, R68, R69, R70: (no value), PCM_Resistor_SMD_AKL:R_0402_1005Metric, symbol Device:R_Small
- removed U10, U12, U13, U9: AP2553W6-7, Package_TO_SOT_SMD:SOT-23-6_Handsoldering, symbol New_Library:AP2553W6-7
- removed U14, U15, U16, U17: (no value), Package_SON:USON-10_2.5x1.0mm_P0.5mm, symbol Power_Protection:TPD4E05U06DQA
- removed Y3: (no value), symbol Device:Crystal_GND24
- added C228: 1u, Capacitor_SMD:C_0201_0603Metric_Pad0.64x0.40mm_HandSolder, symbol New_Library_0:C_Small_edited
- added R218, R219, R220, R221, R235: 0R, PCM_Resistor_SMD_AKL:R_0402_1005Metric, symbol Device:R_Small
- added R222, R223, R224, R225: 15k, PCM_Resistor_SMD_AKL:R_0402_1005Metric, symbol Device:R_Small
- added R226, R227, R228, R229, R236, R237: 100k, PCM_Resistor_SMD_AKL:R_0402_1005Metric, symbol Device:R_Small
- added R230, R231, R232, R233: 2.2k, PCM_Resistor_SMD_AKL:R_0402_1005Metric, symbol Device:R_Small
- added R234: 6.2k, PCM_Resistor_SMD_AKL:R_0402_1005Metric, symbol Device:R_Small
- added U41, U43, U46, U47: AP2553W6-7, symbol New_Library:AP2553W6-7
- added U48, U49, U50, U51: TPD4E05U06DQAR, Package_SON:USON-10_2.5x1.0mm_P0.5mm, symbol Power_Protection:TPD4E05U06DQA
- added Y8: K3A120002010, Crystal:Crystal_SMD_3225-4Pin_3.2x2.5mm_HandSoldering, symbol Device:Crystal_GND24
- J3, J4: value USB3_A_Stacked -> UAA112C-84168-4H
- U11: value (none) -> RTS5411S-GR; LCSC Part (none) -> C5356838; Mouser Part (fill (type none)) -> (none)
Connections:
- net +1.2V_{HUB}: now also C198.1, C199.1, U11.52 (SWR_OUT); no longer C191.1, C192.1, C193.1, C194.1, U11.22 (DV33), U11.4 (DV33), U11.48 (DV33), U11.73 (DV33)
- net +3.3V_{HUB}: now also C228.1; no longer C198.1, C199.1, U11.52 (SWR_OUT)
- net CUSB_{HOST1}_SSRX1_N: now also U48.1 (D1+)
- net CUSB_{HOST1}_SSRX1_P: now also U48.2 (D1-)
- net CUSB_{HOST1}_SSTX1_N: now also U48.4 (D2+)
- net CUSB_{HOST1}_SSTX1_P: now also U48.5 (D2-)
- net CUSB_{HOST2}_SSRX1_N: now also U51.1 (D1+)
- net CUSB_{HOST2}_SSRX1_P: now also U51.2 (D1-)
- net CUSB_{HOST2}_SSTX1_N: now also U51.4 (D2+)
- net CUSB_{HOST2}_SSTX1_P: now also U51.5 (D2-)
- net CUSB_{HOST3}_SSRX1_N: now also U49.1 (D1+)
- net CUSB_{HOST3}_SSRX1_P: now also U49.2 (D1-)
- net CUSB_{HOST3}_SSTX1_N: now also U49.4 (D2+)
- net CUSB_{HOST3}_SSTX1_P: now also U49.5 (D2-)
- net CUSB_{HOST4}_SSRX1_N: now also U50.1 (D1+)
- net CUSB_{HOST4}_SSRX1_P: now also U50.2 (D1-)
- net CUSB_{HOST4}_SSTX1_N: now also U50.4 (D2+)
- net CUSB_{HOST4}_SSTX1_P: now also U50.5 (D2-)
- net Crystal_{HUB}_IN: now also Y8.1
- net Crystal_{HUB}_OUT: now also Y8.3
- net GND: now also C228.2, R218.2, R219.2, R220.2, R221.2, R222.2, R223.2, R224.2, R225.2, R226.2, R227.2, R228.2, R229.2, R234.2, R235.2, R237.2, U41.2 (GND), U43.2 (GND), U46.2 (GND), U47.2 (GND), U48.3 (GND), U48.8 (GND), U49.3 (GND), U49.8 (GND), U50.3 (GND), U50.8 (GND), U51.3 (GND), U51.8 (GND), Y8.2 (G), Y8.4 (G)
- net USB_{HOST}_PWREN_H: now also R230.2, R231.2, R232.2, R233.2
- net VCC5V0_SYS: now also R236.1, U41.1 (IN), U43.1 (IN), U46.1 (IN), U47.1 (IN)
- net Vbus_USB_{HOST1}: now also U41.6 (OUT)
- net Vbus_USB_{HOST2}: now also U43.6 (OUT)
- net Vbus_USB_{HOST3}: now also U46.6 (OUT)
- net Vbus_USB_{HOST4}: now also U47.6 (OUT)
- net at J4.SH (SHIELD): now also R220.1
- net at J3.SH (SHIELD): now also R218.1
- net at J3.SH (SHIELD): now also R219.1
- net at J4.SH (SHIELD): now also R221.1
- net at U11.1 (RREF): now also R234.1
- net at U11.2 (BPWR_DET): now also R236.2, R237.1
- net at U11.45 (SCS): now also R235.1
- new net: R223.1, U43.5 (ILIM)
- new net: R226.1, R230.1, U41.3 (EN)
- new net: R222.1, U41.5 (ILIM)
- new net: R227.1, R231.1, U43.3 (EN)
- new net: R228.1, R232.1, U46.3 (EN)
- new net: R224.1, U46.5 (ILIM)
- new net: R229.1, R233.1, U47.3 (EN)
- new net: R225.1, U47.5 (ILIM)
- new net DV33: C191.1, C192.1, C193.1, C194.1, U11.22 (DV33), U11.4 (DV33), U11.48 (DV33), U11.73 (DV33)
- no-connect marks 39 -> 40
Other:
- moved on the sheet: C191, C192, C193, C202, C203, C216, C217

Commit message: SBCv0.5
small update for Josa watch the final version
Parts:
- U41, U43, U46, U47: footprint (none) -> PCM_SparkFun-Semiconductor-Standard:SOT23-6-Tight
