File: usd_card.kicad_sch (KiCad schematic)
At the start: 19 parts, among them J11 Micro_SD_Card_Det1, U20 TPD4E05U06DQA, U21 TPD4E05U06DQA

Commit message: Add files via upload
Parts:
- removed C118: 10u, Capacitor_SMD:C_0402_1005Metric, symbol New_Library_0:C_Small_edited
- removed C119: 100n, Capacitor_SMD:C_0201_0603Metric_Pad0.64x0.40mm_HandSolder, symbol New_Library_0:C_Small_edited
- added C376: 22u, Capacitor_SMD:C_0603_1608Metric, symbol New_Library_0:C_Small_edited
- added C377, C378: 1u, Capacitor_SMD:C_0402_1005Metric_Pad0.74x0.62mm_HandSolder, symbol New_Library_0:C_Small_edited
- added D25: SMBJ5.0CA, PCM_Diode_SMD_AKL:D_SMB_TVS, symbol PCM_Diode_TVS_AKL:SMBJ5.0CA
- added R172: 10k, PCM_Resistor_SMD_AKL:R_0402_1005Metric, symbol Device:R_Small
- added R173: 100k, PCM_Resistor_SMD_AKL:R_0402_1005Metric, symbol Device:R_Small
- added R174: 2.2k, PCM_Resistor_SMD_AKL:R_0402_1005Metric, symbol Device:R_Small
- added U35: AP2553W6-7, symbol New_Library:AP2553W6-7
- renumbered J11 to J9, R62 to R120, R63 to R121, R64 to R122, R65 to R123, R66 to R124, R67 to R125, R68 to R126, R69 to R127, R70 to R128, R71 to R129, R72 to R130, R73 to R131, R74 to R132, R75 to R133, U20 to U25, U21 to U26
Connections:
- net GND: now also C376.2, C377.2, C378.2, D25.1 (K), R172.2, R173.2, U35.2 (GND)
- net +3.3V renamed VCC3V3_uSD
- net VCC3V3_uSD: now also C376.1, C378.1, D25.2 (A), U35.6 (OUT)
- new net: R173.1, R174.1, U35.3 (EN)
- new net: R172.1, U35.5 (ILIM)
- new net VCC_3V3_S0: C377.1, U35.1 (IN)
- new net uSD_PWREN_H: R174.2
- no-connect marks 9 -> 10
Other:
- moved on the sheet: J9, R120, R121, R122, R123, R124, R125, R126, R127, R128, R129, R130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

Commit message: SBC Board V0.2
The SBC schematics before footprint and part number check
Parts:
- renumbered C377 to C342, C378 to C343, C376 to C344, D25 to D16, J9 to J8, R174 to R120, R172 to R121, R173 to R122, R120 to R123, R121 to R124, R122 to R125, R123 to R126, R124 to R127, R125 to R128, R126 to R129, R127 to R130, R128 to R131, R129 to R132, R130 to R133, R131 to R134, R132 to R135, R133 to R136, U35 to U27, U25 to U28, U26 to U29

Commit message: SBCv0.3
there is no big thing update just some LCSC & Mouser parts
and Big problem deleted alot of component values (:
Parts:
- C342, C343: footprint Capacitor_SMD:C_0402_1005Metric_Pad0.74x0.62mm_HandSolder -> Capacitor_SMD:C_0201_0603Metric_Pad0.64x0.40mm_HandSolder; LCSC Part (none) -> C5209398; Mouser Part (none) -> CL03A105KP3NSNC
- C344: LCSC Part (none) -> C86295; Mouser Part (none) -> CL10A226MP8NUNE
- D16: LCSC Part (none) -> C113975; Mouser Part (none) -> 581-SMBJ5.0CA
- J8: value Micro_SD_Card_Det1 -> TF PUSH; footprint Connector_Card:microSD_HC_Molex_104031-0811 -> Datasheet_Footprints:TF-PUSH_C393941; LCSC Part (none) -> C393941
- R120: value 2.2k -> (none); LCSC Part (none) -> (do_not_autoplace no)
- R121: LCSC Part (none) -> (at 0 0 0)
- R122: value 100k -> (none); LCSC Part (none) -> (show_name no)
- R123, R124, R125, R126, R127, R128: value 4.7k -> (none); LCSC Part (none) -> (at 0 0 0)
- R129: value 4.7k -> (none); LCSC Part (none) -> (show_name no)
- R130, R131, R132, R133, R134, R135, R136: value 22R -> (none); LCSC Part (none) -> (do_not_autoplace no)
- U27: footprint (none) -> Package_TO_SOT_SMD:SOT-23-6_Handsoldering; LCSC Part (none) -> C212302; Mouser Part (none) -> 621-AP2553W6-7
- U28, U29: value TPD4E05U06DQA -> (none); Mouser Part (none) -> )

Commit message: SBCv0.4
add LCSC & Mouser parts 
and solve the deleted value in the past version
Parts:
- R120: value (none) -> 2.2k; LCSC Part (do_not_autoplace no) -> C114762; Mouser Part (none) -> 603-RC0402FR-072K2L
- R121: LCSC Part (at 0 0 0) -> C60490; Mouser Part (none) -> 603-RC0402FR-0710KL
- R122: value (none) -> 100k; LCSC Part (show_name no) -> C60491; Mouser Part (none) -> 603-RC0402FR-07100KL
- R123, R124, R125, R126, R127, R128: value (none) -> 4.7k; LCSC Part (at 0 0 0) -> C105871; Mouser Part (none) -> 603-RC0402FR-074K7L
- R129: value (none) -> 4.7k; LCSC Part (show_name no) -> C105871; Mouser Part (none) -> 603-RC0402FR-074K7L
- R130, R131, R132, R133, R134, R135, R136: value (none) -> 22R; LCSC Part (do_not_autoplace no) -> C114765; Mouser Part (none) -> 603-RC0402FR-0722RL
- U28, U29: value (none) -> TPD4E05U06DQAR; LCSC Part (none) -> C138714; Mouser Part ) -> 595-TPD4E05U06DQAR
