File: power.kicad_sch (KiCad schematic)
At the start: 92 parts, among them SW1 SW_Push, U26 RK806S-5

Commit message: Add files via upload
Parts:
- removed C173, C174: 2.2u, Capacitor_SMD:C_0402_1005Metric, symbol New_Library_0:C_Small_edited
- removed C226, C227: 22u, Capacitor_SMD:C_0603_1608Metric, symbol New_Library_0:C_Small_edited
- removed C228: 47u, Capacitor_SMD:C_0805_2012Metric, symbol New_Library_0:C_Small_edited
- removed L14: FTC252012SR24MBCA, Inductor_SMD:L_1008_2520Metric, symbol Device:L_Small
- removed R102, R93, R96: 100k, PCM_Resistor_SMD_AKL:R_0402_1005Metric, symbol Device:R_Small
- added C11, C16, C22, C363: 2.2u, Capacitor_SMD:C_0402_1005Metric, symbol New_Library_0:C_Small_edited
- added C57, C58: 22u, Capacitor_SMD:C_0603_1608Metric, symbol New_Library_0:C_Small_edited
- added C59: 47u, Capacitor_SMD:C_0805_2012Metric, symbol New_Library_0:C_Small_edited
- added L10: FTC252012SR24MBCA, Inductor_SMD:L_1008_2520Metric, symbol Device:L_Small
- added R11, R5, R9: 100k, PCM_Resistor_SMD_AKL:R_0402_1005Metric, symbol Device:R_Small
- C30: renamed from C214; value 100n -> 1u
- R10: renamed from R101; symbol Device:R_US -> Device:R_Small
- R3: renamed from R92; symbol Device:R_US -> Device:R_Small
- R8: renamed from R94; symbol Device:R_US -> Device:R_Small
- renumbered C177 to C1, C189 to C10, C191 to C12, C192 to C13, C193 to C14, C194 to C15, C196 to C17, C197 to C18, C198 to C19, C178 to C2, C199 to C20, C181 to C21, C208 to C23, C209 to C24, C200 to C25, C201 to C26, C202 to C27, C203 to C28, C175 to C29, C179 to C3, C215 to C31, C216 to C32, C204 to C33, C190 to C34, C176 to C35, C205 to C36, C206 to C37, C207 to C38, C182 to C39, C180 to C4, C210 to C40, C211 to C41, C212 to C42, C213 to C43, C183 to C44, C217 to C45, C218 to C46, C219 to C47, C220 to C48, C195 to C49, C171 to C5, C184 to C50, C221 to C51, C222 to C52, C223 to C53, C224 to C54, C185 to C55, C225 to C56, C172 to C6, C186 to C7, C187 to C8, C188 to C9, D13 to D1, L5 to L1, L6 to L2, L7 to L3, L8 to L4, L9 to L5, L10 to L6, L11 to L7, L12 to L8, L13 to L9, R95 to R1, R97 to R2, R98 to R4, R99 to R6, R100 to R7, U26 to U1
Connections:
- net PMIC_PWRON is gone; now on net PMIC_PWRON_L: D1.2 (A), SW1.1
- net +5v: no longer C21.1, C23.1, C24.1, C49.1, U1.21 (VCCA), U1.64 (VCC12), U1.9 (VCC14)
- net GND: now also R7.2, U1.31 (FB6), U1.47 (FB5), U1.66 (FB9), C11.2, C16.2, C22.2, C363.2, R11.2, R5.2, R9.2
- net VDDA_DDR_PLL_S0: now also C39.1
- net VDD_DDR_S0: now also C57.1, C58.1, C59.1, L10.2
- net at R6.1: now also C31.1, C32.1, U1.4 (PWRON)
- net PMIC_PWRON_L: now reaches R6.2
- net at R8.2: now also R9.1; no longer U1.31 (FB6)
- net VCCA1V8_PLDO2_S0: now reaches U1.58 (PLDO2)
- net VCCA1V8_PLDO2_S0: now also C11.1
- net at U1.26 (SW10): now also L10.1
- net VCCA1V8_PLDO6_S3: now reaches U1.20 (VCCIO)
- net VCCA1V8_PLDO6_S3: now also C363.1
- net at C30.1, U1.32 (VDC): now also R2.2, R7.1
- net at U1.40 (~{RESETB}): now also R4.1
- net RESET_L: now reaches R4.2
- net VCC5V0_SYS: now reaches R2.1
- net VCC5V0_SYS: now also C21.1, C23.1, C24.1, U1.21 (VCCA), U1.64 (VCC12)
- net at R3.2: now also R5.1; no longer U1.47 (FB5)
- net at R10.2: now also R11.1; no longer U1.66 (FB9)
- net +0.75_{HDMI}v renamed VDDA0V75_HDMI_S0
- net VDDA0V75_HDMI_S0: now also C44.1; no longer C35.1
- removed net +0.75v: C39.1, C44.1, U1.14 (NLDO1), U1.8 (NLDO5)
- net +0.85v renamed VDDA_0V85_S0
- net +1.2v renamed VDDA_1V2_S0
- net VDDA_1V2_S0: now also C16.1
- net +1.8v renamed VCCA_1V8_S0
- net VCCA_1V8_S0: no longer R1.1
- net +1.8v_S3 renamed VCC_1V8_S3
- net VCC_1V8_S3: now also R1.1
- net +2v renamed VCC_2V0_PLDO_S3
- net VCC_2V0_PLDO_S3: now also C49.1, U1.9 (VCC14)
- net +3.3v renamed VCCA_3V3_S0
- net VCCA_3V3_S0: now also C22.1
- net +3.3v_S0 renamed VCC_3V3_S0
- net +DDR_PLLv renamed VDDA_0V75_S0
- net VDDA_0V75_S0: now also U1.8 (NLDO5)
- net +SD Cardv renamed VCCIO_SD_S0
- net PMIC_CLK renamed SPI2_CLK_M0
- net PMIC_EXT_EN renamed PMIC_EXT_EN_OUT
- net PMIC_INT renamed PMIC_INT_L
- net PMIC_MISO renamed SPI2_MISO_M0
- net PMIC_MOSI renamed SPI2_MOSI_M0
- net PMIC_PWRCRTL1 renamed PMIC_PWR_CTRL1
- net PMIC_PWRCRTL2 renamed PMIC_PWR_CTRL2
- new net: C57.2, C58.2, C59.2
- new net VDD_0V75_S3: C35.1, U1.14 (NLDO1)
- no-connect marks 7 -> 5
Other:
- note added: "1.05V NOM"
- moved on the sheet: C1, C10, C12, C13, C14, C15, C17, C18, C19, C2, C20, C21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

Commit message: SBC Board V0.2
The SBC schematics before footprint and part number check
Parts:
- added C45, C46, C47, C48, C50, C51: 2.2u, Capacitor_SMD:C_0402_1005Metric, symbol New_Library_0:C_Small_edited
- added U2: MAX14713EWL+T, Datasheet_Footprints:WLP-15_MAX14713, symbol Datasheet_Symbols:MAX14713EWL+T
- renumbered C9 to C10, C10 to C11, C23 to C12, C24 to C13, C11 to C14, C30 to C15, C12 to C16, C13 to C17, C14 to C18, C15 to C19, C16 to C20, C31 to C21, C32 to C22, C17 to C23, C18 to C24, C19 to C25, C20 to C26, C21 to C27, C22 to C28, C25 to C29, C26 to C30, C27 to C31, C28 to C32, C29 to C33, C33 to C34, C34 to C35, C35 to C36, C36 to C37, C37 to C38, C38 to C39, C39 to C40, C40 to C41, C41 to C42, C42 to C43, C43 to C44, C44 to C49, C45 to C52, C46 to C53, C47 to C54, C48 to C55, C49 to C56, C50 to C57, C51 to C58, C52 to C59, C53 to C60, C54 to C61, C55 to C62, C56 to C63, C57 to C64, C58 to C65, C59 to C66, C363 to C7, C7 to C8, C8 to C9, R4 to R3, R6 to R4, R7 to R5, R3 to R6, R5 to R7
Connections:
- net GND: now also C45.2, C46.2, C47.2, C48.2, C50.2, C51.2, U2.C3 (GND)
- net VCC5V0_SYS: now also C47.1, C48.1, U2.A2 (OUT), U2.A3 (OUT), U2.A4 (OUT), U2.B3 (OUT)
- new net IN1: C45.1, C46.1, U2.B1 (IN1), U2.B2 (IN1), U2.C1 (IN1), U2.C2 (IN1)
- new net IN2: C50.1, C51.1, U2.B4 (IN2), U2.B5 (IN2), U2.C4 (IN2), U2.C5 (IN2)
- new net TYPEC_PWR-IN_SEL1: U2.A1 (~{EN1})
- new net TYPEC_PWR-IN_SEL2: U2.A5 (~{EN2})
Other:
- moved on the sheet: C1, C10, C11, C12, C13, C14, C15, C16, C17, C18, C19, C2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

Commit message: SBCv0.3
there is no big thing update just some LCSC & Mouser parts
and Big problem deleted alot of component values (:
Parts:
- C1, C10, C16, C17, C18, C2, C23, C24, C25, C29, C3, C30, C31, C34, C37, C38, C41, C42, C43, C52, C53, C54, C58, C59, C60, C63, C64, C65, C8, C9: LCSC Part (none) -> C86295; Mouser Part (none) -> CL10A226MP8NUNE
- C11, C19, C26, C32, C39, C4, C44, C55, C61, C66: LCSC Part (none) -> C16780; Mouser Part (none) -> 187-CL21A476MQYNNNE
- C12, C13, C14, C20, C27, C28, C33, C35, C36, C40, C45, C46, C47, C48, C49, C5, C50, C51, C56, C57, C6, C62, C7: LCSC Part (none) -> C170151; Mouser Part (none) -> 187-CL05A225KO5NQNC
- C15: LCSC Part (none) -> C5209398; Mouser Part (none) -> CL03A105KP3NSNC
- C21, C22: LCSC Part (none) -> C87461; Mouser Part (none) -> 187-CL03B103KP3NNNC
- D1: LCSC Part (none) -> C113975; Mouser Part (none) -> 581-SMBJ5.0CA
- L1, L10, L2, L3, L4, L5, L6, L7, L8, L9: LCSC Part C5832366 -> (at 0 0 0)
- NT1, NT10, NT2, NT3, NT4, NT5, NT6, NT7, NT8, NT9: LCSC Part (none) -> )
- R1: LCSC Part (none) -> (at 0 0 0)
- R10: value 110k -> (none); Mouser Part (none) -> (font (size 1.27 1.27))
- R11, R2, R5, R7, R9: value 100k -> (none); LCSC Part (none) -> (show_name no)
- R3, R4: value 22R -> (none); LCSC Part (none) -> (do_not_autoplace no)
- R6: value 49.9k -> (none); LCSC Part (none) -> (hide yes)
- R8: value 2k -> (none); LCSC Part (none) -> (effects
- SW1: value SW_Push -> (none); Mouser Part (none) -> (pts
- U1: value RK806S-5 -> (none); LCSC Part C49174044 -> (none); Mouser Part (none) -> (fill (type none))
- U2: value MAX14713EWL+T -> (none); LCSC Part C2150266 -> )
Connections:
- net VCC5V0_SYS is gone; now on net VCC1: C12.1, C13.1, C27.1, C47.1, C48.1, R2.1, U1.21 (VCCA), U1.64 (VCC12), U2.A2 (OUT), U2.A3 (OUT), U2.A4 (OUT), U2.B3 (OUT)
- net +5v renamed VCC1

Commit message: SBCv0.4
add LCSC & Mouser parts 
and solve the deleted value in the past version
Parts:
- removed R10, R11, R2, R3, R4, R9: (no value), PCM_Resistor_SMD_AKL:R_0402_1005Metric, symbol Device:R_Small
- removed U1: (no value), Package_DFN_QFN:QFN-68-1EP_8x8mm_P0.4mm_EP6.4x6.4mm_ThermalVias, symbol Datasheet_Symbols:RK806S-5
- removed U2: (no value), Datasheet_Footprints:WLP-15_MAX14713, symbol Datasheet_Symbols:MAX14713EWL+T
- added R190: 49.9k, PCM_Resistor_SMD_AKL:R_0402_1005Metric, symbol Device:R_Small
- added R191, R193, R195: 100k, PCM_Resistor_SMD_AKL:R_0402_1005Metric, symbol Device:R_Small
- added R192: 2k, PCM_Resistor_SMD_AKL:R_0402_1005Metric, symbol Device:R_Small
- added R194: 110k, PCM_Resistor_SMD_AKL:R_0402_1005Metric, symbol Device:R_Small
- added U10: MAX14713EWL+T, Datasheet_Footprints:WLP-15_MAX14713, symbol Datasheet_Symbols:MAX14713EWL+T
- added U9: RK806S-5, Package_DFN_QFN:QFN-68-1EP_8x8mm_P0.4mm_EP6.4x6.4mm_ThermalVias, symbol Datasheet_Symbols:RK806S-5
- L1, L10, L2, L3, L4, L5, L6, L7, L8, L9: LCSC Part (at 0 0 0) -> C5832366
- NT1, NT10, NT2, NT3, NT4, NT5, NT6, NT7, NT8, NT9: LCSC Part ) -> (none)
- R1: LCSC Part (at 0 0 0) -> C60490; Mouser Part (none) -> 603-RC0402FR-0710KL
- R5: value (none) -> 22R; LCSC Part (show_name no) -> C114765; Mouser Part (none) -> 603-RC0402FR-0722RL
- R6: value (none) -> 100k; LCSC Part (hide yes) -> C60491; Mouser Part (none) -> 603-RC0402FR-07100KL
- R7: value (none) -> 100k; LCSC Part (show_name no) -> C60491; Mouser Part (none) -> 603-RC0402FR-07100KL
- R8: value (none) -> 22R; LCSC Part (effects -> C114765; Mouser Part (none) -> 603-RC0402FR-0722RL
- SW1: value (none) -> SKRTLAE010; footprint Button_Switch_SMD:SW_Push_1P1T_NO_CK_PTS125Sx85SMTR -> easyeda2kicad:SKRTLAE010; LCSC Part (none) -> C110293; Mouser Part (pts -> (none)
Connections:
- net GND: now also R191.2, R193.2, R195.2, U10.C3 (GND), U9.31 (FB6), U9.47 (FB5), U9.66 (FB9), U9.69 (EP); no longer R5.2
- net IN1: now also U10.B1 (IN1), U10.B2 (IN1), U10.C1 (IN1), U10.C2 (IN1)
- net IN2: now also U10.B4 (IN2), U10.B5 (IN2), U10.C4 (IN2), U10.C5 (IN2)
- net PMIC_EXT_EN_OUT: now also U9.39 (EXT_EN)
- net PMIC_INT_L: now also U9.19 (INT)
- net PMIC_PWRON_L: now also R8.2
- net PMIC_PWR_CTRL1: now also U9.62 (PWRCRTL1)
- net PMIC_PWR_CTRL2: now also U9.61 (PWRCRTL2)
- net RESET_L: now also R5.2
- net SPI2_CLK_M0: now also U9.17 (CLK/SCL)
- net SPI2_MISO_M0: now also U9.16 (MISO/PWRCRTL3)
- net SPI2_MOSI_M0: now also U9.15 (MOSI/SDA)
- net TYPEC_PWR-IN_SEL1: now also U10.A1 (~{EN1})
- net TYPEC_PWR-IN_SEL2: now also U10.A5 (~{EN2})
- net VCC1: now also R6.1, U10.A2 (OUT), U10.A3 (OUT), U10.A4 (OUT), U10.B3 (OUT), U9.1 (VCC9), U9.21 (VCCA), U9.22 (VCC4), U9.27 (VCC10), U9.28 (VCC6), U9.33 (VCC2), U9.34 (VCC2), U9.43 (VCC7), U9.44 (VCC5), U9.52 (VCC1), U9.53 (VCC1), U9.54 (VCC3), U9.64 (VCC12), U9.7 (VCC8)
- net VCCA1V8_PLDO2_S0: now also U9.58 (PLDO2)
- net VCCA1V8_PLDO6_S3: now also U9.20 (VCCIO)
- net VCCA_1V8_S0: now also U9.60 (PLDO1)
- net VCCA_3V3_S0: now also U9.63 (PLDO4)
- net VCCIO_SD_S0: now also U9.65 (PLDO5)
- net VCC_2V0_PLDO_S3: now also U9.13 (VCC13), U9.59 (VCC11), U9.9 (VCC14)
- net VDD2_DDR_S3: now also R194.1
- net VDDA0V75_HDMI_S0: now also U9.11 (NLDO3)
- net VDDA_0V75_S0: now also U9.8 (NLDO5)
- net VDDA_0V85_S0: now also U9.10 (NLDO4)
- net VDDA_1V2_S0: now also U9.57 (PLDO3)
- net VDDA_DDR_PLL_S0: now also U9.12 (NLDO2)
- net VDDQ_DDR_S0: now also R192.1; no longer R8.1
- net VDD_0V75_S3: now also U9.14 (NLDO1)
- net VDD_GPU_S0: now also R190.1; no longer R6.1
- net at L4.1: now also U9.23 (SW4)
- net at L6.1: now also U9.29 (SW6)
- net at NT10.1: now also U9.25 (VOUT10)
- net at C21.1, C22.1: now also R8.1, U9.4 (PWRON)
- net at L9.1: now also U9.68 (SW9)
- net at NT4.1: now also U9.24 (VOUT4)
- net at L3.1: now also U9.55 (SW3)
- net at NT9.1: now also U9.67 (VOUT9)
- net at L5.1: now also U9.45 (SW5)
- net at C15.1: now also R6.2, R7.1, U9.32 (VDC); no longer R5.1
- net at NT6.1: now also U9.30 (VOUT6)
- net at NT7.1: now also U9.41 (VOUT7)
- net at L1.1: now also U9.50 (SW1), U9.51 (SW1)
- net at L7.1: now also U9.42 (SW7)
- net at L8.1: now also U9.6 (SW8)
- net at L10.1: now also U9.26 (SW10)
- net at L2.1: now also U9.35 (SW2), U9.36 (SW2)
- net at NT2.1: now also U9.37 (VOUT2)
- net at NT5.1: now also U9.46 (VOUT5)
- net at NT1.1: now also U9.49 (VOUT1)
- net at NT8.1: now also U9.5 (VOUT8)
- net at NT3.1: now also U9.56 (VOUT3)
- new net: R194.2, R195.1
- new net: R192.2, R193.1
- new net: R190.2, R191.1
- new net: R5.1, U9.40 (~{RESETB})

Commit message: Release v2: replace main with RK3576 SBCv2, archive v1 to branch archive/v1
- main now shows only v2 (RK3576 SBCv2.kicad_pro)
- v1 preserved in branch archive/v1 + tag v1.0
- Add .gitignore for KiCad (*.bak, *.lck, .history/)
- Update README with version switcher
- Cleaned: dropped 141M .history, Resources ref PDF, *.bak/*.lck
Parts:
- removed C1, C10, C16, C17, C18, C2, C23, C24, C25, C29, C3, C30, C31, C34, C37, C38, C41, C42, C43, C52, C53, C54, C58, C59, C60, C63, C64, C65, C8, C9: 22u, Capacitor_SMD:C_0603_1608Metric, symbol New_Library_0:C_Small_edited
- removed C11, C19, C26, C32, C39, C4, C44, C55, C61, C66: 47u, Capacitor_SMD:C_0805_2012Metric, symbol New_Library_0:C_Small_edited
- removed C12, C13, C14, C20, C27, C28, C33, C35, C36, C40, C45, C46, C47, C48, C49, C5, C50, C51, C56, C57, C6, C62, C7: 2.2u, Capacitor_SMD:C_0402_1005Metric, symbol New_Library_0:C_Small_edited
- removed C15: 1u, Capacitor_SMD:C_0201_0603Metric_Pad0.64x0.40mm_HandSolder, symbol New_Library_0:C_Small_edited
- removed C21, C22: 10n, Capacitor_SMD:C_0201_0603Metric_Pad0.64x0.40mm_HandSolder, symbol New_Library_0:C_Small_edited
- removed D1: SMBJ5.0CA, PCM_Diode_SMD_AKL:D_SMB_TVS, symbol PCM_Diode_TVS_AKL:SMBJ5.0CA
- removed L1, L10, L2, L3, L4, L5, L6, L7, L8, L9: FTC252012SR24MBCA, Inductor_SMD:L_1008_2520Metric, symbol Device:L_Small
- removed NT1, NT10, NT2, NT3, NT4, NT5, NT6, NT7, NT8, NT9: NetTie_2, NetTie:NetTie-2_SMD_Pad0.5mm, symbol Device:NetTie_2
- removed R1: 10k, PCM_Resistor_SMD_AKL:R_0402_1005Metric, symbol Device:R_Small
- removed R190: 49.9k, PCM_Resistor_SMD_AKL:R_0402_1005Metric, symbol Device:R_Small
- removed R191, R193, R195, R6, R7: 100k, PCM_Resistor_SMD_AKL:R_0402_1005Metric, symbol Device:R_Small
- removed R192: 2k, PCM_Resistor_SMD_AKL:R_0402_1005Metric, symbol Device:R_Small
- removed R194: 110k, PCM_Resistor_SMD_AKL:R_0402_1005Metric, symbol Device:R_Small
- removed R5, R8: 22R, PCM_Resistor_SMD_AKL:R_0402_1005Metric, symbol Device:R_Small
- removed SW1: SKRTLAE010, easyeda2kicad:SKRTLAE010, symbol Switch:SW_Push
- removed U10: MAX14713EWL+T, Datasheet_Footprints:WLP-15_MAX14713, symbol Datasheet_Symbols:MAX14713EWL+T
- removed U9: RK806S-5, Package_DFN_QFN:QFN-68-1EP_8x8mm_P0.4mm_EP6.4x6.4mm_ThermalVias, symbol Datasheet_Symbols:RK806S-5
Connections:
- no-connect marks 5 -> 0
Other:
- note removed: "1.05V NOM"
