File: 40pin_GPIO.kicad_sch (KiCad schematic)
At the start: 21 parts, among them J16 B3B-XH-A(LF)(SN), J17 B-2100S40P-B110, U33 AP2553W6-7, U34 AP2553W6-7

Commit message: Replace v2 with updated RK3576_SBCv2 (Copy) Oct 2
- Update 18 sheets to Oct 2 15:37 local versions
- Keep cleaned layout: exclude .history/, Resources/, *.bak, *.lck,
  project.kicad_dru, .hs_rules.json, lowercase dup placeholders
  (fixtures/power), empty orphans (digital, mechanical, output,
  USBC_MCU, eMMC_UFS)
- Preserve LICENSE, README.md, .gitignore
Parts:
- R117: LCSC Part C106231 -> C60490; Mouser Part 603-RC0402FR-070RL -> 603-RC0402FR-0710KL
- R198, R199: LCSC Part C114761 -> C60490; Mouser Part 603-RC0402FR-0715KL -> 603-RC0402FR-0710KL
- R200, R201: LCSC Part C60491 -> C60490; Mouser Part 603-RC0402FR-07100KL -> 603-RC0402FR-0710KL
Connections:
- net 40GPIOs_GPIO(3_A0)_UART(3)_RX-M1: no longer names the net of J17.24 (~{CE0}_SPI0/GPIO08)
- net 40GPIOs_GPIO(3_A1)_UART(3)_RX-M1: no longer names the net of J17.26 (~{CE1}_SPI0/GPIO07)
- net 40GPIOs_GPIO(3_B2)_I2C(8)_SDA-M3 renamed I2C2_SDA_M0_CC_RTC_EEPROM
- net 40GPIOs_GPIO(3_B3)_I2C(8)_SCL-M3 renamed I2C2_SCL_M0_CC_RTC_EEPROM
- net 40GPIOs_GPIO(3_C2)_I2C(5)_SCL-M3 renamed 40GPIOs_GPIO(3_C4)_I2C(5)_SCL-M3
- net 40GPIOs_GPIO(3_C4)_I2C(9)_SCL-M3 renamed 40GPIOs_GPIO(3_C2)_I2C(9)_SCL-M3
- net 40GPIOs_GPIO(3_D1)_I3C(1)_SDA_PU-M2: no longer names the net of J17.7 (GPCLK0/GPIO04)
- net 40GPIOs_GPIO(3_D2)_I3C(1)_SDA-M2: no longer names the net of J17.29 (GPCLK1/GPIO05)
- net 40GPIOs_GPIO(3_D3)_I3C(1)_SCL-M2: no longer names the net of J17.31 (GPCLK2/GPIO06)
- no-connect marks 2 -> 7

Commit message: Relink hierarchical root: 18 sheets into RK3576 SBCv2 top level
Root was empty (no sheet boxes); all subsheets orphaned.
Rebuilt A1 top level linking RK3576, LPDDR5, Power, Ethernet,
HDMI, MIPI, PCIe, USB-A/C, Wireless, RTC, uSD, GPIO, OLED,
RP2350A, Connectors, Fixtures, DC_Power. block_diagrame kept
docs-only (unlinked, avoids double-instantiation). Lowercase
stub duplicates excluded. ERC: 1388 -> 770 violations.
Parts:
- renumbered C378 to C264, C379 to C265, C380 to C266, C381 to C267, D21 to D15, D22 to D16, D23 to D17, D24 to D18, J16 to J18, J17 to J19, R137 to R187, R117 to R188, R176 to R189, R198 to R190, R199 to R191, R200 to R192, R201 to R193, R202 to R194, R203 to R195, U34 to U35, U33 to U36

Commit message: block diagrame with Hierarchical labels and NVMe SSD footprint
Parts:
- added D31, D32, D33, D34, D35, D36, D37, D38, D39, D40, D41, D42, D43, D44, D45, D46, D47, D48, D49, D50, D51, D52, D54, D56: PESD5V0S1BA, PCM_Diode_SMD_AKL:D_SOD-323_TVS, symbol PCM_Diode_TVS_AKL:PESD5V0S1BA
- J18: renamed from J19; footprint #kicad Library:40-pin GPIO Header for Raspberry Pi -> Connector_PinSocket_2.54mm:PinSocket_2x20_P2.54mm_Horizontal
- renumbered D17 to D53, D18 to D55, D15 to D57, D16 to D58, J18 to J19, R187 to R196
Connections:
- net GND: now also D31.1 (K), D32.1 (K), D33.1 (K), D34.1 (K), D35.1 (K), D36.1 (K), D37.1 (K), D38.1 (K), D39.1 (K), D40.1 (K), D41.1 (K), D42.1 (K), D43.1 (K), D44.1 (K), D45.1 (K), D46.1 (K), D47.1 (K), D48.1 (K), D49.1 (K), D50.1 (K), D51.1 (K), D52.1 (K), D54.1 (K), D56.1 (K)
- net I2C2_SCL_M0_CC_RTC_EEPROM: now also D49.2 (A)
- net I2C2_SDA_M0_CC_RTC_EEPROM: now also D47.2 (A)
- net VCC_{GPIO}_3V3_S0: now also D46.2 (A)
- net VCC_{GPIO}_5V0_S0: now also D44.2 (A)
- net 40GPIOs_GPIO(3_A6)_UART(1)_RX-M2 renamed 40GPIOs.GPIO(3_A6)_UART(1)_RX-M2
- net 40GPIOs.GPIO(3_A6)_UART(1)_RX-M2: now also D43.2 (A)
- net 40GPIOs_GPIO(3_A7)_UART(1)_TX-M2 renamed 40GPIOs.GPIO(3_A7)_UART(1)_TX-M2
- net 40GPIOs.GPIO(3_A7)_UART(1)_TX-M2: now also D45.2 (A)
- net 40GPIOs_GPIO(3_B0)_UART(10)_RX-M0 renamed 40GPIOs.GPIO(3_B0)_UART(10)_RX-M0
- net 40GPIOs.GPIO(3_B0)_UART(10)_RX-M0: now also D38.2 (A)
- net 40GPIOs_GPIO(3_B1)_UART(10)_TX-M0 renamed 40GPIOs.GPIO(3_B1)_UART(10)_TX-M0
- net 40GPIOs.GPIO(3_B1)_UART(10)_TX-M0: now also D36.2 (A)
- net 40GPIOs_GPIO(3_B4)_PWM(1)_CH4-M3 renamed 40GPIOs.GPIO(3_B4)_PWM(1)_CH4-M3
- net 40GPIOs.GPIO(3_B4)_PWM(1)_CH4-M3: now also D39.2 (A)
- net 40GPIOs_GPIO(3_B5)_PWM(1)_CH5-M3 renamed 40GPIOs.GPIO(3_B5)_PWM(1)_CH5-M3
- net 40GPIOs.GPIO(3_B5)_PWM(1)_CH5-M3: now also D40.2 (A)
- net 40GPIOs_GPIO(3_B6)_PWM(0)_CH1-M3 renamed 40GPIOs.GPIO(3_B6)_PWM(0)_CH1-M3
- net 40GPIOs.GPIO(3_B6)_PWM(0)_CH1-M3: now also D42.2 (A)
- net 40GPIOs_GPIO(3_B7)_UART(2)_RX-M2 renamed 40GPIOs.GPIO(3_B7)_UART(2)_RX-M2
- net 40GPIOs.GPIO(3_B7)_UART(2)_RX-M2: now also D37.2 (A)
- net 40GPIOs_GPIO(3_C0)_UART(2)_TX-M2 renamed 40GPIOs.GPIO(3_C0)_UART(2)_TX-M2
- net 40GPIOs.GPIO(3_C0)_UART(2)_TX-M2: now also D35.2 (A)
- net 40GPIOs_GPIO(3_C1)_I2C(5)_SDA-M3 renamed 40GPIOs.GPIO(3_C1)_I2C(5)_SDA-M3
- net 40GPIOs.GPIO(3_C1)_I2C(5)_SDA-M3: now also D33.2 (A)
- net 40GPIOs_GPIO(3_C2)_I2C(9)_SCL-M3 renamed 40GPIOs.GPIO(3_C2)_I2C(9)_SCL-M3
- net 40GPIOs.GPIO(3_C2)_I2C(9)_SCL-M3: now also D54.2 (A)
- net 40GPIOs_GPIO(3_C3)_I2C(9)_SDA-M3 renamed 40GPIOs.GPIO(3_C3)_I2C(9)_SDA-M3
- net 40GPIOs.GPIO(3_C3)_I2C(9)_SDA-M3: now also D51.2 (A)
- net 40GPIOs_GPIO(3_C4)_I2C(5)_SCL-M3 renamed 40GPIOs.GPIO(3_C4)_I2C(5)_SCL-M3
- net 40GPIOs.GPIO(3_C4)_I2C(5)_SCL-M3: now also D31.2 (A)
- net 40GPIOs_GPIO(3_C5)_PWM(2)_CH2-M3 renamed 40GPIOs.GPIO(3_C5)_PWM(2)_CH2-M3
- net 40GPIOs.GPIO(3_C5)_PWM(2)_CH2-M3: now also D41.2 (A)
- net 40GPIOs_GPIO(3_C6) renamed 40GPIOs.GPIO(3_C6)
- net 40GPIOs.GPIO(3_C6): now also D34.2 (A)
- net 40GPIOs_GPIO(3_C7) renamed 40GPIOs.GPIO(3_C7)
- net 40GPIOs.GPIO(3_C7): now also D32.2 (A)
- net SPI1_{MCU}_CS renamed SPI1_{MCU}.CS
- net SPI1_{MCU}.CS: now also D48.2 (A)
- net SPI1_{MCU}_SCK renamed SPI1_{MCU}.SCK
- net SPI1_{MCU}.SCK: now also D56.2 (A)
- net SPI1_{MCU}_SDI renamed SPI1_{MCU}.SDI
- net SPI1_{MCU}.SDI: now also D52.2 (A)
- net SPI1_{MCU}_SDO renamed SPI1_{MCU}.SDO
- net SPI1_{MCU}.SDO: now also D50.2 (A)
Other:
- moved on the sheet: D57, D58, J19, R196
