File: Ethernet.kicad_sch (KiCad schematic)
At the start: 100 parts, among them J10 LPJG0926HENL, J12 POE Connector, J6 LPJG0926HENL, J8 POE Connector, U25 RTL8211F-CG, U26 RTL8211F-CG, Y4 SX32Y025000BC1T001, Y6 SX32Y025000BC1T001

Commit message: Replace v2 with updated RK3576_SBCv2 (Copy) Oct 2
- Update 18 sheets to Oct 2 15:37 local versions
- Keep cleaned layout: exclude .history/, Resources/, *.bak, *.lck,
  project.kicad_dru, .hs_rules.json, lowercase dup placeholders
  (fixtures/power), empty orphans (digital, mechanical, output,
  USBC_MCU, eMMC_UFS)
- Preserve LICENSE, README.md, .gitignore
Parts:
- C313, C314, C332, C334: footprint Capacitor_SMD:C_0402_1005Metric_Pad0.74x0.62mm_HandSolder -> Capacitor_SMD:C_0402_1005Metric
- R118, R119, R147, R157, R158, R164, R165, R166, R173, R174, R179, R180: LCSC Part C114765 -> C106231; Mouser Part 603-RC0402FR-0722RL -> 603-RC0402FR-070RL
Connections:
- net AVDD33: no longer R73.1, R74.1
- new net VCCA_1V8_S3: R73.1, R74.1

Commit message: Relink hierarchical root: 18 sheets into RK3576 SBCv2 top level
Root was empty (no sheet boxes); all subsheets orphaned.
Rebuilt A1 top level linking RK3576, LPDDR5, Power, Ethernet,
HDMI, MIPI, PCIe, USB-A/C, Wireless, RTC, uSD, GPIO, OLED,
RP2350A, Connectors, Fixtures, DC_Power. block_diagrame kept
docs-only (unlinked, avoids double-instantiation). Lowercase
stub duplicates excluded. ERC: 1388 -> 770 violations.
Parts:
- removed J10, J6: LPJG0926HENL, Datasheet_Footprints:LPJG0926HENL, symbol LPJG0926HENL:LPJG0926HENL
- added J8, J9: LPJG0926HENL, Datasheet_Footprints:LPJG0926HENL, symbol LPJG0926HENL:LPJG0926HENL
- renumbered C308 to C197, C330 to C198, C309 to C199, C331 to C200, C332 to C201, C313 to C202, C334 to C203, C314 to C204, C335 to C205, C312 to C206, C306 to C207, C311 to C208, C300 to C209, C304 to C210, C350 to C211, C351 to C212, C301 to C213, C349 to C214, C353 to C215, C400 to C216, C417 to C217, C302 to C218, C310 to C219, C416 to C220, C415 to C221, C418 to C222, C419 to C223, C303 to C224, C329 to C225, C333 to C226, J8 to J10, J12 to J11, L14 to L2, L12 to L3, R143 to R100, R73 to R101, R150 to R102, R268 to R103, R74 to R104, R75 to R105, R157 to R106, R164 to R107, R165 to R108, R166 to R109, R179 to R110, R180 to R111, R118 to R112, R119 to R113, R147 to R114, R158 to R115, R173 to R116, R174 to R117, R95 to R118, R168 to R119, R77 to R120, R181 to R121, R79 to R122, R96 to R123, R99 to R124, R100 to R125, R101 to R126, R185 to R127, R169 to R128, R170 to R129, R171 to R130, R172 to R131, R78 to R132, R186 to R133, R97 to R134, R182 to R135, R98 to R136, R187 to R137, R76 to R78, R80 to R79, R90 to R80, R92 to R81, R94 to R82, R123 to R83, R128 to R84, R130 to R85, R135 to R86, R139 to R87, R140 to R88, R141 to R89, R142 to R90, R72 to R91, R82 to R92, R83 to R93, R84 to R94, R85 to R95, R87 to R96, R89 to R97, R91 to R98, R93 to R99, U25 to U24, U26 to U25, Y6 to Y5, Y4 to Y6
Connections:
- net ETH0_{PHY}_MDI0_N: now also J8.2 (TD1-)
- net ETH0_{PHY}_MDI0_P: now also J8.1 (TD1+)
- net ETH0_{PHY}_MDI1_N: now also J8.6 (TD2-)
- net ETH0_{PHY}_MDI1_P: now also J8.3 (TD2+)
- net ETH0_{PHY}_MDI2_N: now also J8.8 (TD3-)
- net ETH0_{PHY}_MDI2_P: now also J8.7 (TD3+)
- net ETH0_{PHY}_MDI3_N: now also J8.10 (TD4-)
- net ETH0_{PHY}_MDI3_P: now also J8.9 (TD4+)
- net ETH1_{PHY}_MDI0_N: now also J9.2 (TD1-)
- net ETH1_{PHY}_MDI0_P: now also J9.1 (TD1+)
- net ETH1_{PHY}_MDI1_N: now also J9.6 (TD2-)
- net ETH1_{PHY}_MDI1_P: now also J9.3 (TD2+)
- net ETH1_{PHY}_MDI2_N: now also J9.8 (TD3-)
- net ETH1_{PHY}_MDI2_P: now also J9.7 (TD3+)
- net ETH1_{PHY}_MDI3_N: now also J9.10 (TD4-)
- net ETH1_{PHY}_MDI3_P: now also J9.9 (TD4+)
- net GND: now also J8.15, J8.17, J8.S1 (SHIELD), J8.S2 (SHIELD), J9.15, J9.17, J9.S1 (SHIELD), J9.S2 (SHIELD)
- net RJ45_CT_C0: now also J8.4 (CT), J8.5 (CT)
- net RJ45_CT_C1: now also J9.4 (CT), J9.5 (CT)
- net RJ45_VC1_C0: now also J8.11 (VC1)
- net RJ45_VC1_C1: now also J9.11 (VC1)
- net RJ45_VC2_C0: now also J8.12 (VC2)
- net RJ45_VC2_C1: now also J9.12 (VC2)
- net RJ45_VC3_C0: now also J8.13 (VC3)
- net RJ45_VC3_C1: now also J9.13 (VC3)
- net RJ45_VC4_C0: now also J8.14 (VC4)
- net RJ45_VC4_C1: now also J9.14 (VC4)
- net at R78.1: now also J8.16
- net at R81.1: now also J9.18
- net at R80.1: now also J9.16
- net at R79.1: now also J8.18

Commit message: block diagrame with Hierarchical labels and NVMe SSD footprint
Parts:
- renumbered R92 to R82, R93 to R83, R94 to R84, R95 to R85, R96 to R86, R97 to R87, R98 to R88, R99 to R89, R84 to R90, R85 to R91, R86 to R92, R87 to R93, R88 to R94, R82 to R95, R83 to R96, R89 to R97, R90 to R98, R91 to R99
Connections:
- net ETH0_{PHY}_MDC renamed ETH0_{PHY}.MDC
- net ETH0_{PHY}_MDIO renamed ETH0_{PHY}.MDIO
- net ETH0_{PHY}_RESET renamed ETH0_{PHY}_nRST
- net ETH0_{PHY}_RXC renamed ETH0_{PHY}.RXC
- net ETH0_{PHY}_RXCTL renamed ETH0_{PHY}.RXCTL
- net ETH0_{PHY}_RXD0 renamed ETH0_{PHY}.RXD0
- net ETH0_{PHY}_RXD1 renamed ETH0_{PHY}.RXD1
- net ETH0_{PHY}_RXD2 renamed ETH0_{PHY}.RXD2
- net ETH0_{PHY}_RXD3 renamed ETH0_{PHY}.RXD3
- net ETH0_{PHY}_TXC renamed ETH0_{PHY}.TXC
- net ETH0_{PHY}_TXCTL renamed ETH0_{PHY}.TXCTL
- net ETH0_{PHY}_TXD0 renamed ETH0_{PHY}.TXD0
- net ETH0_{PHY}_TXD1 renamed ETH0_{PHY}.TXD1
- net ETH0_{PHY}_TXD2 renamed ETH0_{PHY}.TXD2
- net ETH0_{PHY}_TXD3 renamed ETH0_{PHY}.TXD3
- net ETH1_{PHY}_MDC renamed ETH1_{PHY}.MDC
- net ETH1_{PHY}_MDIO renamed ETH1_{PHY}.MDIO
- net ETH1_{PHY}_RESET renamed ETH1_{PHY}_nRST
- net ETH1_{PHY}_RXC renamed ETH1_{PHY}.RXC
- net ETH1_{PHY}_RXCTL renamed ETH1_{PHY}.RXCTL
- net ETH1_{PHY}_RXD0 renamed ETH1_{PHY}.RXD0
- net ETH1_{PHY}_RXD1 renamed ETH1_{PHY}.RXD1
- net ETH1_{PHY}_RXD2 renamed ETH1_{PHY}.RXD2
- net ETH1_{PHY}_RXD3 renamed ETH1_{PHY}.RXD3
- net ETH1_{PHY}_TXC renamed ETH1_{PHY}.TXC
- net ETH1_{PHY}_TXCTL renamed ETH1_{PHY}.TXCTL
- net ETH1_{PHY}_TXD0 renamed ETH1_{PHY}.TXD0
- net ETH1_{PHY}_TXD1 renamed ETH1_{PHY}.TXD1
- net ETH1_{PHY}_TXD2 renamed ETH1_{PHY}.TXD2
- net ETH1_{PHY}_TXD3 renamed ETH1_{PHY}.TXD3
Other:
- moved on the sheet: C197, C198, C199, C200, C201, C202, C203, C204, C205, C206, C207, C208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
