File: Fixtures.kicad_sch (KiCad schematic)
At the start: 19 parts

Commit message: Relink hierarchical root: 18 sheets into RK3576 SBCv2 top level
Root was empty (no sheet boxes); all subsheets orphaned.
Rebuilt A1 top level linking RK3576, LPDDR5, Power, Ethernet,
HDMI, MIPI, PCIe, USB-A/C, Wireless, RTC, uSD, GPIO, OLED,
RP2350A, Connectors, Fixtures, DC_Power. block_diagrame kept
docs-only (unlinked, avoids double-instantiation). Lowercase
stub duplicates excluded. ERC: 1388 -> 770 violations.
Parts:
- removed H5, H6, H7, H8: MountingHole_Pad, MountingHole:MountingHole_2.2mm_M2_DIN965_Pad_TopBottom, symbol Mechanical:MountingHole_Pad
- added H1, H2, H3, H4: MountingHole_Pad, MountingHole:MountingHole_2.7mm_Pad_Via, symbol Mechanical:MountingHole_Pad
- renumbered FID5 to FID1, FID6 to FID2, FID7 to FID3, FID8 to FID4, R252 to R207, R255 to R208, R256 to R209, R257 to R210, TP8 to TP1, TP9 to TP2, TP10 to TP3, TP11 to TP4, TP12 to TP5, TP13 to TP6, TP14 to TP7
Connections:
- net at R210.1: now also H4.1
- net at R208.1: now also H2.1
- net at R207.1: now also H1.1
- net at R209.1: now also H3.1

Commit message: Update v2 schematics + PCB: impedance profiles, design rules, sheet fixes
- pro: copper/track widths, microvias, 40/50 OHM + DIFF 85/90/100 tuning profiles
- dru/pcb: updated constraints and layout
- sheets: RK3576, RP2350A, Fixtures, MIPI, PCIe, HDMI, LPDDR5, UFS/eMMC, OLED, block diagram
Parts:
- H1, H2, H3, H4: footprint MountingHole:MountingHole_2.7mm_Pad_Via -> MountingHole:MountingHole_3.2mm_M3_Pad_Via

Commit message: block diagrame with Hierarchical labels and NVMe SSD footprint
Parts:
- renumbered R207 to R208, R208 to R209, R209 to R210, R210 to R211
Changed lines of the file:
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@@
 		(in_pos_files yes)
 		(dnp no)
-		(property "Reference" "#PWR0527"
+		(property "Reference" "#PWR0536"
 			(at 33.02 99.06 0)
 			(hide yes)
@@
 			(project "RK3576 SBCv2"
 				(path "/802f5b9f-44c6-4b1a-a63a-2c094d5816db/b1762425-fa86-48de-998c-9dee18dd9420"
-					(reference "#PWR0527")
+					(reference "#PWR0536")
 					(unit 1)
 				)
@@
 		(in_pos_files yes)
 		(dnp no)
-		(property "Reference" "#PWR0529"
+		(property "Reference" "#PWR0538"
 			(at 124.46 55.88 0)
 			(hide yes)
@@
 			(project "RK3576 SBCv2"
 				(path "/802f5b9f-44c6-4b1a-a63a-2c094d5816db/b1762425-fa86-48de-998c-9dee18dd9420"
-					(reference "#PWR0529")
+					(reference "#PWR0538")
 					(unit 1)
 				)
@@
 		(in_pos_files yes)
 		(dnp no)
-		(property "Reference" "#PWR0522"
+		(property "Reference" "#PWR0531"
 			(at 33.02 52.07 0)
 			(hide yes)
@@
 			(project "RK3576 SBCv2"
 				(path "/802f5b9f-44c6-4b1a-a63a-2c094d5816db/b1762425-fa86-48de-998c-9dee18dd9420"
-					(reference "#PWR0522")
+					(reference "#PWR0531")
 					(unit 1)
 				)
@@
 		(in_pos_files yes)
 		(dnp no)
-		(property "Reference" "#PWR0525"
+		(property "Reference" "#PWR0534"
 			(at 33.02 78.74 0)
 			(hide yes)
@@
 			(project "RK3576 SBCv2"
 				(path "/802f5b9f-44c6-4b1a-a63a-2c094d5816db/b1762425-fa86-48de-998c-9dee18dd9420"
-					(reference "#PWR0525")
+					(reference "#PWR0534")
 					(unit 1)
 				)
@@
 		(in_pos_files yes)
 		(dnp no)
-		(property "Reference" "#PWR0530"
+		(property "Reference" "#PWR0539"
 			(at 148.59 55.88 0)
 			(hide yes)
@@
 			(project "RK3576 SBCv2"
 				(path "/802f5b9f-44c6-4b1a-a63a-2c094d5816db/b1762425-fa86-48de-998c-9dee18dd9420"
-					(reference "#PWR0530")
+					(reference "#PWR0539")
 					(unit 1)
 				)
@@
 		(in_pos_files yes)
 		(dnp no)
-		(property "Reference" "#PWR0521"
+		(property "Reference" "#PWR0530"
 			(at 33.02 43.18 0)
 			(hide yes)
@@
 			(project "RK3576 SBCv2"
 				(path "/802f5b9f-44c6-4b1a-a63a-2c094d5816db/b1762425-fa86-48de-998c-9dee18dd9420"
-					(reference "#PWR0521")
+					(reference "#PWR0530")
 					(unit 1)
 				)
@@
 		(in_pos_files yes)
 		(dnp no)
-		(property "Reference" "R208"
+		(property "Reference" "R209"
 			(at 125.984 45.72 0)
 			(show_name no)
@@
 			(project "RK3576 SBCv2"
 				(path "/802f5b9f-44c6-4b1a-a63a-2c094d5816db/b1762425-fa86-48de-998c-9dee18dd9420"
-					(reference "R208")
+					(reference "R209")
 					(unit 1)
 				)
@@
 		(in_pos_files yes)
 		(dnp no)
-		(property "Reference" "#PWR0526"
+		(property "Reference" "#PWR0535"
 			(at 33.02 91.44 0)
 			(hide yes)
@@
 			(project "RK3576 SBCv2"
 				(path "/802f5b9f-44c6-4b1a-a63a-2c094d5816db/b1762425-fa86-48de-998c-9dee18dd9420"
-					(reference "#PWR0526")
+					(reference "#PWR0535")
 					(unit 1)
 				)
@@
 		(in_pos_files yes)
 		(dnp no)
-		(property "Reference" "#PWR0531"
+		(property "Reference" "#PWR0540"
 			(at 172.72 55.88 0)
 			(hide yes)
@@
 			(project "RK3576 SBCv2"
 				(path "/802f5b9f-44c6-4b1a-a63a-2c094d5816db/b1762425-fa86-48de-998c-9dee18dd9420"
-					(reference "#PWR0531")
+					(reference "#PWR0540")
 					(unit 1)
 				)
@@
 		(in_pos_files yes)
 		(dnp no)
-		(property "Reference" "#PWR0524"
+		(property "Reference" "#PWR0533"
 			(at 33.02 69.85 0)
 			(hide yes)
@@
 			(project "RK3576 SBCv2"
 				(path "/802f5b9f-44c6-4b1a-a63a-2c094d5816db/b1762425-fa86-48de-998c-9dee18dd9420"
-					(reference "#PWR0524")
+					(reference "#PWR0533")
 					(unit 1)
 				)
@@
 		(in_pos_files yes)
 		(dnp no)
-		(property "Reference" "#PWR0528"
+		(property "Reference" "#PWR0537"
 			(at 100.33 55.88 0)
 			(hide yes)
@@
 			(project "RK3576 SBCv2"
 				(path "/802f5b9f-44c6-4b1a-a63a-2c094d5816db/b1762425-fa86-48de-998c-9dee18dd9420"
-					(reference "#PWR0528")
+					(reference "#PWR0537")
 					(unit 1)
 				)
@@
 		(in_pos_files yes)
 		(dnp no)
-		(property "Reference" "R207"
+		(property "Reference" "R208"
 			(at 101.854 45.72 0)
 			(show_name no)
@@
 			(project "RK3576 SBCv2"
 				(path "/802f5b9f-44c6-4b1a-a63a-2c094d5816db/b1762425-fa86-48de-998c-9dee18dd9420"
-					(reference "R207")
+					(reference "R208")
 					(unit 1)
 				)
@@
 		(in_pos_files yes)
 		(dnp no)
-		(property "Reference" "R210"
+		(property "Reference" "R211"
 			(at 174.244 45.72 0)
 			(show_name no)
@@
 			(project "RK3576 SBCv2"
 				(path "/802f5b9f-44c6-4b1a-a63a-2c094d5816db/b1762425-fa86-48de-998c-9dee18dd9420"
-					(reference "R210")
+					(reference "R211")
 					(unit 1)
 				)
@@
 		(in_pos_files yes)
 		(dnp no)
-		(property "Reference" "R209"
+		(property "Reference" "R210"
 			(at 150.114 45.72 0)
 			(show_name no)
@@
 			(project "RK3576 SBCv2"
 				(path "/802f5b9f-44c6-4b1a-a63a-2c094d5816db/b1762425-fa86-48de-998c-9dee18dd9420"
-					(reference "R209")
+					(reference "R210")
 					(unit 1)
 				)
@@
 		(in_pos_files yes)
 		(dnp no)
-		(property "Reference" "#PWR0523"
+		(property "Reference" "#PWR0532"
 			(at 33.02 60.96 0)
 			(hide yes)
@@
 			(project "RK3576 SBCv2"
 				(path "/802f5b9f-44c6-4b1a-a63a-2c094d5816db/b1762425-fa86-48de-998c-9dee18dd9420"
-					(reference "#PWR0523")
-					(unit 1)
-				)
+					(reference "#PWR0532")
+					(unit 1)
+				)
