File: HDMI.kicad_sch (KiCad schematic)
At the start: 41 parts, among them J7 HDMI-001S, Q2 2SK3018, Q3 2SK3018, Q4 2SK3018, Q5 2SK3018, U20 AP2553W6-7, U21 TXB0104PWR, U22 TPD4E05U06DQAR, U23 TPD4E05U06DQAR, U24 TPD4E05U06DQAR

Commit message: Replace v2 with updated RK3576_SBCv2 (Copy) Oct 2
- Update 18 sheets to Oct 2 15:37 local versions
- Keep cleaned layout: exclude .history/, Resources/, *.bak, *.lck,
  project.kicad_dru, .hs_rules.json, lowercase dup placeholders
  (fixtures/power), empty orphans (digital, mechanical, output,
  USBC_MCU, eMMC_UFS)
- Preserve LICENSE, README.md, .gitignore
Parts:
- R112: LCSC Part C60491 -> C60490; Mouser Part 603-RC0402FR-07100KL -> 603-RC0402FR-0710KL

Commit message: Relink hierarchical root: 18 sheets into RK3576 SBCv2 top level
Root was empty (no sheet boxes); all subsheets orphaned.
Rebuilt A1 top level linking RK3576, LPDDR5, Power, Ethernet,
HDMI, MIPI, PCIe, USB-A/C, Wireless, RTC, uSD, GPIO, OLED,
RP2350A, Connectors, Fixtures, DC_Power. block_diagrame kept
docs-only (unlinked, avoids double-instantiation). Lowercase
stub duplicates excluded. ERC: 1388 -> 770 violations.
Parts:
- renumbered C316 to C227, C325 to C228, C326 to C229, C317 to C230, C318 to C231, C319 to C232, C320 to C233, C321 to C234, C322 to C235, C323 to C236, C324 to C237, C315 to C238, C327 to C239, C328 to C240, D14 to D12, D18 to D13, J7 to J12, R116 to R138, R111 to R139, R112 to R140, R102 to R141, R103 to R142, R104 to R143, R105 to R144, R106 to R145, R115 to R146, R107 to R147, R108 to R148, R113 to R149, R109 to R150, R114 to R151, R110 to R152, U22 to U26, U20 to U27, U23 to U28, U24 to U29, U21 to U30

Commit message: block diagrame with Hierarchical labels and NVMe SSD footprint
Parts:
- renumbered D12 to D28, D13 to D29
Connections:
- net CHDMI_CEC: now also U29.10 (NC)
- net CHDMI_CK_N: now also U28.6 (NC)
- net CHDMI_CK_P: now also U28.7 (NC)
- net CHDMI_D0_N: now also U28.9 (NC)
- net CHDMI_D0_P: now also U28.10 (NC)
- net CHDMI_D1_N: now also U26.6 (NC)
- net CHDMI_D1_P: now also U26.7 (NC)
- net CHDMI_D2_N: now also U26.9 (NC)
- net CHDMI_D2_P: now also U26.10 (NC)
- net CHDMI_UTILITY: now also U29.6 (NC)
- net CSCL: now also U29.9 (NC)
- net CSDA: now also U29.7 (NC)
- net HDMI_CK_N renamed HDMI.CK_N
- net HDMI_CK_P renamed HDMI.CK_P
- net HDMI_D0_N renamed HDMI.D0_N
- net HDMI_D0_P renamed HDMI.D0_P
- net HDMI_D1_N renamed HDMI.D1_N
- net HDMI_D1_P renamed HDMI.D1_P
- net HDMI_D2_N renamed HDMI.D2_N
- net HDMI_D2_P renamed HDMI.D2_P
- net HDMI_TX_SBD_N renamed HDMI.TX_SBD_N
- net HDMI_TX_SBD_P renamed HDMI.TX_SBD_P
- no-connect marks 13 -> 1
