File: LPDDR5.kicad_sch (KiCad schematic)
At the start: 64 parts, among them U18 MT62F1G32D4DR-031 WT:B

Commit message: Replace v2 with updated RK3576_SBCv2 (Copy) Oct 2
- Update 18 sheets to Oct 2 15:37 local versions
- Keep cleaned layout: exclude .history/, Resources/, *.bak, *.lck,
  project.kicad_dru, .hs_rules.json, lowercase dup placeholders
  (fixtures/power), empty orphans (digital, mechanical, output,
  USBC_MCU, eMMC_UFS)
- Preserve LICENSE, README.md, .gitignore
Parts:
- R138: LCSC Part C106231 -> C114755; Mouser Part 603-RC0402FR-070RL -> 603-RC0402FR-07240RL

Commit message: Relink hierarchical root: 18 sheets into RK3576 SBCv2 top level
Root was empty (no sheet boxes); all subsheets orphaned.
Rebuilt A1 top level linking RK3576, LPDDR5, Power, Ethernet,
HDMI, MIPI, PCIe, USB-A/C, Wireless, RTC, uSD, GPIO, OLED,
RP2350A, Connectors, Fixtures, DC_Power. block_diagrame kept
docs-only (unlinked, avoids double-instantiation). Lowercase
stub duplicates excluded. ERC: 1388 -> 770 violations.
Parts:
- removed U18: MT62F1G32D4DR-031 WT:B, easyeda2kicad:LPDDR5 BGA 315, symbol antmicroMemory:MT62F1G32D4DR-031
- added C324, C332, C333: 22u, Capacitor_SMD:C_0603_1608Metric, symbol New_Library_0:C_Small_edited
- added C325: 1u, Capacitor_SMD:C_0201_0603Metric_Pad0.64x0.40mm_HandSolder, symbol New_Library_0:C_Small_edited
- added L4: XRIM252012S2R2MBCA, Inductor_SMD:L_1008_2520Metric, symbol Device:L_Small
- added R197: 100k, PCM_Resistor_SMD_AKL:R_0402_1005Metric, symbol Device:R_Small
- added R198: 200k, PCM_Resistor_SMD_AKL:R_0402_1005Metric, symbol Device:R_Small
- added U37: MT62F1G32D4DR-031 WT:B, easyeda2kicad:LPDDR5 BGA 315, symbol antmicroMemory:MT62F1G32D4DR-031
- added U38: SY8089AAAC, Package_TO_SOT_SMD:SOT-23-5, symbol Regulator_Switching:TLV62568DBV
- renumbered C270 to C268, C285 to C269, C271 to C270, C286 to C271, C287 to C273, C273 to C274, C288 to C275, C274 to C276, C289 to C277, C275 to C278, C290 to C279, C276 to C280, C291 to C281, C266 to C282, C277 to C283, C292 to C284, C267 to C285, C278 to C286, C293 to C287, C268 to C288, C279 to C289, C294 to C290, C269 to C291, C238 to C292, C252 to C293, C280 to C294, C239 to C296, C253 to C297, C281 to C298, C296 to C299, C240 to C300, C254 to C301, C282 to C302, C297 to C303, C241 to C304, C255 to C305, C397 to C306, C298 to C307, C242 to C308, C256 to C309, C284 to C310, C299 to C311, C243 to C312, C257 to C313, C244 to C314, C258 to C315, C245 to C316, C259 to C317, C246 to C318, C260 to C319, C247 to C320, C261 to C321, C248 to C322, C262 to C323, C249 to C326, C263 to C327, C250 to C328, C264 to C329, C251 to C330, C265 to C331, R138 to R196
Connections:
- net GND: now also C324.2, C325.2, C332.2, C333.2, R198.2, U37.A11 (VSS), U37.A5 (VSS), U37.AA11 (VSS), U37.AA5 (VSS), U37.B12 (VSS), U37.B4 (VSS), U37.B8 (VSS), U37.C11 (VSS), U37.C5 (VSS), U37.C8 (VSS), U37.D10 (VSS), U37.D14 (VSS), U37.D2 (VSS), U37.D6 (VSS), U37.D7 (VSS), U37.D9 (VSS), U37.E1 (VSS), U37.E13 (VSS), U37.E15 (VSS), U37.E3 (VSS), U37.E8 (VSS), U37.F14 (VSS), U37.F2 (VSS), U37.F8 (VSS), U37.G11 (VSS), U37.G13 (VSS), U37.G3 (VSS), U37.G5 (VSS), U37.G7 (VSS), U37.G9 (VSS), U37.H10 (VSS), U37.H12 (VSS), U37.H3 (VSS), U37.H4 (VSS), U37.H6 (VSS), U37.H8 (VSS), U37.J1 (VSS), U37.J10 (VSS), U37.J12 (VSS), U37.J13 (VSS), U37.J15 (VSS), U37.J3 (VSS), U37.J7 (VSS), U37.J8 (VSS), U37.K7 (VSS), U37.K8 (VSS), U37.K9 (VSS), U37.L1 (VSS), U37.L11 (VSS), U37.L12 (VSS), U37.L13 (VSS), U37.L14 (VSS), U37.L15 (VSS), U37.L2 (VSS), U37.L3 (VSS), U37.L4 (VSS), U37.L5 (VSS), U37.M7 (VSS), U37.M8 (VSS), U37.M9 (VSS), U37.N1 (VSS), U37.N10 (VSS), U37.N12 (VSS), U37.N13 (VSS), U37.N15 (VSS), U37.N3 (VSS), U37.N4 (VSS), U37.N6 (VSS), U37.N8 (VSS), U37.N9 (VSS), U37.P10 (VSS), U37.P12 (VSS), U37.P13 (VSS), U37.P4 (VSS), U37.P6 (VSS), U37.P8 (VSS), U37.R11 (VSS), U37.R13 (VSS), U37.R3 (VSS), U37.R5 (VSS), U37.R7 (VSS), U37.R9 (VSS), U37.T14 (VSS), U37.T2 (VSS), U37.T8 (VSS), U37.U1 (VSS), U37.U13 (VSS), U37.U15 (VSS), U37.U3 (VSS), U37.U8 (VSS), U37.V10 (VSS), U37.V14 (VSS), U37.V2 (VSS), U37.V6 (VSS), U37.V7 (VSS), U37.V9 (VSS), U37.W11 (VSS), U37.W5 (VSS), U37.W8 (VSS), U37.Y12 (VSS), U37.Y4 (VSS), U37.Y8 (VSS), U38.2 (GND)
- net LPDDR5_A.CA0: now also U37.G4 (CA0_A)
- net LPDDR5_A.CA1: now also U37.H5 (CA1_A)
- net LPDDR5_A.CA2: now also U37.G8 (CA2_A)
- net LPDDR5_A.CA3: now also U37.H11 (CA3_A)
- net LPDDR5_A.CA4: now also U37.G10 (CA4_A)
- net LPDDR5_A.CA5: now also U37.H13 (CA5_A)
- net LPDDR5_A.CA6: now also U37.G12 (CA6_A)
- net LPDDR5_A.CK_N: now also U37.J9 (CK_c_A)
- net LPDDR5_A.CK_P: now also U37.H9 (CK_t_A)
- net LPDDR5_A.CS0: now also U37.H7 (CS0_A)
- net LPDDR5_A.CS1: now also U37.G6 (CS1_A)
- net LPDDR5_A.DMI0: now also U37.A4 (DMI0_A)
- net LPDDR5_A.DMI1: now also U37.A12 (DMI1_A)
- net LPDDR5_A.DQ0: now also U37.D1 (DQ0_A)
- net LPDDR5_A.DQ1: now also U37.C2 (DQ1_A)
- net LPDDR5_A.DQ10: now also U37.E14 (DQ10_A)
- net LPDDR5_A.DQ11: now also U37.D13 (DQ11_A)
- net LPDDR5_A.DQ12: now also U37.B11 (DQ12_A)
- net LPDDR5_A.DQ13: now also U37.C10 (DQ13_A)
- net LPDDR5_A.DQ14: now also U37.E10 (DQ14_A)
- net LPDDR5_A.DQ15: now also U37.F11 (DQ15_A)
- net LPDDR5_A.DQ2: now also U37.E2 (DQ2_A)
- net LPDDR5_A.DQ3: now also U37.D3 (DQ3_A)
- net LPDDR5_A.DQ4: now also U37.B5 (DQ4_A)
- net LPDDR5_A.DQ5: now also U37.C6 (DQ5_A)
- net LPDDR5_A.DQ6: now also U37.E6 (DQ6_A)
- net LPDDR5_A.DQ7: now also U37.F5 (DQ7_A)
- net LPDDR5_A.DQ8: now also U37.D15 (DQ8_A)
- net LPDDR5_A.DQ9: now also U37.C14 (DQ9_A)
- net LPDDR5_A.RDQS0_N: now also U37.C4 (RDQS0_c_A)
- net LPDDR5_A.RDQS0_P: now also U37.B3 (RDQS0_t_A)
- net LPDDR5_A.RDQS1_N: now also U37.C12 (RDQS1_c_A)
- net LPDDR5_A.RDQS1_P: now also U37.B13 (RDQS1_t_A)
- net LPDDR5_A.WCK0_N: now also U37.D5 (WCK0_c_A)
- net LPDDR5_A.WCK0_P: now also U37.E4 (WCK0_t_A)
- net LPDDR5_A.WCK1_N: now also U37.D11 (WCK1_c_A)
- net LPDDR5_A.WCK1_P: now also U37.E12 (WCK1_t_A)
- net LPDDR5_B.CA0: now also U37.R12 (CA0_B)
- net LPDDR5_B.CA1: now also U37.P11 (CA1_B)
- net LPDDR5_B.CA2: now also U37.R8 (CA2_B)
- net LPDDR5_B.CA3: now also U37.P5 (CA3_B)
- net LPDDR5_B.CA4: now also U37.R6 (CA4_B)
- net LPDDR5_B.CA5: now also U37.P3 (CA5_B)
- net LPDDR5_B.CA6: now also U37.R4 (CA6_B)
- net LPDDR5_B.CK_N: now also U37.N7 (CK_c_B)
- net LPDDR5_B.CK_P: now also U37.P7 (CK_t_B)
- net LPDDR5_B.CS0: now also U37.P9 (CS0_B)
- net LPDDR5_B.CS1: now also U37.R10 (CS1_B)
- net LPDDR5_B.DMI0: now also U37.AA12 (DMI0_B)
- net LPDDR5_B.DMI1: now also U37.AA4 (DMI1_B)
- net LPDDR5_B.DQ0: now also U37.V15 (DQ0_B)
- net LPDDR5_B.DQ1: now also U37.W14 (DQ1_B)
- net LPDDR5_B.DQ10: now also U37.U2 (DQ10_B)
- net LPDDR5_B.DQ11: now also U37.V3 (DQ11_B)
- net LPDDR5_B.DQ12: now also U37.Y5 (DQ12_B)
- net LPDDR5_B.DQ13: now also U37.W6 (DQ13_B)
- net LPDDR5_B.DQ14: now also U37.U6 (DQ14_B)
- net LPDDR5_B.DQ15: now also U37.T5 (DQ15_B)
- net LPDDR5_B.DQ2: now also U37.U14 (DQ2_B)
- net LPDDR5_B.DQ3: now also U37.V13 (DQ3_B)
- net LPDDR5_B.DQ4: now also U37.Y11 (DQ4_B)
- net LPDDR5_B.DQ5: now also U37.W10 (DQ5_B)
- net LPDDR5_B.DQ6: now also U37.U10 (DQ6_B)
- net LPDDR5_B.DQ7: now also U37.T11 (DQ7_B)
- net LPDDR5_B.DQ8: now also U37.V1 (DQ8_B)
- net LPDDR5_B.DQ9: now also U37.W2 (DQ9_B)
- net LPDDR5_B.RDQS0_N: now also U37.W12 (RDQS0_c_B)
- net LPDDR5_B.RDQS0_P: now also U37.Y13 (RDQS0_t_B)
- net LPDDR5_B.RDQS1_N: now also U37.W4 (RDQS1_c_B)
- net LPDDR5_B.RDQS1_P: now also U37.Y3 (RDQS1_t_B)
- net LPDDR5_B.WCK0_N: now also U37.V11 (WCK0_c_B)
- net LPDDR5_B.WCK0_P: now also U37.U12 (WCK0_t_B)
- net LPDDR5_B.WCK1_N: now also U37.V5 (WCK1_c_B)
- net LPDDR5_B.WCK1_P: now also U37.U4 (WCK1_t_B)
- net LPDDR5_RESET: now also U37.H1 (RESET_n)
- net VCC_1V8_S3: now also U37.C1 (VDD1), U37.C15 (VDD1), U37.W1 (VDD1), U37.W15 (VDD1)
- net VDD2L_0V9_DDR_S3: now also C332.1, C333.1, L4.2, R197.1, U37.A10 (VDD2L), U37.A6 (VDD2L), U37.AA10 (VDD2L), U37.AA6 (VDD2L), U37.B10 (VDD2L), U37.B6 (VDD2L), U37.H14 (VDD2L), U37.H2 (VDD2L), U37.J14 (VDD2L), U37.J2 (VDD2L), U37.N14 (VDD2L), U37.N2 (VDD2L), U37.P14 (VDD2L), U37.P2 (VDD2L), U37.Y10 (VDD2L), U37.Y6 (VDD2L)
- net VDD2_DDR_S3: now also U37.A7 (VDD2H), U37.A8 (VDD2H), U37.A9 (VDD2H), U37.AA7 (VDD2H), U37.AA8 (VDD2H), U37.AA9 (VDD2H), U37.B7 (VDD2H), U37.B9 (VDD2H), U37.C7 (VDD2H), U37.C9 (VDD2H), U37.D8 (VDD2H), U37.E7 (VDD2H), U37.E9 (VDD2H), U37.F10 (VDD2H), U37.F6 (VDD2H), U37.F7 (VDD2H), U37.F9 (VDD2H), U37.J11 (VDD2H), U37.J5 (VDD2H), U37.K1 (VDD2H), U37.K10 (VDD2H), U37.K11 (VDD2H), U37.K12 (VDD2H), U37.K13 (VDD2H), U37.K14 (VDD2H), U37.K15 (VDD2H), U37.K2 (VDD2H), U37.K3 (VDD2H), U37.K4 (VDD2H), U37.K5 (VDD2H), U37.K6 (VDD2H), U37.L10 (VDD2H), U37.L6 (VDD2H), U37.L7 (VDD2H), U37.L8 (VDD2H), U37.L9 (VDD2H), U37.M1 (VDD2H), U37.M10 (VDD2H), U37.M11 (VDD2H), U37.M12 (VDD2H), U37.M13 (VDD2H), U37.M14 (VDD2H), U37.M15 (VDD2H), U37.M2 (VDD2H), U37.M3 (VDD2H), U37.M4 (VDD2H), U37.M5 (VDD2H), U37.M6 (VDD2H), U37.N11 (VDD2H), U37.N5 (VDD2H), U37.T10 (VDD2H), U37.T6 (VDD2H), U37.T7 (VDD2H), U37.T9 (VDD2H), U37.U7 (VDD2H), U37.U9 (VDD2H), U37.V8 (VDD2H), U37.W7 (VDD2H), U37.W9 (VDD2H), U37.Y7 (VDD2H), U37.Y9 (VDD2H)
- net VDDQ_DDR_S0: now also U37.A13 (VDDQ), U37.A3 (VDDQ), U37.AA13 (VDDQ), U37.AA3 (VDDQ), U37.B14 (VDDQ), U37.B2 (VDDQ), U37.C13 (VDDQ), U37.C3 (VDDQ), U37.D12 (VDDQ), U37.D4 (VDDQ), U37.E11 (VDDQ), U37.E5 (VDDQ), U37.F1 (VDDQ), U37.F12 (VDDQ), U37.F13 (VDDQ), U37.F15 (VDDQ), U37.F3 (VDDQ), U37.F4 (VDDQ), U37.G1 (VDDQ), U37.G14 (VDDQ), U37.G15 (VDDQ), U37.G2 (VDDQ), U37.R1 (VDDQ), U37.R14 (VDDQ), U37.R15 (VDDQ), U37.R2 (VDDQ), U37.T1 (VDDQ), U37.T12 (VDDQ), U37.T13 (VDDQ), U37.T15 (VDDQ), U37.T3 (VDDQ), U37.T4 (VDDQ), U37.U11 (VDDQ), U37.U5 (VDDQ), U37.V12 (VDDQ), U37.V4 (VDDQ), U37.W13 (VDDQ), U37.W3 (VDDQ), U37.Y14 (VDDQ), U37.Y2 (VDDQ)
- net at R196.2: now also U37.H15 (ZQ_A)
- new net: L4.1, U38.3 (SW)
- new net: R197.2, R198.1, U38.5 (FB)
- new net VCC5V0_SYS: C324.1, C325.1, U38.1 (EN), U38.4 (VIN)

Commit message: block diagrame with Hierarchical labels and NVMe SSD footprint
Parts:
- renumbered C324 to C322, C322 to C323, C323 to C324, R196 to R197, R197 to R198, R198 to R199
Connections:
- net LPDDR5_RESET renamed LPDDR5_nRTS
Other:
- moved on the sheet: C322, C325, C332, C333, L4, R198, R199, U37C, U38
