File: Power.kicad_sch (KiCad schematic)
At the start: 121 parts, among them J1 Barrel_Jack_Switch, Q8 AO3401A, SW1 SKRTLAE010, U10 RK806S-5, U14 SY8388ARHC, U15 SY8089AAAC

Commit message: Replace v2 with updated RK3576_SBCv2 (Copy) Oct 2
- Update 18 sheets to Oct 2 15:37 local versions
- Keep cleaned layout: exclude .history/, Resources/, *.bak, *.lck,
  project.kicad_dru, .hs_rules.json, lowercase dup placeholders
  (fixtures/power), empty orphans (digital, mechanical, output,
  USBC_MCU, eMMC_UFS)
- Preserve LICENSE, README.md, .gitignore
Parts:
- removed U10: RK806S-5, Package_DFN_QFN:QFN-68-1EP_8x8mm_P0.4mm_EP6.4x6.4mm_ThermalVias, symbol Datasheet_Symbols:RK806S-5
- added R124, R125: 2.2k, PCM_Resistor_SMD_AKL:R_0402_1005Metric, symbol Device:R_Small
- added U13: RK806S-5, symbol Datasheet_Symbols:RK806S-5
- J1: footprint Connector_BarrelJack:BarrelJack_CUI_PJ-063AH_Horizontal -> Datasheet_Footprints:DC-JACK-TH-2.5_HC-DC-007B-2.5; LCSC Part (none) -> C3010538
- R191, R193, R195, R6, R7: LCSC Part C60491 -> C60490; Mouser Part 603-RC0402FR-07100KL -> 603-RC0402FR-0710KL
- R216: LCSC Part C60490 -> C138065; Mouser Part 603-RC0402FR-0710KL -> 603-RC0402FR-07110KL
- R5, R8: LCSC Part C114765 -> C106231; Mouser Part 603-RC0402FR-0722RL -> 603-RC0402FR-070RL
Connections:
- net GND: now also U13.31 (FB6), U13.47 (FB5), U13.66 (FB9), U13.69 (EP)
- net I2C1_SCL_M0_RK806: now also R125.2, U13.17 (CLK/SCL)
- net I2C1_SDA_M0_RK806: now also R124.2, U13.15 (MOSI/SDA)
- net PMIC_EXT_EN_OUT: now also U13.39 (EXT_EN)
- net PMIC_INT_L: now also U13.19 (INT)
- net PMIC_PWR_CTRL1: now also U13.62 (PWRCRTL1)
- net PMIC_PWR_CTRL2: now also U13.61 (PWRCRTL2)
- net PMIC_PWR_CTRL3: now also U13.16 (MISO/PWRCRTL3)
- net VCC1: now also U13.1 (VCC9), U13.21 (VCCA), U13.22 (VCC4), U13.27 (VCC10), U13.28 (VCC6), U13.33 (VCC2), U13.34 (VCC2), U13.43 (VCC7), U13.44 (VCC5), U13.52 (VCC1), U13.53 (VCC1), U13.54 (VCC3), U13.64 (VCC12), U13.7 (VCC8)
- net VCCA1V8_PLDO2_S0: now also U13.58 (PLDO2)
- net VCCA1V8_PLDO6_S3: now also U13.20 (VCCIO)
- net VCCA_1V8_S0: now also U13.60 (PLDO1)
- net VCCA_3V3_S0: now also U13.63 (PLDO4)
- net VCCIO_SD_S0: now also U13.65 (PLDO5)
- net VCC_1V8_S3: now also R124.1, R125.1
- net VCC_2V0_PLDO_S3: now also U13.13 (VCC13), U13.59 (VCC11), U13.9 (VCC14)
- net VDDA0V75_HDMI_S0: now also U13.11 (NLDO3)
- net VDDA_0V75_S0: now also U13.8 (NLDO5)
- net VDDA_0V85_S0: now also U13.10 (NLDO4)
- net VDDA_1V2_S0: now also U13.57 (PLDO3)
- net VDDA_DDR_PLL_S0: now also U13.12 (NLDO2)
- net VDD_0V75_S3: now also U13.14 (NLDO1)
- net at L1.1: now also U13.50 (SW1), U13.51 (SW1)
- net at L7.1: now also U13.42 (SW7)
- net at L10.1: now also U13.26 (SW10)
- net at NT9.1: now also U13.67 (VOUT9)
- net at NT7.1: now also U13.41 (VOUT7)
- net at NT4.1: now also U13.24 (VOUT4)
- net at L2.1: now also U13.35 (SW2), U13.36 (SW2)
- net at C21.1, C22.1, R8.1: now also U13.4 (PWRON)
- net at L9.1: now also U13.68 (SW9)
- net at C15.1, R6.2, R7.1: now also U13.32 (VDC)
- net at L4.1: now also U13.23 (SW4)
- net at NT1.1: now also U13.49 (VOUT1)
- net at NT5.1: now also U13.46 (VOUT5)
- net at L3.1: now also U13.55 (SW3)
- net at NT6.1: now also U13.30 (VOUT6)
- net at NT10.1: now also U13.25 (VOUT10)
- net at L5.1: now also U13.45 (SW5)
- net at R5.1: now also U13.40 (~{RESETB})
- net at NT8.1: now also U13.5 (VOUT8)
- net at NT2.1: now also U13.37 (VOUT2)
- net at L6.1: now also U13.29 (SW6)
- net at NT3.1: now also U13.56 (VOUT3)
- net at L8.1: now also U13.6 (SW8)
Other:
- moved on the sheet: R1

Commit message: Relink hierarchical root: 18 sheets into RK3576 SBCv2 top level
Root was empty (no sheet boxes); all subsheets orphaned.
Rebuilt A1 top level linking RK3576, LPDDR5, Power, Ethernet,
HDMI, MIPI, PCIe, USB-A/C, Wireless, RTC, uSD, GPIO, OLED,
RP2350A, Connectors, Fixtures, DC_Power. block_diagrame kept
docs-only (unlinked, avoids double-instantiation). Lowercase
stub duplicates excluded. ERC: 1388 -> 770 violations.
Parts:
- removed J1: Barrel_Jack_Switch, Datasheet_Footprints:DC-JACK-TH-2.5_HC-DC-007B-2.5, symbol Connector:Barrel_Jack_Switch
- removed SW1: SKRTLAE010, easyeda2kicad:SKRTLAE010, symbol Switch:SW_Push
- added J21: Barrel_Jack_Switch, Datasheet_Footprints:DC-JACK-TH-2.5_HC-DC-007B-2.5, symbol Connector:Barrel_Jack_Switch
- added SW5: SKRTLAE010, easyeda2kicad:SKRTLAE010, symbol Switch:SW_Push
- R225: renamed from R213; value 10k -> 200k
- R226: renamed from R214; value 10k -> 100k
- U42: renamed from U13; footprint (none) -> Package_DFN_QFN:ArtInChip_QFN-68-1EP_7x7mm_P0.35mm_EP5.49x5.49mm
- renumbered C1 to C347, C8 to C348, C16 to C349, C23 to C350, C29 to C351, C34 to C352, C41 to C353, C52 to C354, C58 to C355, C63 to C356, C2 to C357, C9 to C358, C17 to C359, C24 to C360, C30 to C361, C37 to C362, C42 to C363, C53 to C364, C59 to C365, C64 to C366, C45 to C367, C3 to C368, C10 to C369, C18 to C370, C25 to C371, C31 to C372, C38 to C373, C43 to C374, C54 to C375, C60 to C376, C65 to C377, C4 to C378, C11 to C379, C19 to C380, C26 to C381, C32 to C382, C39 to C383, C44 to C384, C55 to C385, C61 to C386, C66 to C387, C413 to C388, C414 to C389, C305 to C390, C5 to C391, C27 to C392, C35 to C393, C56 to C394, C345 to C395, C50 to C396, C51 to C397, C6 to C398, C14 to C399, C20 to C400, C28 to C401, C33 to C402, C36 to C403, C40 to C404, C49 to C405, C57 to C406, C62 to C407, C46 to C408, C12 to C409, C283 to C410, C7 to C411, C13 to C412, C15 to C413, C21 to C414, C48 to C415, C22 to C416, C47 to C417, D25 to D20, D1 to D21, F4 to F2, L6 to L10, L7 to L11, L8 to L12, L9 to L13, L10 to L14, L13 to L15, L11 to L16, L1 to L5, L2 to L6, L3 to L7, L4 to L8, L5 to L9, Q8 to Q7, R190 to R211, R191 to R212, R192 to R213, R193 to R214, R194 to R215, R195 to R216, R183 to R217, R224 to R218, R217 to R219, R215 to R220, R216 to R221, R223 to R222, R6 to R223, R7 to R224, R5 to R227, R8 to R228, R124 to R229, R125 to R230, R1 to R231, U14 to U43, U15 to U44
Connections:
- net GND: now also J21.2, J21.3, SW5.2
- net PMIC_PWRON_L: now also SW5.1
- net at F2.1: now also J21.1
Other:
- note removed: "SY8089AAAC"

Commit message: block diagrame with Hierarchical labels and NVMe SSD footprint
Parts:
- added R234: 100k, PCM_Resistor_SMD_AKL:R_0402_1005Metric, symbol Device:R_Small
- renumbered C347 to C346, C348 to C347, C349 to C348, C350 to C349, C351 to C350, C352 to C351, C353 to C352, C354 to C353, C355 to C354, C356 to C355, C357 to C356, C358 to C357, C359 to C358, C360 to C359, C361 to C360, C362 to C361, C363 to C362, C364 to C363, C365 to C364, C366 to C365, C367 to C366, C368 to C367, C369 to C368, C370 to C369, C371 to C370, C372 to C371, C373 to C372, C374 to C373, C375 to C374, C376 to C375, C377 to C376, C378 to C377, C379 to C378, C380 to C379, C381 to C380, C382 to C381, C383 to C382, C384 to C383, C385 to C384, C386 to C385, C387 to C386, C388 to C387, C389 to C388, C390 to C389, C391 to C390, C392 to C391, C393 to C392, C394 to C393, C395 to C394, C396 to C395, C397 to C396, C398 to C397, C399 to C398, C400 to C399, C401 to C400, C402 to C401, C403 to C402, C404 to C403, C405 to C404, C406 to C405, C407 to C406, C408 to C407, C409 to C408, C410 to C409, C411 to C410, C412 to C411, C413 to C412, C414 to C413, C415 to C414, C416 to C415, C417 to C416, D20 to D60, D21 to D61, R211 to R212, R212 to R213, R213 to R214, R214 to R215, R215 to R216, R216 to R217, R217 to R218, R218 to R219, R219 to R220, R220 to R221, R221 to R222, R222 to R223, R223 to R224, R224 to R225, R225 to R226, R226 to R227, R227 to R228, R228 to R229, R229 to R230, R230 to R231, R231 to R232
Connections:
- net PMIC_EXT_EN_OUT: now also R234.2
- net VCC1: no longer U44.1 (EN)
- net at C415.1, R229.1, U42.4 (PWRON): no longer C413.1
- net at R228.1, U42.40 (~{RESETB}): now also C413.1
- net PMIC_PWR_CTRL3: no longer names the net of U42.16 (MISO/PWRCRTL3)
- net RESET_L renamed PMIC_nRST
- new net: R234.1, U44.1 (EN)
- no-connect marks 6 -> 7
Other:
- moved on the sheet: C407, C409, R230, R231
