File: RK3576 SBCv2.kicad_pcb (KiCad board)
At the start: 2 copper layers, 65 x 56 mm, 5 parts, among them J1 GPIO

Commit message: Relink hierarchical root: 18 sheets into RK3576 SBCv2 top level
Root was empty (no sheet boxes); all subsheets orphaned.
Rebuilt A1 top level linking RK3576, LPDDR5, Power, Ethernet,
HDMI, MIPI, PCIe, USB-A/C, Wireless, RTC, uSD, GPIO, OLED,
RP2350A, Connectors, Fixtures, DC_Power. block_diagrame kept
docs-only (unlinked, avoids double-instantiation). Lowercase
stub duplicates excluded. ERC: 1388 -> 770 violations.
Parts:
- removed MH1, MH2, MH3, MH4: MountingHole_2.7mm_M2.5, MountingHole:MountingHole_2.7mm_M2.5
- added BT1: BS-06-B4AA012, easyeda2kicad:BAT-SMD_BS-06-B4AA012, B.Cu at (164.0, 195.5)
- added C1: 12pF, Capacitor_SMD:C_0402_1005Metric, F.Cu at (303.3, 172.1)
- added C10: 12pF, Capacitor_SMD:C_0402_1005Metric, F.Cu at (303.3, 174.1)
- added C100: 1u, Capacitor_SMD:C_0201_0603Metric_Pad0.64x0.40mm_HandSolder, F.Cu at (298.8, 143.2)
- added C101: 1u, Capacitor_SMD:C_0201_0603Metric_Pad0.64x0.40mm_HandSolder, F.Cu at (298.8, 144.9)
- added C102: 1u, Capacitor_SMD:C_0201_0603Metric_Pad0.64x0.40mm_HandSolder, F.Cu at (298.8, 146.7)
- added C103: 1u, Capacitor_SMD:C_0201_0603Metric_Pad0.64x0.40mm_HandSolder, F.Cu at (298.8, 148.4)
- added C104: 1u, Capacitor_SMD:C_0201_0603Metric_Pad0.64x0.40mm_HandSolder, F.Cu at (298.8, 150.2)
- added C105: 18pF, Capacitor_SMD:C_0402_1005Metric, F.Cu at (303.3, 176.1)
- added C106: 22u, Capacitor_SMD:C_0603_1608Metric, F.Cu at (287.7, 160.1)
- added C107: 22u, Capacitor_SMD:C_0603_1608Metric, F.Cu at (287.7, 162.6)
- added C108: 22u, Capacitor_SMD:C_0603_1608Metric, F.Cu at (287.7, 165.1)
- added C109: 22u, Capacitor_SMD:C_0603_1608Metric, F.Cu at (287.7, 167.6)
- added C11: 1u, Capacitor_SMD:C_0201_0603Metric_Pad0.64x0.40mm_HandSolder, F.Cu at (279.1, 143.2)
- added C110: 22u, Capacitor_SMD:C_0603_1608Metric, F.Cu at (287.7, 170.1)
- added C111: 22u, Capacitor_SMD:C_0603_1608Metric, F.Cu at (287.7, 172.6)
- added C112: 18pF, Capacitor_SMD:C_0402_1005Metric, F.Cu at (303.3, 178.0)
- added C113: 22u, Capacitor_SMD:C_0603_1608Metric, F.Cu at (311.9, 196.5)
- added C114: 1u, Capacitor_SMD:C_0201_0603Metric_Pad0.64x0.40mm_HandSolder, F.Cu at (291.9, 182.1)
- added C115: 1u, Capacitor_SMD:C_0201_0603Metric_Pad0.64x0.40mm_HandSolder, F.Cu at (291.9, 183.8)
- added C116: 1u, Capacitor_SMD:C_0201_0603Metric_Pad0.64x0.40mm_HandSolder, F.Cu at (291.9, 185.6)
- added C117: 1u, Capacitor_SMD:C_0201_0603Metric_Pad0.64x0.40mm_HandSolder, F.Cu at (291.9, 187.3)
- added C118: 34pF, Capacitor_SMD:C_0402_1005Metric, F.Cu at (297.4, 206.2)
- added C119: 34pF, Capacitor_SMD:C_0402_1005Metric, F.Cu at (297.4, 208.2)
- added C12: 10u, Capacitor_SMD:C_0603_1608Metric, F.Cu at (279.7, 170.1)
- added C120: 1u, Capacitor_SMD:C_0201_0603Metric_Pad0.64x0.40mm_HandSolder, F.Cu at (291.9, 189.1)
- added C121: 1u, Capacitor_SMD:C_0201_0603Metric_Pad0.64x0.40mm_HandSolder, F.Cu at (291.9, 190.8)
- added C122: 1u, Capacitor_SMD:C_0201_0603Metric_Pad0.64x0.40mm_HandSolder, F.Cu at (294.7, 182.1)
- added C123: 1u, Capacitor_SMD:C_0201_0603Metric_Pad0.64x0.40mm_HandSolder, F.Cu at (294.7, 183.8)
- added C124: 1u, Capacitor_SMD:C_0201_0603Metric_Pad0.64x0.40mm_HandSolder, F.Cu at (294.7, 185.6)
- added C125: 1u, Capacitor_SMD:C_0201_0603Metric_Pad0.64x0.40mm_HandSolder, F.Cu at (294.7, 187.3)
- added C126: 1u, Capacitor_SMD:C_0201_0603Metric_Pad0.64x0.40mm_HandSolder, F.Cu at (294.7, 189.1)
- added C127: 1u, Capacitor_SMD:C_0201_0603Metric_Pad0.64x0.40mm_HandSolder, F.Cu at (294.7, 190.8)
- added C128: 1u, Capacitor_SMD:C_0201_0603Metric_Pad0.64x0.40mm_HandSolder, F.Cu at (297.5, 182.1)
- added C129: 1u, Capacitor_SMD:C_0201_0603Metric_Pad0.64x0.40mm_HandSolder, F.Cu at (297.5, 183.8)
- added C13: 1u, Capacitor_SMD:C_0201_0603Metric_Pad0.64x0.40mm_HandSolder, F.Cu at (279.1, 144.9)
- added C130: 1u, Capacitor_SMD:C_0201_0603Metric_Pad0.64x0.40mm_HandSolder, F.Cu at (297.5, 185.6)
- added C131: 100n, Capacitor_SMD:C_0201_0603Metric_Pad0.64x0.40mm_HandSolder, F.Cu at (343.6, 92.4)
- added C132: 100n, Capacitor_SMD:C_0201_0603Metric_Pad0.64x0.40mm_HandSolder, F.Cu at (343.6, 94.1)
- added C133: 100n, Capacitor_SMD:C_0201_0603Metric_Pad0.64x0.40mm_HandSolder, F.Cu at (343.6, 95.9)
- added C134: 100n, Capacitor_SMD:C_0201_0603Metric_Pad0.64x0.40mm_HandSolder, F.Cu at (343.6, 97.6)
- added C135: 100n, Capacitor_SMD:C_0201_0603Metric_Pad0.64x0.40mm_HandSolder, F.Cu at (343.6, 99.4)
- added C136: 100n, Capacitor_SMD:C_0201_0603Metric_Pad0.64x0.40mm_HandSolder, F.Cu at (343.6, 101.1)
- added C137: 100n, Capacitor_SMD:C_0201_0603Metric_Pad0.64x0.40mm_HandSolder, F.Cu at (346.5, 92.4)
- added C138: 100n, Capacitor_SMD:C_0201_0603Metric_Pad0.64x0.40mm_HandSolder, F.Cu at (346.5, 94.1)
- added C139: 100n, Capacitor_SMD:C_0201_0603Metric_Pad0.64x0.40mm_HandSolder, F.Cu at (346.5, 95.9)
- added C14: 1u, Capacitor_SMD:C_0201_0603Metric_Pad0.64x0.40mm_HandSolder, F.Cu at (279.1, 146.7)
- added C140: 100n, Capacitor_SMD:C_0201_0603Metric_Pad0.64x0.40mm_HandSolder, F.Cu at (346.5, 97.6)
- added C141: 22u, Capacitor_SMD:C_0603_1608Metric, F.Cu at (353.3, 109.5)
- added C142: DNP, Capacitor_SMD:C_0201_0603Metric_Pad0.64x0.40mm_HandSolder, F.Cu at (346.5, 99.4)
- added C143: 200pF, Capacitor_SMD:C_0402_1005Metric, F.Cu at (356.7, 109.2)
- added C144: 200pF, Capacitor_SMD:C_0402_1005Metric, F.Cu at (356.7, 111.2)
- added C145: 1u, Capacitor_SMD:C_0201_0603Metric_Pad0.64x0.40mm_HandSolder, F.Cu at (346.5, 101.1)
- added C146: 1u, Capacitor_SMD:C_0201_0603Metric_Pad0.64x0.40mm_HandSolder, F.Cu at (349.3, 92.4)
- added C147: 1u, Capacitor_SMD:C_0201_0603Metric_Pad0.64x0.40mm_HandSolder, F.Cu at (349.3, 94.1)
- added C148: 1u, Capacitor_SMD:C_0201_0603Metric_Pad0.64x0.40mm_HandSolder, F.Cu at (349.3, 95.9)
- added C149: 22u, Capacitor_SMD:C_0603_1608Metric, F.Cu at (234.5, 115.6)
- added C15: 1u, Capacitor_SMD:C_0201_0603Metric_Pad0.64x0.40mm_HandSolder, F.Cu at (279.1, 148.4)
- added C150: 22u, Capacitor_SMD:C_0603_1608Metric, F.Cu at (234.5, 118.1)
- added C151: 22u, Capacitor_SMD:C_0603_1608Metric, F.Cu at (234.5, 120.7)
- added C152: 22u, Capacitor_SMD:C_0603_1608Metric, F.Cu at (234.5, 123.2)
- added C153: 100n, Capacitor_SMD:C_0201_0603Metric_Pad0.64x0.40mm_HandSolder, F.Cu at (247.6, 111.9)
- added C154: 100n, Capacitor_SMD:C_0201_0603Metric_Pad0.64x0.40mm_HandSolder, F.Cu at (247.6, 113.6)
- added C155: 100n, Capacitor_SMD:C_0201_0603Metric_Pad0.64x0.40mm_HandSolder, F.Cu at (247.6, 115.4)
- added C156: 100n, Capacitor_SMD:C_0201_0603Metric_Pad0.64x0.40mm_HandSolder, F.Cu at (247.6, 117.1)
- added C157: 100n, Capacitor_SMD:C_0201_0603Metric_Pad0.64x0.40mm_HandSolder, F.Cu at (247.6, 118.9)
- added C158: 100n, Capacitor_SMD:C_0201_0603Metric_Pad0.64x0.40mm_HandSolder, F.Cu at (247.6, 120.6)
- added C159: 100n, Capacitor_SMD:C_0201_0603Metric_Pad0.64x0.40mm_HandSolder, F.Cu at (247.6, 122.4)
- added C16: 1u, Capacitor_SMD:C_0201_0603Metric_Pad0.64x0.40mm_HandSolder, F.Cu at (279.1, 150.2)
- added C160: 100n, Capacitor_SMD:C_0201_0603Metric_Pad0.64x0.40mm_HandSolder, F.Cu at (247.6, 124.1)
- added C161: 100n, Capacitor_SMD:C_0201_0603Metric_Pad0.64x0.40mm_HandSolder, F.Cu at (250.4, 111.9)
- added C162: 100n, Capacitor_SMD:C_0201_0603Metric_Pad0.64x0.40mm_HandSolder, F.Cu at (250.4, 113.6)
- added C163: 100n, Capacitor_SMD:C_0201_0603Metric_Pad0.64x0.40mm_HandSolder, F.Cu at (250.4, 115.4)
- added C164: 100n, Capacitor_SMD:C_0201_0603Metric_Pad0.64x0.40mm_HandSolder, F.Cu at (250.4, 117.1)
- added C165: 100n, Capacitor_SMD:C_0201_0603Metric_Pad0.64x0.40mm_HandSolder, F.Cu at (250.4, 118.9)
- added C166: 100n, Capacitor_SMD:C_0201_0603Metric_Pad0.64x0.40mm_HandSolder, F.Cu at (250.4, 120.6)
- added C167: 100n, Capacitor_SMD:C_0201_0603Metric_Pad0.64x0.40mm_HandSolder, F.Cu at (250.4, 122.4)
- added C168: 100n, Capacitor_SMD:C_0201_0603Metric_Pad0.64x0.40mm_HandSolder, F.Cu at (250.4, 124.1)
- added C169: 1u, Capacitor_SMD:C_0201_0603Metric_Pad0.64x0.40mm_HandSolder, F.Cu at (253.2, 111.9)
- added C17: 10u, Capacitor_SMD:C_0603_1608Metric, F.Cu at (279.7, 172.6)
- added C170: 1u, Capacitor_SMD:C_0201_0603Metric_Pad0.64x0.40mm_HandSolder, F.Cu at (253.2, 113.6)
- added C171: 1u, Capacitor_SMD:C_0201_0603Metric_Pad0.64x0.40mm_HandSolder, F.Cu at (253.2, 115.4)
- added C172: 1u, Capacitor_SMD:C_0201_0603Metric_Pad0.64x0.40mm_HandSolder, F.Cu at (253.2, 117.1)
- added C173: 10u, Capacitor_SMD:C_0603_1608Metric, F.Cu at (234.5, 125.7)
- added C174: 1u, Capacitor_SMD:C_0201_0603Metric_Pad0.64x0.40mm_HandSolder, F.Cu at (253.2, 118.9)
- added C175: 1u, Capacitor_SMD:C_0201_0603Metric_Pad0.64x0.40mm_HandSolder, F.Cu at (253.2, 120.6)
- added C176: 1u, Capacitor_SMD:C_0201_0603Metric_Pad0.64x0.40mm_HandSolder, F.Cu at (253.2, 122.4)
- added C177: 1u, Capacitor_SMD:C_0201_0603Metric_Pad0.64x0.40mm_HandSolder, F.Cu at (253.2, 124.1)
- added C178: 1u, Capacitor_SMD:C_0201_0603Metric_Pad0.64x0.40mm_HandSolder, F.Cu at (256.0, 111.9)
- added C179: 1u, Capacitor_SMD:C_0201_0603Metric_Pad0.64x0.40mm_HandSolder, F.Cu at (256.0, 113.6)
- added C18: 1u, Capacitor_SMD:C_0201_0603Metric_Pad0.64x0.40mm_HandSolder, F.Cu at (279.1, 151.9)
- added C180: 1u, Capacitor_SMD:C_0201_0603Metric_Pad0.64x0.40mm_HandSolder, F.Cu at (256.0, 115.4)
- added C181: 34pF, Capacitor_SMD:C_0402_1005Metric, F.Cu at (247.6, 130.3)
- added C182: 1u, Capacitor_SMD:C_0201_0603Metric_Pad0.64x0.40mm_HandSolder, F.Cu at (256.0, 117.1)
- added C183: 1u, Capacitor_SMD:C_0201_0603Metric_Pad0.64x0.40mm_HandSolder, F.Cu at (256.0, 118.9)
- added C184: 1u, Capacitor_SMD:C_0201_0603Metric_Pad0.64x0.40mm_HandSolder, F.Cu at (256.0, 120.6)
- added C185: 10u, Capacitor_SMD:C_0603_1608Metric, F.Cu at (234.5, 128.2)
- added C186: 1u, Capacitor_SMD:C_0201_0603Metric_Pad0.64x0.40mm_HandSolder, F.Cu at (256.0, 122.4)
- added C187: 1u, Capacitor_SMD:C_0201_0603Metric_Pad0.64x0.40mm_HandSolder, F.Cu at (256.0, 124.1)
- added C188: 1u, Capacitor_SMD:C_0201_0603Metric_Pad0.64x0.40mm_HandSolder, F.Cu at (258.8, 111.9)
- added C189: 10u, Capacitor_SMD:C_0603_1608Metric, F.Cu at (234.5, 130.7)
- added C19: 1u, Capacitor_SMD:C_0201_0603Metric_Pad0.64x0.40mm_HandSolder, F.Cu at (279.1, 153.7)
- added C190: 34pF, Capacitor_SMD:C_0402_1005Metric, F.Cu at (247.6, 132.2)
- added C191: 1u, Capacitor_SMD:C_0201_0603Metric_Pad0.64x0.40mm_HandSolder, F.Cu at (258.8, 113.6)
- added C192: 1u, Capacitor_SMD:C_0201_0603Metric_Pad0.64x0.40mm_HandSolder, F.Cu at (258.8, 115.4)
- added C193: 1u, Capacitor_SMD:C_0201_0603Metric_Pad0.64x0.40mm_HandSolder, F.Cu at (258.8, 117.1)
- added C194: 1u, Capacitor_SMD:C_0201_0603Metric_Pad0.64x0.40mm_HandSolder, F.Cu at (258.8, 118.9)
- added C195: 1u, Capacitor_SMD:C_0201_0603Metric_Pad0.64x0.40mm_HandSolder, F.Cu at (258.8, 120.6)
- added C196: 10u, Capacitor_SMD:C_0603_1608Metric, F.Cu at (234.5, 133.2)
- added C197: 1u, Capacitor_SMD:C_0201_0603Metric_Pad0.64x0.40mm_HandSolder, F.Cu at (262.2, 175.5)
- added C198: 1u, Capacitor_SMD:C_0201_0603Metric_Pad0.64x0.40mm_HandSolder, F.Cu at (262.2, 177.3)
- added C199: 1u, Capacitor_SMD:C_0201_0603Metric_Pad0.64x0.40mm_HandSolder, F.Cu at (262.2, 179.0)
- added C2: 22u, Capacitor_SMD:C_0603_1608Metric, F.Cu at (279.7, 157.5)
- added C20: 1u, Capacitor_SMD:C_0201_0603Metric_Pad0.64x0.40mm_HandSolder, F.Cu at (279.1, 155.4)
- added C200: 1u, Capacitor_SMD:C_0201_0603Metric_Pad0.64x0.40mm_HandSolder, F.Cu at (262.2, 180.8)
- added C201: 18pF, Capacitor_SMD:C_0402_1005Metric, F.Cu at (273.5, 175.6)
- added C202: 18pF, Capacitor_SMD:C_0402_1005Metric, F.Cu at (273.5, 177.6)
- added C203: 18pF, Capacitor_SMD:C_0402_1005Metric, F.Cu at (273.5, 179.6)
- added C204: 18pF, Capacitor_SMD:C_0402_1005Metric, F.Cu at (273.5, 181.5)
- added C205: 1u, Capacitor_SMD:C_0201_0603Metric_Pad0.64x0.40mm_HandSolder, F.Cu at (262.2, 182.5)
- added C206: 1u, Capacitor_SMD:C_0201_0603Metric_Pad0.64x0.40mm_HandSolder, F.Cu at (265.0, 175.5)
- added C207: 1u, Capacitor_SMD:C_0201_0603Metric_Pad0.64x0.40mm_HandSolder, F.Cu at (265.0, 177.3)
- added C208: 1u, Capacitor_SMD:C_0201_0603Metric_Pad0.64x0.40mm_HandSolder, F.Cu at (265.0, 179.0)
- added C209: 1u, Capacitor_SMD:C_0201_0603Metric_Pad0.64x0.40mm_HandSolder, F.Cu at (265.0, 180.8)
- added C21: 1u, Capacitor_SMD:C_0201_0603Metric_Pad0.64x0.40mm_HandSolder, F.Cu at (281.9, 137.9)
- added C210: 1u, Capacitor_SMD:C_0201_0603Metric_Pad0.64x0.40mm_HandSolder, F.Cu at (265.0, 182.5)
- added C211: 1u, Capacitor_SMD:C_0201_0603Metric_Pad0.64x0.40mm_HandSolder, F.Cu at (267.8, 175.5)
- added C212: 1u, Capacitor_SMD:C_0201_0603Metric_Pad0.64x0.40mm_HandSolder, F.Cu at (267.8, 177.3)
- added C213: 1u, Capacitor_SMD:C_0201_0603Metric_Pad0.64x0.40mm_HandSolder, F.Cu at (267.8, 179.0)
- added C214: 1u, Capacitor_SMD:C_0201_0603Metric_Pad0.64x0.40mm_HandSolder, F.Cu at (267.8, 180.8)
- added C215: 1u, Capacitor_SMD:C_0201_0603Metric_Pad0.64x0.40mm_HandSolder, F.Cu at (267.8, 182.5)
- added C216: 1u, Capacitor_SMD:C_0201_0603Metric_Pad0.64x0.40mm_HandSolder, F.Cu at (270.6, 175.5)
- added C217: 10u, Capacitor_SMD:C_0603_1608Metric, F.Cu at (273.7, 138.3)
- added C218: 1u, Capacitor_SMD:C_0201_0603Metric_Pad0.64x0.40mm_HandSolder, F.Cu at (270.6, 177.3)
- added C219: 1u, Capacitor_SMD:C_0201_0603Metric_Pad0.64x0.40mm_HandSolder, F.Cu at (270.6, 179.0)
- added C22: 1u, Capacitor_SMD:C_0201_0603Metric_Pad0.64x0.40mm_HandSolder, F.Cu at (281.9, 139.7)
- added C220: 10u, Capacitor_SMD:C_0603_1608Metric, F.Cu at (273.7, 140.8)
- added C221: 1u, Capacitor_SMD:C_0201_0603Metric_Pad0.64x0.40mm_HandSolder, F.Cu at (270.6, 180.8)
- added C222: 10u, Capacitor_SMD:C_0603_1608Metric, F.Cu at (273.7, 143.3)
- added C223: 10u, Capacitor_SMD:C_0603_1608Metric, F.Cu at (273.7, 145.8)
- added C224: 1u, Capacitor_SMD:C_0201_0603Metric_Pad0.64x0.40mm_HandSolder, F.Cu at (270.6, 182.5)
- added C225: 10u, Capacitor_SMD:C_0603_1608Metric, F.Cu at (273.7, 148.3)
- added C226: 10u, Capacitor_SMD:C_0603_1608Metric, F.Cu at (273.7, 150.8)
- added C227: 22u, Capacitor_SMD:C_0603_1608Metric, F.Cu at (357.7, 226.1)
- added C228: 220n, Capacitor_SMD:C_0201_0603Metric_Pad0.64x0.40mm_HandSolder, F.Cu at (351.3, 228.2)
- added C229: 220n, Capacitor_SMD:C_0201_0603Metric_Pad0.64x0.40mm_HandSolder, F.Cu at (351.3, 229.9)
- added C23: 1u, Capacitor_SMD:C_0201_0603Metric_Pad0.64x0.40mm_HandSolder, F.Cu at (281.9, 141.4)
- added C230: 220n, Capacitor_SMD:C_0201_0603Metric_Pad0.64x0.40mm_HandSolder, F.Cu at (351.3, 231.7)
- added C231: 220n, Capacitor_SMD:C_0201_0603Metric_Pad0.64x0.40mm_HandSolder, F.Cu at (351.3, 233.4)
- added C232: 220n, Capacitor_SMD:C_0201_0603Metric_Pad0.64x0.40mm_HandSolder, F.Cu at (351.3, 235.2)
- added C233: 220n, Capacitor_SMD:C_0201_0603Metric_Pad0.64x0.40mm_HandSolder, F.Cu at (354.1, 228.2)
- added C234: 220n, Capacitor_SMD:C_0201_0603Metric_Pad0.64x0.40mm_HandSolder, F.Cu at (354.1, 229.9)
- added C235: 220n, Capacitor_SMD:C_0201_0603Metric_Pad0.64x0.40mm_HandSolder, F.Cu at (354.1, 231.7)
- added C236: 220n, Capacitor_SMD:C_0201_0603Metric_Pad0.64x0.40mm_HandSolder, F.Cu at (354.1, 233.4)
- added C237: 220n, Capacitor_SMD:C_0201_0603Metric_Pad0.64x0.40mm_HandSolder, F.Cu at (354.1, 235.2)
- added C238: 1u, Capacitor_SMD:C_0201_0603Metric_Pad0.64x0.40mm_HandSolder, F.Cu at (356.9, 228.2)
- added C239: 1u, Capacitor_SMD:C_0201_0603Metric_Pad0.64x0.40mm_HandSolder, F.Cu at (356.9, 229.9)
- added C24: 1u, Capacitor_SMD:C_0201_0603Metric_Pad0.64x0.40mm_HandSolder, F.Cu at (281.9, 143.2)
- added C240: 1u, Capacitor_SMD:C_0201_0603Metric_Pad0.64x0.40mm_HandSolder, F.Cu at (356.9, 231.7)
- added C241: 1u, Capacitor_SMD:C_0201_0603Metric_Pad0.64x0.40mm_HandSolder, F.Cu at (291.7, 111.0)
- added C242: 22u, Capacitor_SMD:C_0603_1608Metric, F.Cu at (288.3, 111.4)
- added C243: 1u, Capacitor_SMD:C_0201_0603Metric_Pad0.64x0.40mm_HandSolder, F.Cu at (291.7, 112.8)
- added C244: 22u, Capacitor_SMD:C_0603_1608Metric, F.Cu at (318.5, 103.5)
- added C245: 1u, Capacitor_SMD:C_0201_0603Metric_Pad0.64x0.40mm_HandSolder, F.Cu at (315.1, 103.2)
- added C246: 1u, Capacitor_SMD:C_0201_0603Metric_Pad0.64x0.40mm_HandSolder, F.Cu at (315.1, 104.9)
- added C247: 1u, Capacitor_SMD:C_0201_0603Metric_Pad0.64x0.40mm_HandSolder, F.Cu at (315.1, 106.7)
- added C248: 1u, Capacitor_SMD:C_0201_0603Metric_Pad0.64x0.40mm_HandSolder, F.Cu at (346.1, 144.3)
- added C249: 1u, Capacitor_SMD:C_0201_0603Metric_Pad0.64x0.40mm_HandSolder, F.Cu at (346.1, 146.0)
- added C25: 100n, Capacitor_SMD:C_0201_0603Metric_Pad0.64x0.40mm_HandSolder, F.Cu at (281.9, 144.9)
- added C250: 1u, Capacitor_SMD:C_0201_0603Metric_Pad0.64x0.40mm_HandSolder, F.Cu at (346.1, 147.8)
- added C251: 22u, Capacitor_SMD:C_0603_1608Metric, F.Cu at (349.5, 144.7)
- added C252: 1u, Capacitor_SMD:C_0201_0603Metric_Pad0.64x0.40mm_HandSolder, F.Cu at (341.8, 124.4)
- added C253: 1u, Capacitor_SMD:C_0201_0603Metric_Pad0.64x0.40mm_HandSolder, F.Cu at (341.8, 126.2)
- added C254: 22u, Capacitor_SMD:C_0603_1608Metric, F.Cu at (338.4, 115.9)
- added C255: 10u, Capacitor_SMD:C_0603_1608Metric, F.Cu at (338.4, 118.4)
- added C256: 22u, Capacitor_SMD:C_0603_1608Metric, F.Cu at (338.4, 120.9)
- added C257: 10u, Capacitor_SMD:C_0603_1608Metric, F.Cu at (338.4, 123.4)
- added C258: 22u, Capacitor_SMD:C_0603_1608Metric, F.Cu at (338.4, 125.9)
- added C259: 1u, Capacitor_SMD:C_0201_0603Metric_Pad0.64x0.40mm_HandSolder, F.Cu at (341.8, 127.9)
- added C26: 100n, Capacitor_SMD:C_0201_0603Metric_Pad0.64x0.40mm_HandSolder, F.Cu at (281.9, 146.7)
- added C260: 22u, Capacitor_SMD:C_0603_1608Metric, F.Cu at (338.4, 128.4)
- added C261: 1u, Capacitor_SMD:C_0201_0603Metric_Pad0.64x0.40mm_HandSolder, F.Cu at (341.8, 129.7)
- added C262: 22u, Capacitor_SMD:C_0603_1608Metric, F.Cu at (338.4, 130.9)
- added C263: 1u, Capacitor_SMD:C_0201_0603Metric_Pad0.64x0.40mm_HandSolder, F.Cu at (341.8, 131.4)
- added C264: 22u, Capacitor_SMD:C_0603_1608Metric, F.Cu at (326.5, 229.1)
- added C265: 22u, Capacitor_SMD:C_0603_1608Metric, F.Cu at (326.5, 231.6)
- added C266: 1u, Capacitor_SMD:C_0201_0603Metric_Pad0.64x0.40mm_HandSolder, F.Cu at (329.9, 228.7)
- added C267: 1u, Capacitor_SMD:C_0201_0603Metric_Pad0.64x0.40mm_HandSolder, F.Cu at (329.9, 230.5)
- added C268: 22u, Capacitor_SMD:C_0603_1608Metric, F.Cu at (352.2, 199.0)
- added C269: 1u, Capacitor_SMD:C_0201_0603Metric_Pad0.64x0.40mm_HandSolder, F.Cu at (337.5, 182.1)
- added C27: 100n, Capacitor_SMD:C_0201_0603Metric_Pad0.64x0.40mm_HandSolder, F.Cu at (281.9, 148.4)
- added C270: 22u, Capacitor_SMD:C_0603_1608Metric, F.Cu at (352.2, 201.5)
- added C271: 1u, Capacitor_SMD:C_0201_0603Metric_Pad0.64x0.40mm_HandSolder, F.Cu at (337.5, 183.8)
- added C272: 22u, Capacitor_SMD:C_0603_1608Metric, F.Cu at (352.2, 204.0)
- added C273: 1u, Capacitor_SMD:C_0201_0603Metric_Pad0.64x0.40mm_HandSolder, F.Cu at (337.5, 185.6)
- added C274: 1u, Capacitor_SMD:C_0201_0603Metric_Pad0.64x0.40mm_HandSolder, F.Cu at (337.5, 187.3)
- added C275: 1u, Capacitor_SMD:C_0201_0603Metric_Pad0.64x0.40mm_HandSolder, F.Cu at (337.5, 189.1)
- added C276: 1u, Capacitor_SMD:C_0201_0603Metric_Pad0.64x0.40mm_HandSolder, F.Cu at (337.5, 190.8)
- added C277: 1u, Capacitor_SMD:C_0201_0603Metric_Pad0.64x0.40mm_HandSolder, F.Cu at (337.5, 192.6)
- added C278: 1u, Capacitor_SMD:C_0201_0603Metric_Pad0.64x0.40mm_HandSolder, F.Cu at (337.5, 194.3)
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Connections:
- J1 pad 1: +3V3 -> VCC_3.3v_S0
- J1 pad 2: +5V -> /RK3576 SOC/JTAG_TCK_M1 & UART0_TX_M0
- J1 pad 3: /GPIO2/SDA1 -> /RK3576 SOC/JTAG_TMS_M1 & UART0_RX_M0
- J1 pad 4: +5V -> GND
Other:
- board size 65 x 56 mm -> 100 x 80 mm
- board text removed: "CAMERA (OPTIONAL)"
- board text removed: "DISPLAY (OPTIONAL)"
- board text removed: "Extend PCB edge 0.5mm if using SMT header"
- board text removed: "PoE"
- board text removed: "RJ45"

Commit message: Update v2 schematics + PCB: impedance profiles, design rules, sheet fixes
- pro: copper/track widths, microvias, 40/50 OHM + DIFF 85/90/100 tuning profiles
- dru/pcb: updated constraints and layout
- sheets: RK3576, RP2350A, Fixtures, MIPI, PCIe, HDMI, LPDDR5, UFS/eMMC, OLED, block diagram
Parts:
- added R232: 0R, PCM_Resistor_SMD_AKL:R_0402_1005Metric, F.Cu at (274.1, 118.6)
- added R233: 0R, PCM_Resistor_SMD_AKL:R_0402_1005Metric, F.Cu at (274.1, 120.8)
- H1, H2, H3, H4: footprint MountingHole:MountingHole_2.7mm_Pad_Via -> MountingHole:MountingHole_3.2mm_M3_Pad_Via
- moved J3 220.7 mm to (360.8, 160.5), turned to -90 degrees
- moved U4 190.4 mm to (124.5, 146.1), turned to 180 degrees
- moved J18 128.2 mm to (89.2, 161.5)
- moved J13 117.2 mm to (198.8, 141.7), turned to -90 degrees
- moved J1 117.2 mm to (88.1, 152.5)
- moved H3 100.7 mm to (201.5, 123.8)
- moved J12 87.0 mm to (202.7, 167.5), turned to 90 degrees
- moved J19 84.9 mm to (187.9, 131.8), turned to -90 degrees
- moved J17 84.8 mm to (201.6, 142.5)
- moved J16 83.9 mm to (194.0, 142.5)
- moved H4 62.6 mm to (201.5, 194.8)
- moved J7 62.3 mm to (122.0, 192.1), turned to 0 degrees
- moved J4 58.1 mm to (128.9, 131.7), turned to -90 degrees
- moved U40 52.5 mm to (343.1, 218.3)
- moved U42 48.8 mm to (293.6, 184.3)
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Connections:
- U1 pad AB28: unconnected-(U1GPIO0-I2C0_SCL_M1-PadAB28) -> /RK3576 SOC/40GPIOs_PWR_EN
- U1 pad AD28: /RK3576 SOC/40GPIOs_PWR_EN -> /RK3576 SOC/PWM_FAN
Routing:
- net /MIPI/DSI0_TX_D0_P: track 0.00 -> 4.82 mm
- net /LPDDR5/LPDDR5_A.WCK0_N: track 0.00 -> 3.74 mm
- net /LPDDR5/LPDDR5_A.DQ5: track 0.00 -> 3.62 mm
- net /MIPI/CSI0_RX_D3_P: track 0.00 -> 2.82 mm
- net /MIPI/DSI0_TX_D0_N: track 0.00 -> 2.52 mm
- net /LPDDR5/LPDDR5_A.DQ0: track 0.00 -> 1.58 mm
- net /LPDDR5/LPDDR5_A.CS0: track 0.00 -> 1.50 mm
- net /RK3576 SOC/LPDDR5_B.DQ11: track 0.00 -> 1.03 mm
- net GND: track 0.00 -> 0.96 mm
Other:
- board size 100 x 80 mm -> 120 x 80 mm
- copper layers 2 -> 8

Commit message: block diagrame with Hierarchical labels and NVMe SSD footprint
Parts:
- removed C417: 22u, Capacitor_SMD:C_0603_1608Metric
- removed the J19 at (187.9, 131.8)
- removed the U41 at (388.4, 100.8)
- added D22: PESD5V0S1BA, PCM_Diode_SMD_AKL:D_SOD-323_TVS, F.Cu at (342.7, 156.4)
- added D23: PESD5V0S1BA, PCM_Diode_SMD_AKL:D_SOD-323_TVS, F.Cu at (342.7, 159.6)
- added D24: SMBJ5.0CA, PCM_Diode_SMD_AKL:D_SMB_TVS, F.Cu at (299.9, 124.8)
- added D25: SMBJ5.0CA, PCM_Diode_SMD_AKL:D_SMB_TVS, F.Cu at (299.9, 130.5)
- added D26: SMBJ5.0CA, PCM_Diode_SMD_AKL:D_SMB_TVS, F.Cu at (299.9, 136.2)
- added D27: SMBJ5.0CA, PCM_Diode_SMD_AKL:D_SMB_TVS, F.Cu at (299.9, 141.9)
- added D28: SMBJ5.0CA, PCM_Diode_SMD_AKL:D_SMB_TVS, F.Cu at (340.2, 215.6)
- added D29: PESD5V0S1BA, PCM_Diode_SMD_AKL:D_SOD-323_TVS, F.Cu at (333.5, 214.6)
- added D30: SMBJ5.0CA, PCM_Diode_SMD_AKL:D_SMB_TVS, F.Cu at (345.2, 124.8)
- added D31: PESD5V0S1BA, PCM_Diode_SMD_AKL:D_SOD-323_TVS, F.Cu at (332.9, 165.5)
- added D32: PESD5V0S1BA, PCM_Diode_SMD_AKL:D_SOD-323_TVS, F.Cu at (332.9, 168.6)
- added D33: PESD5V0S1BA, PCM_Diode_SMD_AKL:D_SOD-323_TVS, F.Cu at (332.9, 171.7)
- added D34: PESD5V0S1BA, PCM_Diode_SMD_AKL:D_SOD-323_TVS, F.Cu at (332.9, 174.8)
- added D35: PESD5V0S1BA, PCM_Diode_SMD_AKL:D_SOD-323_TVS, F.Cu at (332.9, 178.0)
- added D36: PESD5V0S1BA, PCM_Diode_SMD_AKL:D_SOD-323_TVS, F.Cu at (332.9, 181.1)
- added D37: PESD5V0S1BA, PCM_Diode_SMD_AKL:D_SOD-323_TVS, F.Cu at (332.9, 184.2)
- added D38: PESD5V0S1BA, PCM_Diode_SMD_AKL:D_SOD-323_TVS, F.Cu at (337.4, 165.5)
- added D39: PESD5V0S1BA, PCM_Diode_SMD_AKL:D_SOD-323_TVS, F.Cu at (337.4, 168.6)
- added D40: PESD5V0S1BA, PCM_Diode_SMD_AKL:D_SOD-323_TVS, F.Cu at (337.4, 171.7)
- added D41: PESD5V0S1BA, PCM_Diode_SMD_AKL:D_SOD-323_TVS, F.Cu at (337.4, 174.8)
- added D42: PESD5V0S1BA, PCM_Diode_SMD_AKL:D_SOD-323_TVS, F.Cu at (337.4, 178.0)
- added D43: PESD5V0S1BA, PCM_Diode_SMD_AKL:D_SOD-323_TVS, F.Cu at (337.4, 181.1)
- added D44: PESD5V0S1BA, PCM_Diode_SMD_AKL:D_SOD-323_TVS, F.Cu at (337.4, 184.2)
- added D45: PESD5V0S1BA, PCM_Diode_SMD_AKL:D_SOD-323_TVS, F.Cu at (342.0, 165.5)
- added D46: PESD5V0S1BA, PCM_Diode_SMD_AKL:D_SOD-323_TVS, F.Cu at (342.0, 168.6)
- added D47: PESD5V0S1BA, PCM_Diode_SMD_AKL:D_SOD-323_TVS, F.Cu at (342.0, 171.7)
- added D48: PESD5V0S1BA, PCM_Diode_SMD_AKL:D_SOD-323_TVS, F.Cu at (342.0, 174.8)
- added D49: PESD5V0S1BA, PCM_Diode_SMD_AKL:D_SOD-323_TVS, F.Cu at (342.0, 178.0)
- added D50: PESD5V0S1BA, PCM_Diode_SMD_AKL:D_SOD-323_TVS, F.Cu at (342.0, 181.1)
- added D51: PESD5V0S1BA, PCM_Diode_SMD_AKL:D_SOD-323_TVS, F.Cu at (342.0, 184.2)
- added D52: PESD5V0S1BA, PCM_Diode_SMD_AKL:D_SOD-323_TVS, F.Cu at (346.5, 165.5)
- added D53: SMBJ5.0CA, PCM_Diode_SMD_AKL:D_SMB_TVS, F.Cu at (326.4, 166.8)
- added D54: PESD5V0S1BA, PCM_Diode_SMD_AKL:D_SOD-323_TVS, F.Cu at (346.5, 168.6)
- added D55: SMBJ5.0CA, PCM_Diode_SMD_AKL:D_SMB_TVS, F.Cu at (326.4, 172.5)
- added D56: PESD5V0S1BA, PCM_Diode_SMD_AKL:D_SOD-323_TVS, F.Cu at (346.5, 171.7)
- added D57: SMBJ5.0CA, PCM_Diode_SMD_AKL:D_SMB_TVS, F.Cu at (326.4, 178.2)
- added D58: SMBJ5.0CA, PCM_Diode_SMD_AKL:D_SMB_TVS, F.Cu at (326.4, 183.9)
- added D59: SMBJ5.0CA, PCM_Diode_SMD_AKL:D_SMB_TVS, F.Cu at (353.9, 206.8)
- added D60: SMBJ5.0CA, PCM_Diode_SMD_AKL:D_SMB_TVS, F.Cu at (289.4, 142.8)
- added D61: SMBJ5.0CA, PCM_Diode_SMD_AKL:D_SMB_TVS, F.Cu at (289.4, 148.5)
- added J18: B-2100S40P-B110, Connector_PinSocket_2.54mm:PinSocket_2x20_P2.54mm_Horizontal, F.Cu at (189.7, 130.9)
- added R234: 100k, PCM_Resistor_SMD_AKL:R_0402_1005Metric, F.Cu at (283.6, 147.4)
- added U34: TXS0108EPW, Datasheet_Footprints:TXS0108ERGYR_VQFN-20-EP_C90706, F.Cu at (359.0, 151.4)
- C180, C188: value 1u -> 34pF; footprint Capacitor_SMD:C_0201_0603Metric_Pad0.64x0.40mm_HandSolder -> Capacitor_SMD:C_0402_1005Metric
- C181: value 34pF -> 1u; footprint Capacitor_SMD:C_0402_1005Metric -> Capacitor_SMD:C_0201_0603Metric_Pad0.64x0.40mm_HandSolder
- C185, C189, C389: value 10u -> 1u; footprint Capacitor_SMD:C_0603_1608Metric -> Capacitor_SMD:C_0201_0603Metric_Pad0.64x0.40mm_HandSolder
- C190: value 34pF -> 10u; footprint Capacitor_SMD:C_0402_1005Metric -> Capacitor_SMD:C_0603_1608Metric
- C192: value 1u -> 10u; footprint Capacitor_SMD:C_0201_0603Metric_Pad0.64x0.40mm_HandSolder -> Capacitor_SMD:C_0603_1608Metric
- C24: value 1u -> 100n
- C28: value 100n -> 1u
- C322: value 1u -> 22u; footprint Capacitor_SMD:C_0201_0603Metric_Pad0.64x0.40mm_HandSolder -> Capacitor_SMD:C_0603_1608Metric
- C324: value 22u -> 1u; footprint Capacitor_SMD:C_0603_1608Metric -> Capacitor_SMD:C_0201_0603Metric_Pad0.64x0.40mm_HandSolder
- C346: value 10u -> 22u
- C366, C377: value 22u -> 47u; footprint Capacitor_SMD:C_0603_1608Metric -> Capacitor_SMD:C_0805_2012Metric
- C367: value 47u -> 22u; footprint Capacitor_SMD:C_0805_2012Metric -> Capacitor_SMD:C_0603_1608Metric
- C387: value 47u -> 10u; footprint Capacitor_SMD:C_0805_2012Metric -> Capacitor_SMD:C_0603_1608Metric
- C390, C410: value 1u -> 2.2u; footprint Capacitor_SMD:C_0201_0603Metric_Pad0.64x0.40mm_HandSolder -> Capacitor_SMD:C_0402_1005Metric
- C394: value 2.2u -> 0.1u; footprint Capacitor_SMD:C_0402_1005Metric -> Capacitor_SMD:C_0201_0603Metric_Pad0.64x0.40mm_HandSolder
- C395: value 0.1u -> 22u; footprint Capacitor_SMD:C_0201_0603Metric_Pad0.64x0.40mm_HandSolder -> Capacitor_SMD:C_0603_1608Metric
- C397, C408: value 22u -> 2.2u; footprint Capacitor_SMD:C_0603_1608Metric -> Capacitor_SMD:C_0402_1005Metric
- C407: value 2.2u -> 22u; footprint Capacitor_SMD:C_0402_1005Metric -> Capacitor_SMD:C_0603_1608Metric
- C409, C412: value 2.2u -> 1u; footprint Capacitor_SMD:C_0402_1005Metric -> Capacitor_SMD:C_0201_0603Metric_Pad0.64x0.40mm_HandSolder
- C413: value 1u -> 10n
- C414, C416: value 10n -> 22u; footprint Capacitor_SMD:C_0201_0603Metric_Pad0.64x0.40mm_HandSolder -> Capacitor_SMD:C_0603_1608Metric
- C415: value 22u -> 10n; footprint Capacitor_SMD:C_0603_1608Metric -> Capacitor_SMD:C_0201_0603Metric_Pad0.64x0.40mm_HandSolder
- D10, D11, D12, D14, D15, D16, D17, D18, D19, D20, D5, D8, D9: value SMBJ5.0CA -> PESD5V0S1BA; footprint PCM_Diode_SMD_AKL:D_SMB_TVS -> PCM_Diode_SMD_AKL:D_SOD-323_TVS
- J20: footprint Datasheet_Footprints:RADXA_UFS_MOD_30P34P -> Datasheet_Footprints:SBC_UFS_EMMC_2x513383474
- J4: footprint Connector_PinHeader_2.54mm:PinHeader_2x10_P2.54mm_Vertical_SMD -> Connector_PinSocket_2.54mm:PinSocket_2x10_P2.54mm_Horizontal
- R176, R203: value 22R -> 10k
- R182: value 10k -> 22R
- R183: value 2.2k -> 10k
- R187: value 22R -> 2.2k
- R196, R205: value 240R -> 22R
- R197: value 100k -> 240R
- R198, R225: value 200k -> 100k
- R199: value 2.2k -> 200k
- R2: value 4.7k -> 22R
- R201, R231: value 10k -> 2.2k
- R206: value 10k -> 240R
- R207, R232: value 0R -> 10k
- R211: value 49.9k -> 0R
- R212: value 100k -> 49.9k
- R213: value 2k -> 100k
- R214: value 100k -> 2k
- R215: value 110k -> 100k
- R216: value 100k -> 110k
- R217: value 10k -> 100k
- R221: value 110k -> 10k
- R222: value 15k -> 110k
- R223: value 100k -> 15k
- R226: value 100k -> 200k
- R227: value 22R -> 100k
- R229: value 2.2k -> 22R
- R24: value 4.7k -> 8.2k
- R25: value 200R -> 8.2k
- R28: value 8.2k -> 4.7k
- R29: value 8.2k -> 200R
- R4: value 22R -> 510k
- R6: value 510k -> 4.7k
- R84, R91: value 4.7k -> 0R
- R90, R99: value 0R -> 4.7k
- U2: value W25Q128JVS -> ETA7014S2G; footprint Package_SO:SOIC-8_5.3x5.3mm_P1.27mm -> PCM_Package_TO_SOT_SMD_AKL:TSOT-23-6
- U3: value ETA7014S2G -> W25Q128JVS; footprint PCM_Package_TO_SOT_SMD_AKL:TSOT-23-6 -> Package_SO:SOIC-8_5.3x5.3mm_P1.27mm
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- renumbered J18 to J19, U45 to U41
Connections:
- net /HDMI/HDMI_CK_N renamed /HDMI/HDMI.CK_N
- net /HDMI/HDMI_CK_P renamed /HDMI/HDMI.CK_P
- net /HDMI/HDMI_D0_N renamed /HDMI/HDMI.D0_N
- net /HDMI/HDMI_D0_P renamed /HDMI/HDMI.D0_P
- net /HDMI/HDMI_D1_N renamed /HDMI/HDMI.D1_N
- net /HDMI/HDMI_D1_P renamed /HDMI/HDMI.D1_P
- net /HDMI/HDMI_D2_N renamed /HDMI/HDMI.D2_N
- net /HDMI/HDMI_D2_P renamed /HDMI/HDMI.D2_P
- net /HDMI/HDMI_TX_SBD_N renamed /HDMI/HDMI.TX_SBD_N
- net /HDMI/HDMI_TX_SBD_P renamed /HDMI/HDMI.TX_SBD_P
- net /MIPI/CSI0_RX_CLK_N renamed /MIPI/CSI1_RX_CLK_P
- net /MIPI/CSI0_RX_CLK_P renamed /MIPI/CSI1_RX_CLK_N
- net /MIPI/CSI0_RX_D0_N renamed /MIPI/CSI1_RX_D0_P
- net /MIPI/CSI0_RX_D0_P renamed /MIPI/CSI1_RX_D0_N
- net /MIPI/CSI0_RX_D1_N renamed /MIPI/CSI1_RX_D1_P
- net /MIPI/CSI0_RX_D1_P renamed /MIPI/CSI1_RX_D1_N
- net /MIPI/CSI0_RX_D2_N renamed /MIPI/CSI1_RX_D2_P
- net /MIPI/CSI0_RX_D2_P renamed /MIPI/CSI1_RX_D2_N
- net /MIPI/CSI0_RX_D3_N renamed /MIPI/CSI1_RX_D3_P
- net /MIPI/CSI0_RX_D3_P renamed /MIPI/CSI1_RX_D3_N
- net /RK3576 SOC/FSPI0_CMD/EMMC_CMD renamed /RK3576 SOC/FSPI0/EMMC.CMD
- net /RK3576 SOC/FSPI0_D0/EMMC_D0 renamed /RK3576 SOC/FSPI0/EMMC.D0
- net /RK3576 SOC/FSPI0_D1/EMMC_D1 renamed /RK3576 SOC/FSPI0/EMMC.D1
- net /RK3576 SOC/FSPI0_D2/EMMC_D2 renamed /RK3576 SOC/FSPI0/EMMC.D2
- net /RK3576 SOC/FSPI0_D3/EMMC_D3 renamed /RK3576 SOC/FSPI0/EMMC.D3
- net /RK3576 SOC/FSPI0_D4/EMMC_D4 renamed /RK3576 SOC/FSPI0/EMMC.D4
- net /RK3576 SOC/FSPI0_D5/EMMC_D5 renamed /RK3576 SOC/FSPI0/EMMC.D5
- net /RK3576 SOC/FSPI0_D6/EMMC_D6 renamed /RK3576 SOC/FSPI0/EMMC.D6
- net /RK3576 SOC/FSPI0_D7/EMMC_D7 renamed /RK3576 SOC/FSPI0/EMMC.D7
- net /RK3576 SOC/HDMI_CK_N renamed /RK3576 SOC/HDMI.CK_N
- net /RK3576 SOC/HDMI_CK_P renamed /RK3576 SOC/HDMI.CK_P
- net /RK3576 SOC/HDMI_D0_N renamed /RK3576 SOC/HDMI.D0_N
- net /RK3576 SOC/HDMI_D0_P renamed /RK3576 SOC/HDMI.D0_P
- net /RK3576 SOC/HDMI_D1_N renamed /RK3576 SOC/HDMI.D1_N
- net /RK3576 SOC/HDMI_D1_P renamed /RK3576 SOC/HDMI.D1_P
- net /RK3576 SOC/HDMI_D2_N renamed /RK3576 SOC/HDMI.D2_N
- net /RK3576 SOC/HDMI_D2_P renamed /RK3576 SOC/HDMI.D2_P
- net /RK3576 SOC/HDMI_TX_SBD_N renamed /RK3576 SOC/HDMI.TX_SBD_N
- net /RK3576 SOC/HDMI_TX_SBD_P renamed /RK3576 SOC/HDMI.TX_SBD_P
- net /RK3576 SOC/SAI2_LRCK_M0 renamed /RK3576 SOC/SAI2.LRCK_M0
- net /RK3576 SOC/SAI2_SCLK_M0 renamed /RK3576 SOC/SAI2.SCLK_M0
- net /RK3576 SOC/SAI2_SDI_M0 renamed /RK3576 SOC/SAI2.SDI_M0
- net /RK3576 SOC/SAI2_SDO_M0 renamed /RK3576 SOC/SAI2.SDO_M0
- net /RK3576 SOC/SDMMC1_D0_M0 renamed /RK3576 SOC/SDMMC1.D0_M0
- net /RK3576 SOC/SDMMC1_D1_M0 renamed /RK3576 SOC/SDMMC1.D1_M0
- net /RK3576 SOC/SDMMC1_D2_M0 renamed /RK3576 SOC/SDMMC1.D2_M0
- net /RK3576 SOC/SDMMC1_D3_M0 renamed /RK3576 SOC/SDMMC1.D3_M0
- net /RK3576 SOC/UART4_CTSN_M1 renamed /RK3576 SOC/UART4.CTSN_M1
- net /RK3576 SOC/UART4_RTSN_M1 renamed /RK3576 SOC/UART4.RTSN_M1
- net /RK3576 SOC/UART4_RX_M1 renamed /RK3576 SOC/UART4.RX_M1
- net /RK3576 SOC/UART4_TX_M1 renamed /RK3576 SOC/UART4.TX_M1
- net /RK3576 SOC/USB_{HUB}_SSRX1_N renamed /RK3576 SOC/USB_{HUB}.SSRX1_N
- net /RK3576 SOC/USB_{HUB}_SSRX1_P renamed /RK3576 SOC/USB_{HUB}.SSRX1_P
- net /RK3576 SOC/USB_{HUB}_SSTX1_N renamed /RK3576 SOC/USB_{HUB}.SSTX1_N
- net /RK3576 SOC/USB_{HUB}_SSTX1_P renamed /RK3576 SOC/USB_{HUB}.SSTX1_P
- net /RK3576 SOC/USB_{SOC}_AUX_N renamed /RK3576 SOC/USB_{SOC}.AUX_N
- net /RK3576 SOC/USB_{SOC}_AUX_P renamed /RK3576 SOC/USB_{SOC}.AUX_P
- net /RK3576 SOC/USB_{SOC}_RX1_N renamed /RK3576 SOC/USB_{SOC}.RX1_N
- net /RK3576 SOC/USB_{SOC}_RX1_P renamed /RK3576 SOC/USB_{SOC}.RX1_P
- net /RK3576 SOC/USB_{SOC}_RX2_N renamed /RK3576 SOC/USB_{SOC}.RX2_N
- net /RK3576 SOC/USB_{SOC}_RX2_P renamed /RK3576 SOC/USB_{SOC}.RX2_P
- net /RK3576 SOC/USB_{SOC}_TX1_N renamed /RK3576 SOC/USB_{SOC}.TX1_N
- net /RK3576 SOC/USB_{SOC}_TX1_P renamed /RK3576 SOC/USB_{SOC}.TX1_P
- net /RK3576 SOC/USB_{SOC}_TX2_N renamed /RK3576 SOC/USB_{SOC}.TX2_N
- net /RK3576 SOC/USB_{SOC}_TX2_P renamed /RK3576 SOC/USB_{SOC}.TX2_P
- net /RK3576 SOC/uSD_CLK renamed /RK3576 SOC/uSD.CLK
- net /RK3576 SOC/uSD_CMD renamed /RK3576 SOC/uSD.CMD
- net /RK3576 SOC/uSD_D0 renamed /RK3576 SOC/uSD.D0
- net /RK3576 SOC/uSD_D1 renamed /RK3576 SOC/uSD.D1
- net /RK3576 SOC/uSD_D2 renamed /RK3576 SOC/uSD.D2
- net /RK3576 SOC/uSD_D3 renamed /RK3576 SOC/uSD.D3
- net /UFS\eMMC/FSPI0_CMD/EMMC_CMD renamed /UFS\eMMC/FSPI0/EMMC.CMD
- net /UFS\eMMC/FSPI0_D0/EMMC_D0 renamed /UFS\eMMC/FSPI0/EMMC.D0
- net /UFS\eMMC/FSPI0_D1/EMMC_D1 renamed /UFS\eMMC/FSPI0/EMMC.D1
- net /UFS\eMMC/FSPI0_D2/EMMC_D2 renamed /UFS\eMMC/FSPI0/EMMC.D2
- net /UFS\eMMC/FSPI0_D3/EMMC_D3 renamed /UFS\eMMC/FSPI0/EMMC.D3
- net /UFS\eMMC/FSPI0_D4/EMMC_D4 renamed /UFS\eMMC/FSPI0/EMMC.D4
- net /UFS\eMMC/FSPI0_D5/EMMC_D5 renamed /UFS\eMMC/FSPI0/EMMC.D5
- net /UFS\eMMC/FSPI0_D6/EMMC_D6 renamed /UFS\eMMC/FSPI0/EMMC.D6
- net /UFS\eMMC/FSPI0_D7/EMMC_D7 renamed /UFS\eMMC/FSPI0/EMMC.D7
- net /USB-A Host/USB_{HUB}_SSRX1_N renamed /USB-A Host/USB_{HUB}.SSRX1_N
- net /USB-A Host/USB_{HUB}_SSRX1_P renamed /USB-A Host/USB_{HUB}.SSRX1_P
- net /USB-A Host/USB_{HUB}_SSTX1_N renamed /USB-A Host/USB_{HUB}.SSTX1_N
- net /USB-A Host/USB_{HUB}_SSTX1_P renamed /USB-A Host/USB_{HUB}.SSTX1_P
- net /USB-C SOC/USB_{SOC}_AUX_N renamed /USB-C SOC/USB_{SOC}.AUX_N
- net /USB-C SOC/USB_{SOC}_AUX_P renamed /USB-C SOC/USB_{SOC}.AUX_P
- net /USB-C SOC/USB_{SOC}_RX1_N renamed /USB-C SOC/USB_{SOC}.RX1_N
- net /USB-C SOC/USB_{SOC}_RX1_P renamed /USB-C SOC/USB_{SOC}.RX1_P
- net /USB-C SOC/USB_{SOC}_RX2_N renamed /USB-C SOC/USB_{SOC}.RX2_N
- net /USB-C SOC/USB_{SOC}_RX2_P renamed /USB-C SOC/USB_{SOC}.RX2_P
- net /USB-C SOC/USB_{SOC}_TX1_N renamed /USB-C SOC/USB_{SOC}.TX1_N
- net /USB-C SOC/USB_{SOC}_TX1_P renamed /USB-C SOC/USB_{SOC}.TX1_P
- net /USB-C SOC/USB_{SOC}_TX2_N renamed /USB-C SOC/USB_{SOC}.TX2_N
- net /USB-C SOC/USB_{SOC}_TX2_P renamed /USB-C SOC/USB_{SOC}.TX2_P
- net /Wireless/SAI2_LRCK_M0 renamed /Wireless/SAI2.LRCK_M0
- net /Wireless/SAI2_SCLK_M0 renamed /Wireless/SAI2.SCLK_M0
- net /Wireless/SAI2_SDI_M0 renamed /Wireless/SAI2.SDI_M0
- net /Wireless/SAI2_SDO_M0 renamed /Wireless/SAI2.SDO_M0
- net /Wireless/SDMMC1_CLK_M0 renamed /Wireless/SDMMC1.D3_M0
- net /Wireless/SDMMC1_D1_M0 renamed /Wireless/SDMMC1.D0_M0
- net /Wireless/SDMMC1_D2_M0 renamed /Wireless/SDMMC1.D1_M0
- net /Wireless/SDMMC1_D3_M0 renamed /Wireless/SDMMC1.D2_M0
- net /Wireless/UART4_CTSN_M1 renamed /Wireless/UART4.CTSN_M1
- net /Wireless/UART4_RTSN_M1 renamed /Wireless/UART4.RTSN_M1
- net /Wireless/UART4_RX_M1 renamed /Wireless/UART4.RX_M1
- net /Wireless/UART4_TX_M1 renamed /Wireless/UART4.TX_M1
- net /uSD Card/uSD_CLK renamed /uSD Card/uSD.CLK
- net /uSD Card/uSD_CMD renamed /uSD Card/uSD.CMD
- net /uSD Card/uSD_D0 renamed /uSD Card/uSD.D0
- net /uSD Card/uSD_D1 renamed /uSD Card/uSD.D1
- net /uSD Card/uSD_D2 renamed /uSD Card/uSD.D2
- net /uSD Card/uSD_D3 renamed /uSD Card/uSD.D3
- C114 pad 1: Net-(U3-VCC) -> Net-(U2-VCC)
- C180 pad 1: VCC5V0_SYS -> /USB-A Host/Crystal_{HUB}_OUT
- C181 pad 1: /USB-A Host/Crystal_{HUB}_OUT -> VCC_{HUB}_1V2_S0
- C182 pad 1: VCC_{HUB}_1V2_S0 -> +3.3V
- C183 pad 1: +3.3V -> VCC_{HUB}_1V2_S0
- C185 pad 1: VCC5V0_SYS -> +3.3V
- C187 pad 1: +3.3V -> VCC5V0_SYS
- C188 pad 1: VCC_{HUB}_1V2_S0 -> /USB-A Host/Crystal_{HUB}_IN
- C189 pad 1: VCC5V0_SYS -> VCC_{HUB}_1V2_S0
- C190 pad 1: /USB-A Host/Crystal_{HUB}_IN -> VCC5V0_SYS
- C192 pad 1: VCC_{HUB}_1V2_S0 -> VCC5V0_SYS
- C205 pad 1: /Ethernet/ETH1_{PHY}_RESET -> /Ethernet/ETH1_{PHY}_nRST
- C206 pad 1: /Ethernet/ETH0_{PHY}_RESET -> /Ethernet/ETH0_{PHY}_nRST
- C21 pad 1: VCC_3.3v_S0 -> VCCA_1V8_S3
- C22 pad 1: VCCA_1V8_S3 -> VDD_CPU_LIT_S0
- C23 pad 1: VDD_CPU_LIT_S0 -> VDD_LOGIC_S0
- C24 pad 1: VDD_LOGIC_S0 -> VDD_NPU_S0
- C246 pad 2: /PCIe/PCIE0_RX_N -> /PCIe/PCIE0.RX_N
- C247 pad 2: /PCIe/PCIE0_RX_P -> /PCIe/PCIE0.RX_P
- C25 pad 1: VDD_NPU_S0 -> VDD_CPU_LIT_S0
- C253 pad 1: VCC_1V8_S3 -> VCCA_1V8_S0
- C258 pad 1: VCC_1V8_S3 -> VCCA_1V8_S0
- C259 pad 1: VCC_1V8_S3 -> VCCA_1V8_S0
- C26 pad 1: VDD_CPU_LIT_S0 -> VDD_LOGIC_S0
- C27 pad 1: VDD_LOGIC_S0 -> VDD_NPU_S0
- C28 pad 1: VDD_NPU_S0 -> VCC_3.3v_S0
- C282 pad 1: VCC_1V8_S3 -> VCCA_1V8_S0
- C285 pad 1: VCC_1V8_S3 -> VCCA_1V8_S0
- C288 pad 1: VCC_1V8_S3 -> VCCA_1V8_S0
- C291 pad 1: VCC_1V8_S3 -> VCCA_1V8_S0
- C322 pad 1: VDD2_DDR_S3 -> VCC5V0_SYS
- C324 pad 1: VCC5V0_SYS -> VDD2_DDR_S3
- C345 pad 1: /OLED Screen/OLED_LED -> /OLED Screen/OLED.LED
- C346 pad 1: /OLED Screen/OLED_LED -> VCC5V0_SYS
- C356 pad 1: VCC5V0_SYS -> VDD_CPU_BIG_S0
- C357 pad 1: VDD_CPU_BIG_S0 -> VDD_NPU_S0
- C358 pad 1: VDD_NPU_S0 -> VDD_CPU_LIT_S0
- C359 pad 1: VDD_CPU_LIT_S0 -> VCC_3V3_S0
- C360 pad 1: VCC_3V3_S0 -> VDD_GPU_S0
- C361 pad 1: VDD_GPU_S0 -> VDDQ_DDR_S0
- C361 pad 2: GND -> Net-(C361-Pad2)
- C362 pad 1: VDDQ_DDR_S0 -> VDD_LOGIC_S0
- C363 pad 1: VDD_LOGIC_S0 -> VCCA_1V8_S0
- C364 pad 1: VCC_1V8_S3 -> VDD2_DDR_S3
- C365 pad 1: VDD2_DDR_S3 -> VDD_DDR_S0
- C366 pad 1: VDD_DDR_S0 -> VCC5V0_SYS
- C366 pad 2: Net-(C366-Pad2) -> GND
- C367 pad 1: VCC5V0_SYS -> VDD_CPU_BIG_S0
- C368 pad 1: VDD_CPU_BIG_S0 -> VDD_NPU_S0
- C369 pad 1: VDD_NPU_S0 -> VDD_CPU_LIT_S0
- C370 pad 1: VDD_CPU_LIT_S0 -> VCC_3V3_S0
- C371 pad 1: VCC_3V3_S0 -> VDD_GPU_S0
- C372 pad 1: VDD_GPU_S0 -> VDDQ_DDR_S0
- C372 pad 2: GND -> Net-(C361-Pad2)
- C373 pad 1: VDDQ_DDR_S0 -> VDD_LOGIC_S0
- C374 pad 1: VDD_LOGIC_S0 -> VCCA_1V8_S0
- C375 pad 1: VCC_1V8_S3 -> VDD2_DDR_S3
- C376 pad 1: VDD2_DDR_S3 -> VDD_DDR_S0
- C377 pad 1: VDD_DDR_S0 -> VDD_CPU_BIG_S0
- C377 pad 2: Net-(C366-Pad2) -> GND
- C378 pad 1: VDD_CPU_BIG_S0 -> VDD_NPU_S0
- C379 pad 1: VDD_NPU_S0 -> VDD_CPU_LIT_S0
- C380 pad 1: VDD_CPU_LIT_S0 -> VCC_3V3_S0
- C381 pad 1: VCC_3V3_S0 -> VDD_GPU_S0
- C382 pad 1: VDD_GPU_S0 -> VDDQ_DDR_S0
- C382 pad 2: GND -> Net-(C361-Pad2)
- C383 pad 1: VDDQ_DDR_S0 -> VDD_LOGIC_S0
- C384 pad 1: VDD_LOGIC_S0 -> VCCA_1V8_S0
- C385 pad 1: VCC_1V8_S3 -> VDD2_DDR_S3
- C386 pad 1: VDD2_DDR_S3 -> VDD_DDR_S0
- C387 pad 1: VDD_DDR_S0 -> VCC5V0_SYS
- C387 pad 2: Net-(C366-Pad2) -> GND
- C389 pad 1: VCC5V0_SYS -> Net-(U43-VCC)
- C390 pad 1: Net-(U43-VCC) -> VCC_2V0_PLDO_S3
- C391 pad 1: VCC_2V0_PLDO_S3 -> VCC5V0_SYS
- C392 pad 1: VCC5V0_SYS -> VCC_2V0_PLDO_S3
- C394 pad 1: VCC_2V0_PLDO_S3 -> Net-(C394-Pad1)
- C394 pad 2: GND -> Net-(U43-BS)
- C395 pad 1: Net-(C395-Pad1) -> VCC5V0_SYS
- C395 pad 2: Net-(U43-BS) -> GND
- C397 pad 1: VCC5V0_SYS -> VCCA_1V8_S0
- C398 pad 1: VCCA_1V8_S0 -> VCCA1V8_PLDO2_S0
- C399 pad 1: VCCA1V8_PLDO2_S0 -> VDDA_1V2_S0
- C400 pad 1: VDDA_1V2_S0 -> +3.3V
- C401 pad 1: +3.3V -> VCCIO_SD_S0
- C402 pad 1: VCCIO_SD_S0 -> VDD_0V75_S3
- C403 pad 1: VDD_0V75_S3 -> VDDA_DDR_PLL_S0
- C404 pad 1: VDDA_DDR_PLL_S0 -> VDDA0V75_HDMI_S0
- C405 pad 1: VDDA0V75_HDMI_S0 -> VDDA_0V85_S0
- C406 pad 1: VDDA_0V85_S0 -> VDDA_0V75_S0
- C407 pad 1: VDDA_0V75_S0 -> VCC5V0_SYS
- C410 pad 1: VCC5V0_SYS -> VCCA1V8_PLDO6_S3
- C411 pad 1: VCCA1V8_PLDO6_S3 -> VCC5V0_SYS
- C412 pad 1: VCC5V0_SYS -> Net-(U42C-VDC)
- C413 pad 1: Net-(U42C-VDC) -> Net-(U42C-~{RESETB})
- C414 pad 1: Net-(U42C-PWRON) -> VCC_2V0_PLDO_S3
- C415 pad 1: VCC_2V0_PLDO_S3 -> Net-(U42C-PWRON)
- C416 pad 1: Net-(U42C-PWRON) -> VCC_2V0_PLDO_S3
- C89 pad 1: VCCA_1V8_S0 -> VDDA_0V85_S0
- C91 pad 1: VDDA_0V85_S0 -> VCCA_1V8_S0
- D10 pad 2: Vbus_USB_{HOST3} -> /RP2350A MCU/ADC1_{MCU}
- D11 pad 1: GND -> Net-(D11-K)
- D11 pad 2: Vbus_USB_{HOST4} -> VCC_{GPIO}_3V3_S0
- D12 pad 2: VCC_{HDMI}_5V_S0 -> /RP2350A MCU/ADC0_{MCU}
- D13 pad 1: GND -> Net-(D11-K)
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Routing:
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Other:
- board text removed: "USB"
