File: RTC.kicad_sch (KiCad schematic)
At the start: 15 parts, among them Q7 AO3401A, U16 M24C64-RMN6TP, U32 RV-3028-C7

Commit message: Replace v2 with updated RK3576_SBCv2 (Copy) Oct 2
- Update 18 sheets to Oct 2 15:37 local versions
- Keep cleaned layout: exclude .history/, Resources/, *.bak, *.lck,
  project.kicad_dru, .hs_rules.json, lowercase dup placeholders
  (fixtures/power), empty orphans (digital, mechanical, output,
  USBC_MCU, eMMC_UFS)
- Preserve LICENSE, README.md, .gitignore
Parts:
- R163, R250: LCSC Part C114765 -> C106231; Mouser Part 603-RC0402FR-0722RL -> 603-RC0402FR-070RL
Connections:
- net I2C2_SCL_M0_CC_RTC_EEPROM renamed I2C8_SCL_M3_RTC_EEPROM
- net I2C2_SDA_M0_CC_RTC_EEPROM renamed I2C8_SDA_M3_RTC_EEPROM
Changed lines of the file:
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@@
 		)
 	)
-	(label "I2C2_SDA_M0_CC_RTC_EEPROM"
-		(at 74.93 109.22 180)
+	(label "I2C8_SCL_M3_RTC_EEPROM"
+		(at 31.75 73.66 0)
 		(effects
 			(font
 				(size 1.016 1.016)
 			)
-			(justify right bottom)
+			(justify left bottom)
 		)
 	)
@@
 		)
 	)
-	(label "RTC_32KOUT_WIFI"
-		(at 158.75 83.82 180)
+	(label "I2C8_SCL_M3_RTC_EEPROM"
+		(at 74.93 111.76 180)
 		(effects
 			(font
 				(size 1.016 1.016)
-				(thickness 0.127)
 			)
 			(justify right bottom)
 		)
 	)
-	(label "I2C2_SCL_M0_CC_RTC_EEPROM"
-		(at 31.75 73.66 0)
+	(label "RTC_32KOUT_WIFI"
+		(at 158.75 83.82 180)
 		(effects
 			(font
 				(size 1.016 1.016)
+				(thickness 0.127)
 			)
-			(justify left bottom)
+			(justify right bottom)
 		)
 	)
-	(label "I2C2_SCL_M0_CC_RTC_EEPROM"
-		(at 74.93 111.76 180)
+	(label "I2C8_SDA_M3_RTC_EEPROM"
+		(at 31.75 76.2 0)
 		(effects
 			(font
 				(size 1.016 1.016)
 			)
-			(justify right bottom)
+			(justify left bottom)
 		)
 	)
@@
 		)
 	)
-	(label "RTC_32KOUT_SOC"
-		(at 158.75 80.01 180)
+	(label "I2C8_SDA_M3_RTC_EEPROM"
+		(at 74.93 109.22 180)
 		(effects
 			(font
 				(size 1.016 1.016)
-				(thickness 0.127)
 			)
 			(justify right bottom)
 		)
 	)
-	(label "I2C2_SDA_M0_CC_RTC_EEPROM"
-		(at 31.75 76.2 0)
+	(label "RTC_32KOUT_SOC"
+		(at 158.75 80.01 180)
 		(effects
 			(font
 				(size 1.016 1.016)
+				(thickness 0.127)
 			)
-			(justify left bottom)
+			(justify right bottom)
 		)
 	)
@@
 		(polyline
 			(pts
-				(xy 55.88 70.485) (xy 29.21 70.485) (xy 29.21 79.375) (xy 55.88 79.375)
+				(xy 53.34 70.485) (xy 29.21 70.485) (xy 29.21 79.375) (xy 53.34 79.375)
 			)
 			(stroke
@@
 			)
 		)
+		(property "Sim.Library" ""
+			(at 125.73 50.8 90)
+			(hide yes)
+			(show_name no)
+			(do_not_autoplace no)
+			(effects
+				(font
+					(size 1.27 1.27)
+				)
+			)
+		)
 		(pin "3"
 		)
@@
 			)
 		)
+		(property "Sim.Library" ""
+			(at 97.79 50.8 0)
+			(hide yes)
+			(show_name no)
+			(do_not_autoplace no)
+			(effects
+				(font
+					(size 1.27 1.27)
+				)
+			)
+		)
 		(pin "1"
 		)
@@
 			)
 		)
+		(property "Sim.Library" ""
+			(at 133.35 53.34 90)
+			(hide yes)
+			(show_name no)
+			(do_not_autoplace no)
+			(effects
+				(font
+					(size 1.27 1.27)
+				)
+			)
+		)
 		(pin "2"
 		)
@@
 			)
 		)
+		(property "Sim.Library" ""
+			(at 39.37 111.76 0)
+			(hide yes)
+			(show_name no)
+			(do_not_autoplace no)
+			(effects
+				(font
+					(size 1.27 1.27)
+				)
+			)
+		)
 		(pin "6"
 		)
@@
 			)
 		)
+		(property "Sim.Library" ""
+			(at 144.78 48.26 0)
+			(hide yes)
+			(show_name no)
+			(do_not_autoplace no)
+			(effects
+				(font
+					(size 1.27 1.27)
+				)
+			)
+		)
 		(pin "1"
 		)
@@
 			)
 		)
+		(property "Sim.Library" ""
+			(at 92.71 78.74 0)
+			(hide yes)
+			(show_name no)
+			(do_not_autoplace no)
+			(effects
+				(font
+					(size 1.27 1.27)
+				)
+			)
+		)
 		(pin "1"
 		)
@@
 			)
 		)
+		(property "Sim.Library" ""
+			(at 30.48 97.79 0)
+			(hide yes)
+			(show_name no)
+			(do_not_autoplace no)
+			(effects
+				(font
+					(size 1.27 1.27)
+				)
+			)
+		)
 		(pin "1"
 		)
@@
 			)
 		)
+		(property "Sim.Library" ""
+			(at 66.04 60.96 0)
+			(hide yes)
+			(show_name no)
+			(do_not_autoplace no)
+			(effects
+				(font
+					(size 1.27 1.27)
+				)
+			)
+		)
 		(pin "1"
 		)
@@
 			)
 		)
-		(property "LCSC Part" "C114765"
+		(property "LCSC Part" "C106231"
 			(at 133.35 83.82 90)
 			(hide yes)
@@
 			)
 		)
-		(property "Mouser Part" "603-RC0402FR-0722RL "
+		(property "Mouser Part" "603-RC0402FR-070RL"
+			(at 133.35 83.82 90)
+			(hide yes)
+			(show_name no)
+			(do_not_autoplace no)
+			(effects
+				(font
+					(size 1.27 1.27)
+				)
+			)
+		)
+		(property "Sim.Library" ""
 			(at 133.35 83.82 90)
 			(hide yes)
@@
 			)
 		)
+		(property "Sim.Library" ""
+			(at 154.94 53.34 0)
+			(hide yes)
+			(show_name no)
+			(do_not_autoplace no)
+			(effects
+				(font
+					(size 1.27 1.27)
+				)
+			)
+		)
 		(pin "2"
 		)
@@
 			)
 		)
-		(property "LCSC Part" "C114765"
+		(property "LCSC Part" "C106231"
 			(at 133.35 80.01 90)
 			(hide yes)
@@
 			)
 		)
-		(property "Mouser Part" "603-RC0402FR-0722RL "
+		(property "Mouser Part" "603-RC0402FR-070RL"
+			(at 133.35 80.01 90)
+			(hide yes)
+			(show_name no)
+			(do_not_autoplace no)
+			(effects
+				(font
+					(size 1.27 1.27)
+				)
+			)
+		)
+		(property "Sim.Library" ""
 			(at 133.35 80.01 90)
 			(hide yes)
@@
 			)
 		)
+		(property "Sim.Library" ""
+			(at 124.46 57.15 0)
+			(hide yes)
+			(show_name no)
+			(do_not_autoplace no)
+			(effects
+				(font
+					(size 1.27 1.27)
+				)
+			)
+		)
 		(pin "1"
 		)
@@
 			)
 		)
+		(property "Sim.Library" ""
+			(at 80.01 50.8 0)
+			(hide yes)
+			(show_name no)
+			(do_not_autoplace no)
+			(effects
+				(font
+					(size 1.27 1.27)
+				)
+			)
+		)
 		(pin "1"
 		)
@@
 			)
 		)
+		(property "Sim.Library" ""
+			(at 111.76 69.85 0)
+			(hide yes)
+			(show_name no)
+			(do_not_autoplace no)
+			(effects
+				(font
+					(size 1.27 1.27)
+				)
+			)
+		)
 		(pin "1"
 		)
@@
 			(at 58.42 60.96 0)
 			(hide yes)
+			(show_name no)
+			(do_not_autoplace no)
+			(effects
+				(font
+					(size 1.27 1.27)
+				)
+			)
+		)
+		(property "Sim.Library" ""
+			(at 58.42 60.96 0)
+			(hide yes)

Commit message: Relink hierarchical root: 18 sheets into RK3576 SBCv2 top level
Root was empty (no sheet boxes); all subsheets orphaned.
Rebuilt A1 top level linking RK3576, LPDDR5, Power, Ethernet,
HDMI, MIPI, PCIe, USB-A/C, Wireless, RTC, uSD, GPIO, OLED,
RP2350A, Connectors, Fixtures, DC_Power. block_diagrame kept
docs-only (unlinked, avoids double-instantiation). Lowercase
stub duplicates excluded. ERC: 1388 -> 770 violations.
Parts:
- renumbered C232 to C340, C370 to C341, C371 to C342, D20 to D19, F3 to F1, Q7 to Q6, R159 to R199, R160 to R200, R161 to R201, R162 to R202, R163 to R203, R250 to R204, U16 to U39, U32 to U40

Commit message: block diagrame with Hierarchical labels and NVMe SSD footprint
Parts:
- renumbered D19 to D59, R199 to R200, R200 to R201, R201 to R202, R202 to R203, R203 to R204, R204 to R205
Other:
- moved on the sheet: BT1, C340, C341, C342, D59, F1, Q6, R200, R201, R202, R203, R204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
