File: USBC_SOC.kicad_sch (KiCad schematic)
At the start: 37 parts, among them J2 USB_C_Receptacle, U2 TPS22953DQCR, U39 ICMEF112P900MFR, U5 FUSB302BMPX, U6 TPD4E05U06DQAR, U7 TPD4E05U06DQAR, U8 TPD4E05U06DQAR

Commit message: Replace v2 with updated RK3576_SBCv2 (Copy) Oct 2
- Update 18 sheets to Oct 2 15:37 local versions
- Keep cleaned layout: exclude .history/, Resources/, *.bak, *.lck,
  project.kicad_dru, .hs_rules.json, lowercase dup placeholders
  (fixtures/power), empty orphans (digital, mechanical, output,
  USBC_MCU, eMMC_UFS)
- Preserve LICENSE, README.md, .gitignore
Parts:
- C177, C178: footprint Capacitor_SMD:C_0402_1005Metric_Pad0.74x0.62mm_HandSolder -> Capacitor_SMD:C_0402_1005Metric
- C200: LCSC Part C5209398 -> (none); Mouser Part CL03A105KP3NSNC -> (none)
- R45: LCSC Part C105871 -> C60490; Mouser Part 603-RC0402FR-074K7L -> 603-RC0402FR-0710KL
Connections:
- net GND is gone; now on net EP: C171.2, C172.2, C174.2, C175.2, C176.2, C177.2, C178.2, C200.2, D11.1 (K), D8.1 (K), D9.1 (K), J2.A1 (GND), J2.A12 (GND), J2.B1 (GND), J2.B12 (GND), R45.2, R46.2, R47.2, R50.2, R53.2, U2.5 (GND), U39.5 (GND), U39.6 (GND), U5.15 (GND), U5.8 (GND), U5.9 (GND), U6.3 (GND), U6.8 (GND), U7.3 (GND), U7.8 (GND), U8.3 (GND), U8.8 (GND)
- net I2C0_SCL_M1_TP renamed I2C2_SCL_M0_USB_Wireless
- net I2C0_SDA_M1_TP renamed I2C2_SDA_M0_USB_Wireless
Other:
- moved on the sheet: U2

Commit message: Relink hierarchical root: 18 sheets into RK3576 SBCv2 top level
Root was empty (no sheet boxes); all subsheets orphaned.
Rebuilt A1 top level linking RK3576, LPDDR5, Power, Ethernet,
HDMI, MIPI, PCIe, USB-A/C, Wireless, RTC, uSD, GPIO, OLED,
RP2350A, Connectors, Fixtures, DC_Power. block_diagrame kept
docs-only (unlinked, avoids double-instantiation). Lowercase
stub duplicates excluded. ERC: 1388 -> 770 violations.
Parts:
- removed J2: USB_C_Receptacle, Datasheet_Footprints:USB-C-SMD-24P_GT-USB-7092B, symbol Connector:USB_C_Receptacle
- added J5: USB_C_Receptacle, Datasheet_Footprints:USB-C-SMD_GT-USB-7092B, symbol Connector:USB_C_Receptacle
- renumbered C179 to C131, C180 to C132, C181 to C133, C182 to C134, C183 to C135, C184 to C136, C185 to C137, C186 to C138, C187 to C139, C188 to C140, C172 to C141, C200 to C142, C177 to C143, C178 to C144, C174 to C145, C175 to C146, C176 to C147, C171 to C148, D11 to D5, D8 to D6, D9 to D7, R50 to R47, R46 to R48, R47 to R49, R48 to R50, R49 to R51, R44 to R52, R45 to R53, R53 to R54, R81 to R55, U8 to U10, U39 to U5, U2 to U6, U5 to U7, U6 to U8, U7 to U9
Connections:
- net CUSB_{SOC}_AUX_N: now also J5.B8 (SBU2)
- net CUSB_{SOC}_AUX_P: now also J5.A8 (SBU1)
- net CUSB_{SOC}_D_N: now also J5.A7 (D-), J5.B7 (D-)
- net CUSB_{SOC}_D_P: now also J5.A6 (D+), J5.B6 (D+)
- net CUSB_{SOC}_RX1_N: now also J5.B10 (RX1-)
- net CUSB_{SOC}_RX1_P: now also J5.B11 (RX1+)
- net CUSB_{SOC}_RX2_N: now also J5.A10 (RX2-)
- net CUSB_{SOC}_RX2_P: now also J5.A11 (RX2+)
- net CUSB_{SOC}_TX1_N: now also J5.A3 (TX1-)
- net CUSB_{SOC}_TX1_P: now also J5.A2 (TX1+)
- net CUSB_{SOC}_TX2_N: now also J5.B3 (TX2-)
- net CUSB_{SOC}_TX2_P: now also J5.B2 (TX2+)
- net EP: now also J5.A1 (GND), J5.A12 (GND), J5.B1 (GND), J5.B12 (GND)
- net USB_{SOC}_CC1: now also J5.A5 (CC1)
- net USB_{SOC}_CC2: now also J5.B5 (CC2)
- net Vbus_USB_{OTG}: now also J5.A4 (VBUS), J5.A9 (VBUS), J5.B4 (VBUS), J5.B9 (VBUS)
- net at R47.1: now also J5.SH (SHIELD)

Commit message: block diagrame with Hierarchical labels and NVMe SSD footprint
Parts:
- renumbered D5 to D21, D6 to D22, D7 to D23
Connections:
- net CUSB_{SOC}_AUX_N: now also U10.6 (NC)
- net CUSB_{SOC}_AUX_P: now also U10.7 (NC)
- net CUSB_{SOC}_D_N: now also U8.10 (NC)
- net CUSB_{SOC}_D_P: now also U8.9 (NC)
- net CUSB_{SOC}_RX1_N: now also U8.7 (NC)
- net CUSB_{SOC}_RX1_P: now also U8.6 (NC)
- net CUSB_{SOC}_RX2_N: now also U9.7 (NC)
- net CUSB_{SOC}_RX2_P: now also U9.6 (NC)
- net CUSB_{SOC}_TX1_N: now also U9.10 (NC)
- net CUSB_{SOC}_TX1_P: now also U9.9 (NC)
- net CUSB_{SOC}_TX2_N: now also U10.10 (NC)
- net CUSB_{SOC}_TX2_P: now also U10.9 (NC)
- net USB_{SOC}_AUX_N renamed USB_{SOC}.AUX_N
- net USB_{SOC}_AUX_P renamed USB_{SOC}.AUX_P
- net USB_{SOC}_D_N renamed USB_{SOC}.D_N
- net USB_{SOC}_D_P renamed USB_{SOC}.D_P
- net USB_{SOC}_PUPDCTRL1 renamed USB_{SOC}.PUPDCTRL1
- net USB_{SOC}_PUPDCTRL2 renamed USB_{SOC}.PUPDCTRL2
- net USB_{SOC}_RX1_N renamed USB_{SOC}.RX1_N
- net USB_{SOC}_RX1_P renamed USB_{SOC}.RX1_P
- net USB_{SOC}_RX2_N renamed USB_{SOC}.RX2_N
- net USB_{SOC}_RX2_P renamed USB_{SOC}.RX2_P
- net USB_{SOC}_TX1_N renamed USB_{SOC}.TX1_N
- net USB_{SOC}_TX1_P renamed USB_{SOC}.TX1_P
- net USB_{SOC}_TX2_N renamed USB_{SOC}.TX2_N
- net USB_{SOC}_TX2_P renamed USB_{SOC}.TX2_P
- no-connect marks 13 -> 1
Other:
- moved on the sheet: C141, C148
