File: uSD_Card.kicad_sch (KiCad schematic)
At the start: 25 parts, among them J23 TF PUSH, U27 AP2553W6-7, U30 TPD4E05U06DQAR, U31 TPD4E05U06DQAR

Commit message: Replace v2 with updated RK3576_SBCv2 (Copy) Oct 2
- Update 18 sheets to Oct 2 15:37 local versions
- Keep cleaned layout: exclude .history/, Resources/, *.bak, *.lck,
  project.kicad_dru, .hs_rules.json, lowercase dup placeholders
  (fixtures/power), empty orphans (digital, mechanical, output,
  USBC_MCU, eMMC_UFS)
- Preserve LICENSE, README.md, .gitignore
Parts:
- R122: LCSC Part C60491 -> C60490; Mouser Part 603-RC0402FR-07100KL -> 603-RC0402FR-0710KL
- R275, R276, R277, R278, R279, R280, R281: LCSC Part C114765 -> C106231; Mouser Part 603-RC0402FR-0722RL -> 603-RC0402FR-070RL

Commit message: Relink hierarchical root: 18 sheets into RK3576 SBCv2 top level
Root was empty (no sheet boxes); all subsheets orphaned.
Rebuilt A1 top level linking RK3576, LPDDR5, Power, Ethernet,
HDMI, MIPI, PCIe, USB-A/C, Wireless, RTC, uSD, GPIO, OLED,
RP2350A, Connectors, Fixtures, DC_Power. block_diagrame kept
docs-only (unlinked, avoids double-instantiation). Lowercase
stub duplicates excluded. ERC: 1388 -> 770 violations.
Parts:
- renumbered C343 to C241, C344 to C242, C342 to C243, D19 to D14, J23 to J13, R167 to R153, R269 to R154, R270 to R155, R271 to R156, R272 to R157, R273 to R158, R274 to R159, R275 to R160, R276 to R161, R277 to R162, R278 to R163, R279 to R164, R280 to R165, R281 to R166, R121 to R167, R122 to R168, R120 to R169, U30 to U31, U31 to U32, U27 to U33

Commit message: block diagrame with Hierarchical labels and NVMe SSD footprint
Parts:
- renumbered D14 to D30
Connections:
- net J_uSD_CLK: now also U31.6 (NC)
- net J_uSD_CMD: now also U31.7 (NC)
- net J_uSD_D0: now also U32.10 (NC)
- net J_uSD_D1: now also U32.9 (NC)
- net J_uSD_D2: now also U31.10 (NC)
- net J_uSD_D3: now also U31.9 (NC)
- net J_uSD_DET: now also U32.7 (NC)
- net uSD_CLK renamed uSD.CLK
- net uSD_CMD renamed uSD.CMD
- net uSD_D0 renamed uSD.D0
- net uSD_D1 renamed uSD.D1
- net uSD_D2 renamed uSD.D2
- net uSD_D3 renamed uSD.D3
- no-connect marks 10 -> 3
